File: kicad/uart-rs232.sch (KiCad schematic (older format))
At the start: 10 parts, among them U2201 MAX3232

Commit message: BOM ist nun fast fertig
Parts:
- R40: renamed from R36; PriceEUR (none) -> 0.01
- R41: renamed from R37; PriceEUR (none) -> 0.01
- renumbered C2201 to C22, C2202 to C23, C2203 to C24, C2204 to C25, C2205 to C26, U2201 to U8

Commit message: BOM Fertig, 3D auch fast fertig. Ein paar Footrpints fehlen noch.
Parts:
- R52: renamed from R40; DistOrderNr (none) -> C113307; Distributor (none) -> LCSC; ManPartNr (none) -> RC1206JR-07100RL; Manufacturer (none) -> YAGEO; Notes (none) -> 100Ω ±5% 0.25W ±100ppm/℃ 1206 Chip Resistor; PriceEUR 0.01 -> 0.0037; PriceForQty (none) -> 500
- R53: renamed from R41; DistOrderNr (none) -> C113307; Distributor (none) -> LCSC; ManPartNr (none) -> RC1206JR-07100RL; Manufacturer (none) -> YAGEO; Notes (none) -> 100Ω ±5% 0.25W ±100ppm/℃ 1206 Chip Resistor; PriceEUR 0.01 -> 0.0037; PriceForQty (none) -> 500
- renumbered C22 to C33, C23 to C34, C24 to C35, C25 to C36, C26 to C37, D10 to D14, D11 to D15, U8 to U10
Changed lines of the file:
@@
 $Descr A4 11693 8268
 encoding utf-8
-Sheet 8 8
+Sheet 9 10
 Title "RS-232 Sniffer"
 Date "2020-11-13"
@@
 AR Path="/5FA85ABF/5F7FE44C/5F65EF92" Ref="U?"  Part="1"
 AR Path="/608DBC83/60A7272B/5F65EF92" Ref="U?"  Part="1"
-AR Path="/60A756E2/5F65EF92" Ref="U8"  Part="1"
-F 0 "U8" H 4850 4900 50  0000 C CNN
+AR Path="/60A756E2/5F65EF92" Ref="U10"  Part="1"
+F 0 "U10" H 4850 4900 50  0000 C CNN
 F 1 "MAX3232" H 4950 4800 50  0000 C CNN
 F 2 "Package_SO:SOIC-16_3.9x9.9mm_P1.27mm" H 5450 2650 50  0001 L CNN
@@
 AR Path="/5FA85ABF/5F7FE44C/5F65EF98" Ref="C?"  Part="1"
 AR Path="/608DBC83/60A7272B/5F65EF98" Ref="C?"  Part="1"
-AR Path="/60A756E2/5F65EF98" Ref="C24"  Part="1"
-F 0 "C24" H 6615 2996 50  0000 L CNN
+AR Path="/60A756E2/5F65EF98" Ref="C35"  Part="1"
+F 0 "C35" H 6615 2996 50  0000 L CNN
 F 1 "100n" H 6615 2905 50  0000 L CNN
 F 2 "Capacitor_SMD:C_1206_3216Metric" H 6538 2800 50  0001 C CNN
@@
 AR Path="/5FA85ABF/5F7FE44C/5F65EF9E" Ref="C?"  Part="1"
 AR Path="/608DBC83/60A7272B/5F65EF9E" Ref="C?"  Part="1"
-AR Path="/60A756E2/5F65EF9E" Ref="C22"  Part="1"
-F 0 "C22" H 4465 2996 50  0000 L CNN
+AR Path="/60A756E2/5F65EF9E" Ref="C33"  Part="1"
+F 0 "C33" H 4465 2996 50  0000 L CNN
 F 1 "100n" H 4465 2905 50  0000 L CNN
 F 2 "Capacitor_SMD:C_1206_3216Metric" H 4388 2800 50  0001 C CNN
@@
 AR Path="/5FA85ABF/5F7FE44C/5F65EFA4" Ref="C?"  Part="1"
 AR Path="/608DBC83/60A7272B/5F65EFA4" Ref="C?"  Part="1"
-AR Path="/60A756E2/5F65EFA4" Ref="C26"  Part="1"
-F 0 "C26" V 6748 3300 50  0000 C CNN
+AR Path="/60A756E2/5F65EFA4" Ref="C37"  Part="1"
+F 0 "C37" V 6748 3300 50  0000 C CNN
 F 1 "100n" V 6839 3300 50  0000 C CNN
 F 2 "Capacitor_SMD:C_1206_3216Metric" H 7038 3150 50  0001 C CNN
@@
 AR Path="/5FA85ABF/5F7FE44C/5F65EFAA" Ref="C?"  Part="1"
 AR Path="/608DBC83/60A7272B/5F65EFAA" Ref="C?"  Part="1"
-AR Path="/60A756E2/5F65EFAA" Ref="C25"  Part="1"
-F 0 "C25" V 6348 3600 50  0000 C CNN
+AR Path="/60A756E2/5F65EFAA" Ref="C36"  Part="1"
+F 0 "C36" V 6348 3600 50  0000 C CNN
 F 1 "100n" V 6439 3600 50  0000 C CNN
 F 2 "Capacitor_SMD:C_1206_3216Metric" H 6638 3450 50  0001 C CNN
@@
 AR Path="/5FA85ABF/5F7FE44C/5F65EFB3" Ref="#PWR?"  Part="1"
 AR Path="/608DBC83/60A7272B/5F65EFB3" Ref="#PWR?"  Part="1"
-AR Path="/60A756E2/5F65EFB3" Ref="#PWR040"  Part="1"
-F 0 "#PWR040" H 7250 3350 50  0001 C CNN
+AR Path="/60A756E2/5F65EFB3" Ref="#PWR062"  Part="1"
+F 0 "#PWR062" H 7250 3350 50  0001 C CNN
 F 1 "GND" V 7255 3472 50  0000 R CNN
 F 2 "" H 7250 3600 50  0001 C CNN
@@
 AR Path="/5FA85ABF/5F7FE44C/5F65EFB9" Ref="#PWR?"  Part="1"
 AR Path="/608DBC83/60A7272B/5F65EFB9" Ref="#PWR?"  Part="1"
-AR Path="/60A756E2/5F65EFB9" Ref="#PWR039"  Part="1"
-F 0 "#PWR039" H 7250 3050 50  0001 C CNN
+AR Path="/60A756E2/5F65EFB9" Ref="#PWR061"  Part="1"
+F 0 "#PWR061" H 7250 3050 50  0001 C CNN
 F 1 "GND" V 7255 3172 50  0000 R CNN
 F 2 "" H 7250 3300 50  0001 C CNN
@@
 AR Path="/5FA85ABF/5F7FE44C/5F65EFC4" Ref="C?"  Part="1"
 AR Path="/608DBC83/60A7272B/5F65EFC4" Ref="C?"  Part="1"
-AR Path="/60A756E2/5F65EFC4" Ref="C23"  Part="1"
-F 0 "C23" V 5598 2300 50  0000 C CNN
+AR Path="/60A756E2/5F65EFC4" Ref="C34"  Part="1"
+F 0 "C34" V 5598 2300 50  0000 C CNN
 F 1 "100n" V 5689 2300 50  0000 C CNN
 F 2 "Capacitor_SMD:C_1206_3216Metric" H 5888 2150 50  0001 C CNN
@@
 AR Path="/5FA85ABF/5F7FE44C/5F65EFCC" Ref="#PWR?"  Part="1"
 AR Path="/608DBC83/60A7272B/5F65EFCC" Ref="#PWR?"  Part="1"
-AR Path="/60A756E2/5F65EFCC" Ref="#PWR038"  Part="1"
-F 0 "#PWR038" H 6150 2050 50  0001 C CNN
+AR Path="/60A756E2/5F65EFCC" Ref="#PWR060"  Part="1"
+F 0 "#PWR060" H 6150 2050 50  0001 C CNN
 F 1 "GND" V 6155 2172 50  0000 R CNN
 F 2 "" H 6150 2300 50  0001 C CNN
@@
 Connection ~ 5400 2300
 $Comp
-L Device:R R40
+L Device:R R52
 U 1 1 60A93B20
 P 8500 3800
-F 0 "R40" V 8293 3800 50  0000 C CNN
+F 0 "R52" V 8293 3800 50  0000 C CNN
 F 1 "100R" V 8384 3800 50  0000 C CNN
 F 2 "Resistor_SMD:R_1206_3216Metric" V 8430 3800 50  0001 C CNN
 F 3 "~" H 8500 3800 50  0001 C CNN
-F 4 "0.01" H 8500 3800 50  0001 C CNN "PriceEUR"
+F 4 "0.0037" H 8500 3800 50  0001 C CNN "PriceEUR"
+F 5 "C113307" H 8500 3800 50  0001 C CNN "DistOrderNr"
+F 6 "LCSC" H 8500 3800 50  0001 C CNN "Distributor"
+F 7 "RC1206JR-07100RL" H 8500 3800 50  0001 C CNN "ManPartNr"
+F 8 "YAGEO" H 8500 3800 50  0001 C CNN "Manufacturer"
+F 9 "100Ω ±5% 0.25W ±100ppm/℃ 1206 Chip Resistor" H 8500 3800 50  0001 C CNN "Notes"
+F 10 "500" H 8500 3800 50  0001 C CNN "PriceForQty"
 	1    8500 3800
 	0    1    1    0
@@
 	8350 3800 7350 3800
 $Comp
-L Device:R R41
+L Device:R R53
 U 1 1 60A93ED5
 P 8500 4200
-F 0 "R41" V 8293 4200 50  0000 C CNN
+F 0 "R53" V 8293 4200 50  0000 C CNN
 F 1 "100R" V 8384 4200 50  0000 C CNN
 F 2 "Resistor_SMD:R_1206_3216Metric" V 8430 4200 50  0001 C CNN
 F 3 "~" H 8500 4200 50  0001 C CNN
-F 4 "0.01" H 8500 4200 50  0001 C CNN "PriceEUR"
+F 4 "0.0037" H 8500 4200 50  0001 C CNN "PriceEUR"
+F 5 "C113307" H 8500 4200 50  0001 C CNN "DistOrderNr"
+F 6 "LCSC" H 8500 4200 50  0001 C CNN "Distributor"
+F 7 "RC1206JR-07100RL" H 8500 4200 50  0001 C CNN "ManPartNr"
+F 8 "YAGEO" H 8500 4200 50  0001 C CNN "Manufacturer"
+F 9 "100Ω ±5% 0.25W ±100ppm/℃ 1206 Chip Resistor" H 8500 4200 50  0001 C CNN "Notes"
+F 10 "500" H 8500 4200 50  0001 C CNN "PriceForQty"
 	1    8500 4200
 	0    1    1    0
@@
 	8350 4200 8000 4200
 $Comp
-L htl_semiconductors:DiodeTVS_Bidirek D10
+L htl_semiconductors:DiodeTVS_Bidirek D14
 U 1 1 60A953FA
 P 7350 4800
-F 0 "D10" V 7312 4879 50  0000 L CNN
+F 0 "D14" V 7312 4879 50  0000 L CNN
 F 1 "SMAJ8.0CA" V 7396 4879 40  0000 L CNN
 F 2 "Diode_SMD:D_SMA" V 7434 4879 60  0001 L CNN
@@
 $EndComp
 $Comp
-L power:GNDPWR #PWR041
+L power:GNDPWR #PWR063
 U 1 1 60A9688D
 P 7350 5050
-F 0 "#PWR041" H 7350 4850 50  0001 C CNN
+F 0 "#PWR063" H 7350 4850 50  0001 C CNN
 F 1 "GNDPWR" H 7354 4896 50  0000 C CNN
 F 2 "" H 7350 5000 50  0001 C CNN
@@
 	7350 3800 6200 3800
 $Comp
-L htl_semiconductors:DiodeTVS_Bidirek D11
+L htl_semiconductors:DiodeTVS_Bidirek D15
 U 1 1 60A993E0
 P 8000 4800
-F 0 "D11" V 7962 4879 50  0000 L CNN
+F 0 "D15" V 7962 4879 50  0000 L CNN
 F 1 "SMAJ8.0CA" V 8046 4879 40  0000 L CNN
 F 2 "Diode_SMD:D_SMA" V 8084 4879 60  0001 L CNN
@@
 $EndComp
 $Comp
-L power:GNDPWR #PWR042
+L power:GNDPWR #PWR064
 U 1 1 60A993E6
 P 8000 5050
-F 0 "#PWR042" H 8000 4850 50  0001 C CNN
+F 0 "#PWR064" H 8000 4850 50  0001 C CNN
 F 1 "GNDPWR" H 8004 4896 50  0000 C CNN
 F 2 "" H 8000 5000 50  0001 C CNN
@@
 	5400 1950 5400 2300
 $Comp
-L power:GNDPWR #PWR037
+L power:GNDPWR #PWR059
 U 1 1 60A9F44C
 P 5400 5050
-F 0 "#PWR037" H 5400 4850 50  0001 C CNN
+F 0 "#PWR059" H 5400 4850 50  0001 C CNN
 F 1 "GNDPWR" H 5404 4896 50  0000 C CNN
 F 2 "" H 5400 5000 50  0001 C CNN
