File: kicad/dcdc-12v.sch (KiCad schematic (older format))
At the start: 12 parts, among them U7 XL7005A

Commit message: BOM ist nun fast fertig
Parts:
- D7: PriceEUR (none) -> 0.0067; PriceForQty (none) -> 50
- R32: renamed from R28; value 0R -> 100R; PriceEUR (none) -> 0.01
- R33: renamed from R29; PriceEUR (none) -> 0.01
- R34: renamed from R30; PriceEUR (none) -> 0.01
- R35: renamed from R31; PriceEUR (none) -> 0.01
- U6: renamed from U7; ManPartNr (none) -> XL7005A; Manufacturer (none) -> XLSEMI; Notes (none) -> 80V 400mA SOP-8_EP_150mil DC-DC Converters; Weblink (none) -> https://lcsc.com/product-detail/DC-DC-Converters_XLSEMI-XL7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
Changed lines of the file:
@@
 AR Path="/608DBC83/60A5D76C" Ref="U?"  Part="1"
 AR Path="/608DBC83/60A447A8/60A5D76C" Ref="U?"  Part="1"
-AR Path="/608DBC83/60A427AE/60A5D76C" Ref="U7"  Part="1"
-F 0 "U7" H 5381 3915 50  0000 C CNN
+AR Path="/608DBC83/60A427AE/60A5D76C" Ref="U6"  Part="1"
+F 0 "U6" H 5381 3915 50  0000 C CNN
 F 1 "XL7005A" H 5381 3824 50  0000 C CNN
 F 2 "htl_smd:SOIC-8-1EP_3.9x4.9mm_P1.27mm_EP2.514x3.2mm_ThermalVias" H 5400 2400 50  0001 C CNN
@@
 F 6 "0.204" H 5350 3550 50  0001 C CNN "PriceEUR"
 F 7 "100" H 5350 3550 50  0001 C CNN "PriceForQty"
+F 8 "XL7005A" H 5350 3550 50  0001 C CNN "ManPartNr"
+F 9 "XLSEMI" H 5350 3550 50  0001 C CNN "Manufacturer"
+F 10 "80V 400mA SOP-8_EP_150mil DC-DC Converters" H 5350 3550 50  0001 C CNN "Notes"
+F 11 "https://lcsc.com/product-detail/DC-DC-Converters_XLSEMI-XL7005A_C50848.html" H 5350 3550 50  0001 C CNN "Weblink"
 	1    5350 3550
 	1    0    0    -1
@@
 AR Path="/608DBC83/60A5D783" Ref="R?"  Part="1"
 AR Path="/608DBC83/60A447A8/60A5D783" Ref="R?"  Part="1"
-AR Path="/608DBC83/60A427AE/60A5D783" Ref="R29"  Part="1"
-F 0 "R29" H 6670 3696 50  0000 L CNN
+AR Path="/608DBC83/60A427AE/60A5D783" Ref="R33"  Part="1"
+F 0 "R33" H 6670 3696 50  0000 L CNN
 F 1 "30k" H 6670 3605 50  0000 L CNN
 F 2 "Resistor_SMD:R_1206_3216Metric" V 6530 3650 50  0001 C CNN
 F 3 "~" H 6600 3650 50  0001 C CNN
+F 4 "0.01" H 6600 3650 50  0001 C CNN "PriceEUR"
 	1    6600 3650
 	1    0    0    -1
@@
 AR Path="/608DBC83/60A5D789" Ref="R?"  Part="1"
 AR Path="/608DBC83/60A447A8/60A5D789" Ref="R?"  Part="1"
-AR Path="/608DBC83/60A427AE/60A5D789" Ref="R30"  Part="1"
-F 0 "R30" H 6670 4296 50  0000 L CNN
+AR Path="/608DBC83/60A427AE/60A5D789" Ref="R34"  Part="1"
+F 0 "R34" H 6670 4296 50  0000 L CNN
 F 1 "3k3" H 6670 4205 50  0000 L CNN
 F 2 "Resistor_SMD:R_1206_3216Metric" V 6530 4250 50  0001 C CNN
 F 3 "~" H 6600 4250 50  0001 C CNN
+F 4 "0.01" H 6600 4250 50  0001 C CNN "PriceEUR"
 	1    6600 4250
 	1    0    0    -1
@@
 AR Path="/608DBC83/60A5D7E4" Ref="R?"  Part="1"
 AR Path="/608DBC83/60A447A8/60A5D7E4" Ref="R?"  Part="1"
-AR Path="/608DBC83/60A427AE/60A5D7E4" Ref="R28"  Part="1"
-F 0 "R28" H 4870 4296 50  0000 L CNN
-F 1 "0R" H 4870 4205 50  0000 L CNN
+AR Path="/608DBC83/60A427AE/60A5D7E4" Ref="R32"  Part="1"
+F 0 "R32" H 4870 4296 50  0000 L CNN
+F 1 "100R" H 4870 4205 50  0000 L CNN
 F 2 "Resistor_SMD:R_1206_3216Metric" V 4730 4250 50  0001 C CNN
 F 3 "~" H 4800 4250 50  0001 C CNN
+F 4 "0.01" H 4800 4250 50  0001 C CNN "PriceEUR"
 	1    4800 4250
 	1    0    0    -1
@@
 AR Path="/608DBC83/60A5D7EC" Ref="R?"  Part="1"
 AR Path="/608DBC83/60A447A8/60A5D7EC" Ref="R?"  Part="1"
-AR Path="/608DBC83/60A427AE/60A5D7EC" Ref="R31"  Part="1"
-F 0 "R31" H 8220 3846 50  0000 L CNN
+AR Path="/608DBC83/60A427AE/60A5D7EC" Ref="R35"  Part="1"
+F 0 "R35" H 8220 3846 50  0000 L CNN
 F 1 "3k3" H 8220 3755 50  0000 L CNN
 F 2 "Resistor_SMD:R_1206_3216Metric" V 8080 3800 50  0001 C CNN
 F 3 "~" H 8150 3800 50  0001 C CNN
+F 4 "0.01" H 8150 3800 50  0001 C CNN "PriceEUR"
 	1    8150 3800
 	1    0    0    -1
@@
 F 5 "C965825" H 8150 4300 50  0001 C CNN "DistOrderNr"
 F 6 "https://lcsc.com/product-detail/Pre-ordered-Products_XINGLIGHT-XL-3216UGC_C965825.html" H 8150 4300 50  0001 C CNN "Weblink"
+F 7 "0.0067" H 8150 4300 50  0001 C CNN "PriceEUR"
+F 8 "50" H 8150 4300 50  0001 C CNN "PriceForQty"
 	1    8150 4300
 	0    -1   -1   0

Commit message: BOM Fertig, 3D auch fast fertig. Ein paar Footrpints fehlen noch.
Parts:
- C28: renamed from C17; footprint TODO -> Capacitor_SMD:CP_Elec_6.3x5.9; DistOrderNr C454667 -> C320569; ManPartNr EEHZA1E101XV -> SVZ1EM101E06E00RAXXX; Manufacturer Panasonic -> AISHI; Notes 100uF ±20% 25V 7.7mm 8mm 2A @ 100kHz 30mΩ @ 100kHz 10000hrs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 -> 100uF ±20% 25V 6.3mm 6mm 2000hrs @ 105℃ -55℃~+105℃ SMD,6.3x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; PriceEUR 0.4258 -> 0.1485; PriceForQty 100 -> 30
- L1: footprint Inductor_SMD:L_7.3x7.3_H4.5_TODO -> Inductor_SMD:L_7.3x7.3_H4.5
- R44: renamed from R32; DistOrderNr (none) -> C113307; Distributor (none) -> LCSC; ManPartNr (none) -> RC1206JR-07100RL; Manufacturer (none) -> YAGEO; Notes (none) -> 100Ω ±5% 0.25W ±100ppm/℃ 1206 Chip Resistor; PriceEUR 0.01 -> 0.0037; PriceForQty (none) -> 500
- R45: renamed from R33; DistOrderNr (none) -> C137314; Distributor (none) -> LCSC
- R46: renamed from R34; DistOrderNr (none) -> C229599; Distributor (none) -> LCSC
- R47: renamed from R35; DistOrderNr (none) -> C229599; Distributor (none) -> LCSC
- renumbered C14 to C25, C15 to C26, C16 to C27, D6 to D10, D7 to D11, U6 to U8
Other:
- note added: "TODO: check footprint!"
Changed lines of the file:
@@
 $Descr A4 11693 8268
 encoding utf-8
-Sheet 6 8
+Sheet 7 10
 Title ""
 Date ""
@@
 AR Path="/608DBC83/60A5D76C" Ref="U?"  Part="1"
 AR Path="/608DBC83/60A447A8/60A5D76C" Ref="U?"  Part="1"
-AR Path="/608DBC83/60A427AE/60A5D76C" Ref="U6"  Part="1"
-F 0 "U6" H 5381 3915 50  0000 C CNN
+AR Path="/608DBC83/60A427AE/60A5D76C" Ref="U8"  Part="1"
+F 0 "U8" H 5381 3915 50  0000 C CNN
 F 1 "XL7005A" H 5381 3824 50  0000 C CNN
 F 2 "htl_smd:SOIC-8-1EP_3.9x4.9mm_P1.27mm_EP2.514x3.2mm_ThermalVias" H 5400 2400 50  0001 C CNN
@@
 F 0 "L1" H 6250 3665 50  0000 C CNN
 F 1 "47u/1A" H 6250 3574 50  0000 C CNN
-F 2 "Inductor_SMD:L_7.3x7.3_H4.5_TODO" H 6250 3450 50  0001 C CNN
+F 2 "Inductor_SMD:L_7.3x7.3_H4.5" H 6250 3450 50  0001 C CNN
 F 3 "~" H 6250 3450 50  0001 C CNN
 F 4 "LCSC" H 6250 3450 50  0001 C CNN "Distributor"
@@
 AR Path="/608DBC83/60A5D77D" Ref="D?"  Part="1"
 AR Path="/608DBC83/60A447A8/60A5D77D" Ref="D?"  Part="1"
-AR Path="/608DBC83/60A427AE/60A5D77D" Ref="D6"  Part="1"
-F 0 "D6" V 5854 4229 50  0000 L CNN
+AR Path="/608DBC83/60A427AE/60A5D77D" Ref="D10"  Part="1"
+F 0 "D10" V 5854 4229 50  0000 L CNN
 F 1 "SS210" V 5945 4229 50  0000 L CNN
 F 2 "Diode_SMD:D_SMA" H 5900 4150 50  0001 C CNN
@@
 AR Path="/608DBC83/60A5D783" Ref="R?"  Part="1"
 AR Path="/608DBC83/60A447A8/60A5D783" Ref="R?"  Part="1"
-AR Path="/608DBC83/60A427AE/60A5D783" Ref="R33"  Part="1"
-F 0 "R33" H 6670 3696 50  0000 L CNN
+AR Path="/608DBC83/60A427AE/60A5D783" Ref="R45"  Part="1"
+F 0 "R45" H 6670 3696 50  0000 L CNN
 F 1 "30k" H 6670 3605 50  0000 L CNN
 F 2 "Resistor_SMD:R_1206_3216Metric" V 6530 3650 50  0001 C CNN
 F 3 "~" H 6600 3650 50  0001 C CNN
 F 4 "0.01" H 6600 3650 50  0001 C CNN "PriceEUR"
+F 5 "C137314" H 6600 3650 50  0001 C CNN "DistOrderNr"
+F 6 "LCSC" H 6600 3650 50  0001 C CNN "Distributor"
 	1    6600 3650
 	1    0    0    -1
@@
 AR Path="/608DBC83/60A5D789" Ref="R?"  Part="1"
 AR Path="/608DBC83/60A447A8/60A5D789" Ref="R?"  Part="1"
-AR Path="/608DBC83/60A427AE/60A5D789" Ref="R34"  Part="1"
-F 0 "R34" H 6670 4296 50  0000 L CNN
+AR Path="/608DBC83/60A427AE/60A5D789" Ref="R46"  Part="1"
+F 0 "R46" H 6670 4296 50  0000 L CNN
 F 1 "3k3" H 6670 4205 50  0000 L CNN
 F 2 "Resistor_SMD:R_1206_3216Metric" V 6530 4250 50  0001 C CNN
 F 3 "~" H 6600 4250 50  0001 C CNN
 F 4 "0.01" H 6600 4250 50  0001 C CNN "PriceEUR"
+F 5 "C229599" H 6600 4250 50  0001 C CNN "DistOrderNr"
+F 6 "LCSC" H 6600 4250 50  0001 C CNN "Distributor"
 	1    6600 4250
 	1    0    0    -1
@@
 AR Path="/608DBC83/60A5D794" Ref="C?"  Part="1"
 AR Path="/608DBC83/60A447A8/60A5D794" Ref="C?"  Part="1"
-AR Path="/608DBC83/60A427AE/60A5D794" Ref="C16"  Part="1"
-F 0 "C16" H 7065 3696 50  0000 L CNN
+AR Path="/608DBC83/60A427AE/60A5D794" Ref="C27"  Part="1"
+F 0 "C27" H 7065 3696 50  0000 L CNN
 F 1 "33n" H 7065 3605 50  0000 L CNN
 F 2 "Capacitor_SMD:C_1206_3216Metric" H 6988 3500 50  0001 C CNN
@@
 AR Path="/608DBC83/60A5D79C" Ref="C?"  Part="1"
 AR Path="/608DBC83/60A447A8/60A5D79C" Ref="C?"  Part="1"
-AR Path="/608DBC83/60A427AE/60A5D79C" Ref="C15"  Part="1"
-F 0 "C15" H 4318 4046 50  0000 L CNN
+AR Path="/608DBC83/60A427AE/60A5D79C" Ref="C26"  Part="1"
+F 0 "C26" H 4318 4046 50  0000 L CNN
 F 1 "100u/63V" H 4318 3955 50  0000 L CNN
 F 2 "Capacitor_SMD:CP_Elec_8x10" H 4238 3850 50  0001 C CNN
@@
 AR Path="/608DBC83/60A5D7A2" Ref="C?"  Part="1"
 AR Path="/608DBC83/60A447A8/60A5D7A2" Ref="C?"  Part="1"
-AR Path="/608DBC83/60A427AE/60A5D7A2" Ref="C17"  Part="1"
-F 0 "C17" H 7418 4246 50  0000 L CNN
+AR Path="/608DBC83/60A427AE/60A5D7A2" Ref="C28"  Part="1"
+F 0 "C28" H 7418 4246 50  0000 L CNN
 F 1 "100u/25V" H 7418 4155 50  0000 L CNN
-F 2 "TODO" H 7338 4050 50  0001 C CNN
+F 2 "Capacitor_SMD:CP_Elec_6.3x5.9" H 7338 4050 50  0001 C CNN
 F 3 "~" H 7300 4200 50  0001 C CNN
-F 4 "C454667" H 7300 4200 50  0001 C CNN "DistOrderNr"
+F 4 "C320569" H 7300 4200 50  0001 C CNN "DistOrderNr"
 F 5 "LCSC" H 7300 4200 50  0001 C CNN "Distributor"
-F 6 "EEHZA1E101XV" H 7300 4200 50  0001 C CNN "ManPartNr"
-F 7 "Panasonic" H 7300 4200 50  0001 C CNN "Manufacturer"
-F 8 "100uF ±20% 25V 7.7mm 8mm 2A @ 100kHz 30mΩ @ 100kHz 10000hrs @ 105℃ -55℃~+105℃ SMD,7.7x8mm Solid Polymer Electrolytic Capacitor" H 7300 4200 50  0001 C CNN "Notes"
-F 9 "0.4258" H 7300 4200 50  0001 C CNN "PriceEUR"
-F 10 "100" H 7300 4200 50  0001 C CNN "PriceForQty"
+F 6 "SVZ1EM101E06E00RAXXX" H 7300 4200 50  0001 C CNN "ManPartNr"
+F 7 "AISHI" H 7300 4200 50  0001 C CNN "Manufacturer"
+F 8 "100uF ±20% 25V 6.3mm 6mm 2000hrs @ 105℃ -55℃~+105℃ SMD,6.3x6mm Solid Polymer Electrolytic Capacitor" H 7300 4200 50  0001 C CNN "Notes"
+F 9 "0.1485" H 7300 4200 50  0001 C CNN "PriceEUR"
+F 10 "30" H 7300 4200 50  0001 C CNN "PriceForQty"
 	1    7300 4200
 	1    0    0    -1
@@
 AR Path="/608DBC83/60A5D7A8" Ref="C?"  Part="1"
 AR Path="/608DBC83/60A447A8/60A5D7A8" Ref="C?"  Part="1"
-AR Path="/608DBC83/60A427AE/60A5D7A8" Ref="C14"  Part="1"
-F 0 "C14" H 3915 4046 50  0000 L CNN
+AR Path="/608DBC83/60A427AE/60A5D7A8" Ref="C25"  Part="1"
+F 0 "C25" H 3915 4046 50  0000 L CNN
 F 1 "100n/100V" H 3915 3955 50  0000 L CNN
 F 2 "Capacitor_SMD:C_1206_3216Metric" H 3838 3850 50  0001 C CNN
@@
 AR Path="/608DBC83/60A5D7E4" Ref="R?"  Part="1"
 AR Path="/608DBC83/60A447A8/60A5D7E4" Ref="R?"  Part="1"
-AR Path="/608DBC83/60A427AE/60A5D7E4" Ref="R32"  Part="1"
-F 0 "R32" H 4870 4296 50  0000 L CNN
+AR Path="/608DBC83/60A427AE/60A5D7E4" Ref="R44"  Part="1"
+F 0 "R44" H 4870 4296 50  0000 L CNN
 F 1 "100R" H 4870 4205 50  0000 L CNN
 F 2 "Resistor_SMD:R_1206_3216Metric" V 4730 4250 50  0001 C CNN
 F 3 "~" H 4800 4250 50  0001 C CNN
-F 4 "0.01" H 4800 4250 50  0001 C CNN "PriceEUR"
+F 4 "0.0037" H 4800 4250 50  0001 C CNN "PriceEUR"
+F 5 "C113307" H 4800 4250 50  0001 C CNN "DistOrderNr"
+F 6 "LCSC" H 4800 4250 50  0001 C CNN "Distributor"
+F 7 "RC1206JR-07100RL" H 4800 4250 50  0001 C CNN "ManPartNr"
+F 8 "YAGEO" H 4800 4250 50  0001 C CNN "Manufacturer"
+F 9 "100Ω ±5% 0.25W ±100ppm/℃ 1206 Chip Resistor" H 4800 4250 50  0001 C CNN "Notes"
+F 10 "500" H 4800 4250 50  0001 C CNN "PriceForQty"
 	1    4800 4250
 	1    0    0    -1
@@
 AR Path="/608DBC83/60A5D7EC" Ref="R?"  Part="1"
 AR Path="/608DBC83/60A447A8/60A5D7EC" Ref="R?"  Part="1"
-AR Path="/608DBC83/60A427AE/60A5D7EC" Ref="R35"  Part="1"
-F 0 "R35" H 8220 3846 50  0000 L CNN
+AR Path="/608DBC83/60A427AE/60A5D7EC" Ref="R47"  Part="1"
+F 0 "R47" H 8220 3846 50  0000 L CNN
 F 1 "3k3" H 8220 3755 50  0000 L CNN
 F 2 "Resistor_SMD:R_1206_3216Metric" V 8080 3800 50  0001 C CNN
 F 3 "~" H 8150 3800 50  0001 C CNN
 F 4 "0.01" H 8150 3800 50  0001 C CNN "PriceEUR"
+F 5 "C229599" H 8150 3800 50  0001 C CNN "DistOrderNr"
+F 6 "LCSC" H 8150 3800 50  0001 C CNN "Distributor"
 	1    8150 3800
 	1    0    0    -1
@@
 AR Path="/608DBC83/60A5D7F6" Ref="D?"  Part="1"
 AR Path="/608DBC83/60A447A8/60A5D7F6" Ref="D?"  Part="1"
-AR Path="/608DBC83/60A427AE/60A5D7F6" Ref="D7"  Part="1"
-F 0 "D7" V 8189 4182 50  0000 R CNN
+AR Path="/608DBC83/60A427AE/60A5D7F6" Ref="D11"  Part="1"
+F 0 "D11" V 8189 4182 50  0000 R CNN
 F 1 "grün" V 8098 4182 50  0000 R CNN
 F 2 "LED_SMD:LED_1206_3216Metric" H 8150 4300 50  0001 C CNN
@@
 P 3500 4600
 AR Path="/608DBC83/60A447A8/60A5D7FE" Ref="#PWR?"  Part="1"
-AR Path="/608DBC83/60A427AE/60A5D7FE" Ref="#PWR033"  Part="1"
-F 0 "#PWR033" H 3500 4400 50  0001 C CNN
+AR Path="/608DBC83/60A427AE/60A5D7FE" Ref="#PWR055"  Part="1"
+F 0 "#PWR055" H 3500 4400 50  0001 C CNN
 F 1 "GNDPWR" H 3504 4446 50  0000 C CNN
 F 2 "" H 3500 4550 50  0001 C CNN
@@
 P 8450 4600
 AR Path="/608DBC83/60A447A8/60A5D815" Ref="#PWR?"  Part="1"
-AR Path="/608DBC83/60A427AE/60A5D815" Ref="#PWR034"  Part="1"
-F 0 "#PWR034" H 8450 4400 50  0001 C CNN
+AR Path="/608DBC83/60A427AE/60A5D815" Ref="#PWR056"  Part="1"
+F 0 "#PWR056" H 8450 4400 50  0001 C CNN
 F 1 "GNDPWR" H 8454 4446 50  0000 C CNN
 F 2 "" H 8450 4550 50  0001 C CNN
@@
 Wire Wire Line
 	7300 3450 8150 3450
+Text Notes 5900 3150 0    50   ~ 0
+TODO: check footprint!
 $EndSCHEMATC

Commit message: kleinere Updates im Schaltplan
Parts:
- C26, C28: symbol Device:CP -> jbc-miniregler-rescue:CP-Device
Changed lines of the file:
@@
 	4800 3850 4800 4100
 $Comp
-L Device:CP C?
+L jbc-miniregler-rescue:CP-Device C?
 U 1 1 60A5D79C
 P 4200 4000
@@
 $EndComp
 $Comp
-L Device:CP C?
+L jbc-miniregler-rescue:CP-Device C?
 U 1 1 60A5D7A2
 P 7300 4200

Commit message: wip
Connections:
- net labels added: fb, sw, ~en
- wire segments 50 -> 51
Changed lines of the file:
@@
 	3800 4600 3800 4150
 Wire Wire Line
-	5200 4250 5200 4350
+	5150 4250 5150 4350
 Wire Wire Line
-	5200 4350 5300 4350
+	5450 4350 5450 4250
 Wire Wire Line
-	5500 4350 5500 4250
+	5350 4250 5350 4350
+Connection ~ 5350 4350
 Wire Wire Line
-	5400 4250 5400 4350
-Connection ~ 5400 4350
+	5350 4350 5450 4350
 Wire Wire Line
-	5400 4350 5500 4350
-Wire Wire Line
-	5300 4250 5300 4350
-Connection ~ 5300 4350
-Wire Wire Line
-	5300 4350 5350 4350
+	5250 4250 5250 4350
 Wire Wire Line
 	5350 4600 5350 4350
-Connection ~ 5350 4350
-Wire Wire Line
-	5350 4350 5400 4350
 Wire Wire Line
 	5750 3850 6600 3850
@@
 	4200 4600 4800 4600
 Connection ~ 4800 4600
-Wire Wire Line
-	4800 4600 5350 4600
-Connection ~ 5350 4600
-Wire Wire Line
-	5350 4600 5900 4600
 Connection ~ 5900 4600
 Wire Wire Line
@@
 Text Notes 5900 3150 0    50   ~ 0
 TODO: check footprint!
+Wire Wire Line
+	5150 4350 5250 4350
+Connection ~ 5250 4350
+Connection ~ 5350 4600
+Wire Wire Line
+	5350 4600 5900 4600
+Wire Wire Line
+	5250 4350 5350 4350
+Wire Wire Line
+	4800 4600 5350 4600
+Wire Wire Line
+	5450 4350 5550 4350
+Wire Wire Line
+	5550 4350 5550 4250
+Connection ~ 5450 4350
+Text Label 5750 3450 0    50   ~ 0
+sw
+Text Label 5950 3850 0    50   ~ 0
+fb
+Text Label 4800 3850 0    50   ~ 0
+~en
 $EndSCHEMATC

Commit message: WIP Layout, TODO: DRC
Parts:
- D10: footprint Diode_SMD:D_SMA -> htl_smd:D_SMA_wide
- L1: footprint Inductor_SMD:L_7.3x7.3_H4.5 -> htl_smd:L_7.3x7.3_H4.5_C216198
Connections:
- net GNDPWR: no longer D11.1 (K)
- new net GND: D11.1 (K)
Other:
- note removed: "TODO: check footprint!"
- moved on the sheet: D11
Changed lines of the file:
@@
 F 0 "L1" H 6250 3665 50  0000 C CNN
 F 1 "47u/1A" H 6250 3574 50  0000 C CNN
-F 2 "Inductor_SMD:L_7.3x7.3_H4.5" H 6250 3450 50  0001 C CNN
+F 2 "htl_smd:L_7.3x7.3_H4.5_C216198" H 6250 3450 50  0001 C CNN
 F 3 "~" H 6250 3450 50  0001 C CNN
 F 4 "LCSC" H 6250 3450 50  0001 C CNN "Distributor"
@@
 F 0 "D10" V 5854 4229 50  0000 L CNN
 F 1 "SS210" V 5945 4229 50  0000 L CNN
-F 2 "Diode_SMD:D_SMA" H 5900 4150 50  0001 C CNN
+F 2 "htl_smd:D_SMA_wide" H 5900 4150 50  0001 C CNN
 F 3 "~" H 5900 4150 50  0001 C CNN
 F 4 "C2683692" H 5900 4150 50  0001 C CNN "DistOrderNr"
@@
 L Device:LED D?
 U 1 1 60A5D7F6
-P 8150 4300
+P 8150 4150
 AR Path="/608DBC83/60A5D7F6" Ref="D?"  Part="1"
 AR Path="/608DBC83/60A447A8/60A5D7F6" Ref="D?"  Part="1"
 AR Path="/608DBC83/60A427AE/60A5D7F6" Ref="D11"  Part="1"
-F 0 "D11" V 8189 4182 50  0000 R CNN
-F 1 "grün" V 8098 4182 50  0000 R CNN
-F 2 "LED_SMD:LED_1206_3216Metric" H 8150 4300 50  0001 C CNN
-F 3 "~" H 8150 4300 50  0001 C CNN
-F 4 "LCSC" H 8150 4300 50  0001 C CNN "Distributor"
-F 5 "C965825" H 8150 4300 50  0001 C CNN "DistOrderNr"
-F 6 "https://lcsc.com/product-detail/Pre-ordered-Products_XINGLIGHT-XL-3216UGC_C965825.html" H 8150 4300 50  0001 C CNN "Weblink"
-F 7 "0.0067" H 8150 4300 50  0001 C CNN "PriceEUR"
-F 8 "50" H 8150 4300 50  0001 C CNN "PriceForQty"
-	1    8150 4300
+F 0 "D11" V 8189 4032 50  0000 R CNN
+F 1 "grün" V 8098 4032 50  0000 R CNN
+F 2 "LED_SMD:LED_1206_3216Metric" H 8150 4150 50  0001 C CNN
+F 3 "~" H 8150 4150 50  0001 C CNN
+F 4 "LCSC" H 8150 4150 50  0001 C CNN "Distributor"
+F 5 "C965825" H 8150 4150 50  0001 C CNN "DistOrderNr"
+F 6 "https://lcsc.com/product-detail/Pre-ordered-Products_XINGLIGHT-XL-3216UGC_C965825.html" H 8150 4150 50  0001 C CNN "Weblink"
+F 7 "0.0067" H 8150 4150 50  0001 C CNN "PriceEUR"
+F 8 "50" H 8150 4150 50  0001 C CNN "PriceForQty"
+	1    8150 4150
 	0    -1   -1   0
 $EndComp
 Wire Wire Line
-	8150 4600 8150 4450
-Wire Wire Line
-	8150 4150 8150 3950
+	8150 4000 8150 3950
 $Comp
 L power:GNDPWR #PWR?
@@
 	6600 4600 7300 4600
 Connection ~ 7300 4600
-Wire Wire Line
-	7300 4600 8150 4600
-Connection ~ 8150 4600
-Wire Wire Line
-	8150 4600 8450 4600
 $Comp
 L power:GNDPWR #PWR?
@@
 Wire Wire Line
 	7300 3450 8150 3450
-Text Notes 5900 3150 0    50   ~ 0
-TODO: check footprint!
 Wire Wire Line
 	5150 4350 5250 4350
@@
 Text Label 4800 3850 0    50   ~ 0
 ~en
+Wire Wire Line
+	7300 4600 8450 4600
+$Comp
+L power:GND #PWR?
+U 1 1 60BCD9D3
+P 8150 4300
+F 0 "#PWR?" H 8150 4050 50  0001 C CNN
+F 1 "GND" H 8155 4127 50  0000 C CNN
+F 2 "" H 8150 4300 50  0001 C CNN
+F 3 "" H 8150 4300 50  0001 C CNN
+	1    8150 4300
+	1    0    0    -1
+$EndComp
 $EndSCHEMATC

Commit message: wip, bugfixes für v21.0.1
Parts:
- R44: DistOrderNr C113307 -> C245445; ManPartNr RC1206JR-07100RL -> CR1206F100RP05Z; Manufacturer YAGEO -> Ever Ohms Tech; Notes 100Ω ±5% 0.25W ±100ppm/℃ 1206 Chip Resistor -> 0.25W ±1% ±100ppm/℃ 100Ω 1206; PriceEUR 0.0037 -> 0.0030
Changed lines of the file:
@@
 Sheet 7 10
 Title "HTL Lötregler Mini"
-Date "2021-06-01"
-Rev "21.0.0"
+Date "2021-09-22"
+Rev "21.0.1-dev"
 Comp "HTL Steyr"
 Comment1 "Prof. Karl Zeilhofer et al."
@@
 F 2 "Resistor_SMD:R_1206_3216Metric" V 4730 4250 50  0001 C CNN
 F 3 "~" H 4800 4250 50  0001 C CNN
-F 4 "0.0037" H 4800 4250 50  0001 C CNN "PriceEUR"
-F 5 "C113307" H 4800 4250 50  0001 C CNN "DistOrderNr"
+F 4 "0.0030" H 4800 4250 50  0001 C CNN "PriceEUR"
+F 5 "C245445" H 4800 4250 50  0001 C CNN "DistOrderNr"
 F 6 "LCSC" H 4800 4250 50  0001 C CNN "Distributor"
-F 7 "RC1206JR-07100RL" H 4800 4250 50  0001 C CNN "ManPartNr"
-F 8 "YAGEO" H 4800 4250 50  0001 C CNN "Manufacturer"
-F 9 "100Ω ±5% 0.25W ±100ppm/℃ 1206 Chip Resistor" H 4800 4250 50  0001 C CNN "Notes"
+F 7 "CR1206F100RP05Z" H 4800 4250 50  0001 C CNN "ManPartNr"
+F 8 "Ever Ohms Tech" H 4800 4250 50  0001 C CNN "Manufacturer"
+F 9 "0.25W ±1% ±100ppm/℃ 100Ω 1206" H 4800 4250 50  0001 C CNN "Notes"
 F 10 "500" H 4800 4250 50  0001 C CNN "PriceForQty"
 	1    4800 4250
