File: kicad/dcdc-12v.sch (KiCad schematic (older format))
At the start: 12 parts, among them U8 XL7005A

Commit message: BOM aktualisiert, Zenerdiode: Pinout IPC-konform gestaltet, ...
siehe https://gitlab.com/kicad/libraries/kicad-symbols/-/issues/3157
Parts:
- C25: Index (none) -> 2
- C26: Index (none) -> 43
- C27: Index (none) -> 31
- C28: Index (none) -> 34
- D10: Index (none) -> 49
- D11: Index (none) -> 47
- L1: Index (none) -> 24
- R44: Index (none) -> 28
- R45: Index (none) -> 17
- R46, R47: Index (none) -> 26
- U8: Index (none) -> 9
Changed lines of the file:
@@
 F 10 "80V 400mA SOP-8_EP_150mil DC-DC Converters" H 5350 3550 50  0001 C CNN "Notes"
 F 11 "https://lcsc.com/product-detail/DC-DC-Converters_XLSEMI-XL7005A_C50848.html" H 5350 3550 50  0001 C CNN "Weblink"
+F 12 "9" H 5350 3550 50  0001 C CNN "Index"
 	1    5350 3550
 	1    0    0    -1
@@
 F 10 "Sunltech Tech" H 6250 3450 50  0001 C CNN "Manufacturer"
 F 11 "47uH ±20% 1A 266mΩ SMD,7.3x7.3x4.5mm" H 6250 3450 50  0001 C CNN "Notes"
+F 12 "24" H 6250 3450 50  0001 C CNN "Index"
 	1    6250 3450
 	1    0    0    -1
@@
 F 10 "200" H 5900 4150 50  0001 C CNN "PriceForQty"
 F 11 "https://lcsc.com/product-detail/Schottky-Barrier-Diodes-SBD_ZHIDE-SS210A-W_C2683692.html" H 5900 4150 50  0001 C CNN "Weblink"
+F 12 "49" H 5900 4150 50  0001 C CNN "Index"
 	1    5900 4150
 	0    1    1    0
@@
 F 5 "C137314" H 6600 3650 50  0001 C CNN "DistOrderNr"
 F 6 "LCSC" H 6600 3650 50  0001 C CNN "Distributor"
+F 7 "17" H 6600 3650 50  0001 C CNN "Index"
 	1    6600 3650
 	1    0    0    -1
@@
 F 5 "C229599" H 6600 4250 50  0001 C CNN "DistOrderNr"
 F 6 "LCSC" H 6600 4250 50  0001 C CNN "Distributor"
+F 7 "26" H 6600 4250 50  0001 C CNN "Index"
 	1    6600 4250
 	1    0    0    -1
@@
 F 8 "0.0144" H 6950 3650 50  0001 C CNN "PriceEUR"
 F 9 "50" H 6950 3650 50  0001 C CNN "PriceForQty"
+F 10 "31" H 6950 3650 50  0001 C CNN "Index"
 	1    6950 3650
 	1    0    0    -1
@@
 F 9 "0.0698" H 4200 4000 50  0001 C CNN "PriceEUR"
 F 10 "150" H 4200 4000 50  0001 C CNN "PriceForQty"
+F 11 "43" H 4200 4000 50  0001 C CNN "Index"
 	1    4200 4000
 	1    0    0    -1
@@
 F 9 "0.1485" H 7300 4200 50  0001 C CNN "PriceEUR"
 F 10 "30" H 7300 4200 50  0001 C CNN "PriceForQty"
+F 11 "34" H 7300 4200 50  0001 C CNN "Index"
 	1    7300 4200
 	1    0    0    -1
@@
 F 9 "0.014" H 3800 4000 50  0001 C CNN "PriceEUR"
 F 10 "200" H 3800 4000 50  0001 C CNN "PriceForQty"
+F 11 "2" H 3800 4000 50  0001 C CNN "Index"
 	1    3800 4000
 	-1   0    0    -1
@@
 F 9 "0.25W ±1% ±100ppm/℃ 100Ω 1206" H 4800 4250 50  0001 C CNN "Notes"
 F 10 "500" H 4800 4250 50  0001 C CNN "PriceForQty"
+F 11 "28" H 4800 4250 50  0001 C CNN "Index"
 	1    4800 4250
 	1    0    0    -1
@@
 F 5 "C229599" H 8150 3800 50  0001 C CNN "DistOrderNr"
 F 6 "LCSC" H 8150 3800 50  0001 C CNN "Distributor"
+F 7 "26" H 8150 3800 50  0001 C CNN "Index"
 	1    8150 3800
 	1    0    0    -1
@@
 F 7 "0.0067" H 8150 4150 50  0001 C CNN "PriceEUR"
 F 8 "50" H 8150 4150 50  0001 C CNN "PriceForQty"
+F 9 "47" H 8150 4150 50  0001 C CNN "Index"
 	1    8150 4150
 	0    -1   -1   0
