File: kicad/dcdc-5v.sch (KiCad schematic (older format))
At the start: 12 parts, among them U8 XL7005A

Commit message: BOM ist nun fast fertig
Parts:
- D9: PriceEUR (none) -> 0.0067; PriceForQty (none) -> 50
- R36: renamed from R32; value 0R -> 100R; PriceEUR (none) -> 0.01
- R37: renamed from R33; PriceEUR (none) -> 0.01
- R38: renamed from R34; PriceEUR (none) -> 0.01
- R39: renamed from R35; PriceEUR (none) -> 0.01
- U7: renamed from U8; ManPartNr (none) -> XL7005A; Manufacturer (none) -> XLSEMI; Notes (none) -> 80V 400mA SOP-8_EP_150mil DC-DC Converters; Weblink (none) -> https://lcsc.com/product-detail/DC-DC-Converters_XLSEMI-XL7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
Changed lines of the file:
@@
 P 5250 3300
 AR Path="/608DBC83/60A48C4E" Ref="U?"  Part="1"
-AR Path="/608DBC83/60A447A8/60A48C4E" Ref="U8"  Part="1"
-F 0 "U8" H 5281 3665 50  0000 C CNN
+AR Path="/608DBC83/60A447A8/60A48C4E" Ref="U7"  Part="1"
+F 0 "U7" H 5281 3665 50  0000 C CNN
 F 1 "XL7005A" H 5281 3574 50  0000 C CNN
 F 2 "htl_smd:SOIC-8-1EP_3.9x4.9mm_P1.27mm_EP2.514x3.2mm_ThermalVias" H 5300 2150 50  0001 C CNN
@@
 F 6 "0.204" H 5250 3300 50  0001 C CNN "PriceEUR"
 F 7 "100" H 5250 3300 50  0001 C CNN "PriceForQty"
+F 8 "XL7005A" H 5250 3300 50  0001 C CNN "ManPartNr"
+F 9 "XLSEMI" H 5250 3300 50  0001 C CNN "Manufacturer"
+F 10 "80V 400mA SOP-8_EP_150mil DC-DC Converters" H 5250 3300 50  0001 C CNN "Notes"
+F 11 "https://lcsc.com/product-detail/DC-DC-Converters_XLSEMI-XL7005A_C50848.html" H 5250 3300 50  0001 C CNN "Weblink"
 	1    5250 3300
 	1    0    0    -1
@@
 P 6500 3400
 AR Path="/608DBC83/60A48C65" Ref="R?"  Part="1"
-AR Path="/608DBC83/60A447A8/60A48C65" Ref="R33"  Part="1"
-F 0 "R33" H 6570 3446 50  0000 L CNN
+AR Path="/608DBC83/60A447A8/60A48C65" Ref="R37"  Part="1"
+F 0 "R37" H 6570 3446 50  0000 L CNN
 F 1 "10k" H 6570 3355 50  0000 L CNN
 F 2 "Resistor_SMD:R_1206_3216Metric" V 6430 3400 50  0001 C CNN
 F 3 "~" H 6500 3400 50  0001 C CNN
+F 4 "0.01" H 6500 3400 50  0001 C CNN "PriceEUR"
 	1    6500 3400
 	1    0    0    -1
@@
 P 6500 4000
 AR Path="/608DBC83/60A48C6B" Ref="R?"  Part="1"
-AR Path="/608DBC83/60A447A8/60A48C6B" Ref="R34"  Part="1"
-F 0 "R34" H 6570 4046 50  0000 L CNN
+AR Path="/608DBC83/60A447A8/60A48C6B" Ref="R38"  Part="1"
+F 0 "R38" H 6570 4046 50  0000 L CNN
 F 1 "3k3" H 6570 3955 50  0000 L CNN
 F 2 "Resistor_SMD:R_1206_3216Metric" V 6430 4000 50  0001 C CNN
 F 3 "~" H 6500 4000 50  0001 C CNN
+F 4 "0.01" H 6500 4000 50  0001 C CNN "PriceEUR"
 	1    6500 4000
 	1    0    0    -1
@@
 P 4700 4000
 AR Path="/608DBC83/60A48CF0" Ref="R?"  Part="1"
-AR Path="/608DBC83/60A447A8/60A48CF0" Ref="R32"  Part="1"
-F 0 "R32" H 4770 4046 50  0000 L CNN
-F 1 "0R" H 4770 3955 50  0000 L CNN
+AR Path="/608DBC83/60A447A8/60A48CF0" Ref="R36"  Part="1"
+F 0 "R36" H 4770 4046 50  0000 L CNN
+F 1 "100R" H 4770 3955 50  0000 L CNN
 F 2 "Resistor_SMD:R_1206_3216Metric" V 4630 4000 50  0001 C CNN
 F 3 "~" H 4700 4000 50  0001 C CNN
+F 4 "0.01" H 4700 4000 50  0001 C CNN "PriceEUR"
 	1    4700 4000
 	1    0    0    -1
@@
 P 8050 3550
 AR Path="/608DBC83/60A48CF8" Ref="R?"  Part="1"
-AR Path="/608DBC83/60A447A8/60A48CF8" Ref="R35"  Part="1"
-F 0 "R35" H 8120 3596 50  0000 L CNN
+AR Path="/608DBC83/60A447A8/60A48CF8" Ref="R39"  Part="1"
+F 0 "R39" H 8120 3596 50  0000 L CNN
 F 1 "3k3" H 8120 3505 50  0000 L CNN
 F 2 "Resistor_SMD:R_1206_3216Metric" V 7980 3550 50  0001 C CNN
 F 3 "~" H 8050 3550 50  0001 C CNN
+F 4 "0.01" H 8050 3550 50  0001 C CNN "PriceEUR"
 	1    8050 3550
 	1    0    0    -1
@@
 F 5 "C965825" H 8050 4050 50  0001 C CNN "DistOrderNr"
 F 6 "https://lcsc.com/product-detail/Pre-ordered-Products_XINGLIGHT-XL-3216UGC_C965825.html" H 8050 4050 50  0001 C CNN "Weblink"
+F 7 "0.0067" H 8050 4050 50  0001 C CNN "PriceEUR"
+F 8 "50" H 8050 4050 50  0001 C CNN "PriceForQty"
 	1    8050 4050
 	0    -1   -1   0

Commit message: BOM Fertig, 3D auch fast fertig. Ein paar Footrpints fehlen noch.
Parts:
- removed C19: DNP, Capacitor_SMD:CP_Elec_8x10, symbol Device:CP
- added C30: 100u/25V, Capacitor_SMD:CP_Elec_6.3x5.9, symbol Device:CP
- C32: renamed from C21; footprint TODO -> Capacitor_SMD:CP_Elec_6.3x5.9; DistOrderNr C454667 -> C320569; ManPartNr EEHZA1E101XV -> SVZ1EM101E06E00RAXXX; Manufacturer Panasonic -> AISHI; Notes 100uF ±20% 25V 7.7mm 8mm 2A @ 100kHz 30mΩ @ 100kHz 10000hrs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 -> 100uF ±20% 25V 6.3mm 6mm 2000hrs @ 105℃ -55℃~+105℃ SMD,6.3x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; PriceEUR 0.4258 -> 0.1485; PriceForQty 100 -> 30
- L2: footprint Inductor_SMD:L_7.3x7.3_H4.5_TODO -> Inductor_SMD:L_7.3x7.3_H4.5
- R48: renamed from R36; DistOrderNr (none) -> C113307; Distributor (none) -> LCSC; ManPartNr (none) -> RC1206JR-07100RL; Manufacturer (none) -> YAGEO; Notes (none) -> 100Ω ±5% 0.25W ±100ppm/℃ 1206 Chip Resistor; PriceEUR 0.01 -> 0.0037; PriceForQty (none) -> 500
- R49: renamed from R37; DistOrderNr (none) -> C118075; Distributor (none) -> LCSC
- R50: renamed from R38; DistOrderNr (none) -> C229599; Distributor (none) -> LCSC
- R51: renamed from R39; DistOrderNr (none) -> C229599; Distributor (none) -> LCSC
- renumbered C18 to C29, C20 to C31, D8 to D12, D9 to D13, U7 to U9
Changed lines of the file:
@@
 $Descr A4 11693 8268
 encoding utf-8
-Sheet 7 8
+Sheet 8 10
 Title ""
 Date ""
@@
 P 5250 3300
 AR Path="/608DBC83/60A48C4E" Ref="U?"  Part="1"
-AR Path="/608DBC83/60A447A8/60A48C4E" Ref="U7"  Part="1"
-F 0 "U7" H 5281 3665 50  0000 C CNN
+AR Path="/608DBC83/60A447A8/60A48C4E" Ref="U9"  Part="1"
+F 0 "U9" H 5281 3665 50  0000 C CNN
 F 1 "XL7005A" H 5281 3574 50  0000 C CNN
 F 2 "htl_smd:SOIC-8-1EP_3.9x4.9mm_P1.27mm_EP2.514x3.2mm_ThermalVias" H 5300 2150 50  0001 C CNN
@@
 F 0 "L2" H 6150 3415 50  0000 C CNN
 F 1 "47u/1A" H 6150 3324 50  0000 C CNN
-F 2 "Inductor_SMD:L_7.3x7.3_H4.5_TODO" H 6150 3200 50  0001 C CNN
+F 2 "Inductor_SMD:L_7.3x7.3_H4.5" H 6150 3200 50  0001 C CNN
 F 3 "~" H 6150 3200 50  0001 C CNN
 F 4 "LCSC" H 6150 3200 50  0001 C CNN "Distributor"
@@
 P 5800 3900
 AR Path="/608DBC83/60A48C5F" Ref="D?"  Part="1"
-AR Path="/608DBC83/60A447A8/60A48C5F" Ref="D8"  Part="1"
-F 0 "D8" V 5754 3979 50  0000 L CNN
+AR Path="/608DBC83/60A447A8/60A48C5F" Ref="D12"  Part="1"
+F 0 "D12" V 5754 3979 50  0000 L CNN
 F 1 "SS210" V 5845 3979 50  0000 L CNN
 F 2 "Diode_SMD:D_SMA" H 5800 3900 50  0001 C CNN
@@
 P 6500 3400
 AR Path="/608DBC83/60A48C65" Ref="R?"  Part="1"
-AR Path="/608DBC83/60A447A8/60A48C65" Ref="R37"  Part="1"
-F 0 "R37" H 6570 3446 50  0000 L CNN
+AR Path="/608DBC83/60A447A8/60A48C65" Ref="R49"  Part="1"
+F 0 "R49" H 6570 3446 50  0000 L CNN
 F 1 "10k" H 6570 3355 50  0000 L CNN
 F 2 "Resistor_SMD:R_1206_3216Metric" V 6430 3400 50  0001 C CNN
 F 3 "~" H 6500 3400 50  0001 C CNN
 F 4 "0.01" H 6500 3400 50  0001 C CNN "PriceEUR"
+F 5 "C118075" H 6500 3400 50  0001 C CNN "DistOrderNr"
+F 6 "LCSC" H 6500 3400 50  0001 C CNN "Distributor"
 	1    6500 3400
 	1    0    0    -1
@@
 P 6500 4000
 AR Path="/608DBC83/60A48C6B" Ref="R?"  Part="1"
-AR Path="/608DBC83/60A447A8/60A48C6B" Ref="R38"  Part="1"
-F 0 "R38" H 6570 4046 50  0000 L CNN
+AR Path="/608DBC83/60A447A8/60A48C6B" Ref="R50"  Part="1"
+F 0 "R50" H 6570 4046 50  0000 L CNN
 F 1 "3k3" H 6570 3955 50  0000 L CNN
 F 2 "Resistor_SMD:R_1206_3216Metric" V 6430 4000 50  0001 C CNN
 F 3 "~" H 6500 4000 50  0001 C CNN
 F 4 "0.01" H 6500 4000 50  0001 C CNN "PriceEUR"
+F 5 "C229599" H 6500 4000 50  0001 C CNN "DistOrderNr"
+F 6 "LCSC" H 6500 4000 50  0001 C CNN "Distributor"
 	1    6500 4000
 	1    0    0    -1
@@
 P 6850 3400
 AR Path="/608DBC83/60A48C7C" Ref="C?"  Part="1"
-AR Path="/608DBC83/60A447A8/60A48C7C" Ref="C20"  Part="1"
-F 0 "C20" H 6965 3446 50  0000 L CNN
+AR Path="/608DBC83/60A447A8/60A48C7C" Ref="C31"  Part="1"
+F 0 "C31" H 6965 3446 50  0000 L CNN
 F 1 "33n" H 6965 3355 50  0000 L CNN
 F 2 "Capacitor_SMD:C_1206_3216Metric" H 6888 3250 50  0001 C CNN
@@
 $Comp
 L Device:CP C?
-U 1 1 60A48C8A
-P 4100 3750
-AR Path="/608DBC83/60A48C8A" Ref="C?"  Part="1"
-AR Path="/608DBC83/60A447A8/60A48C8A" Ref="C19"  Part="1"
-F 0 "C19" H 4218 3796 50  0000 L CNN
-F 1 "DNP" H 4218 3705 50  0000 L CNN
-F 2 "Capacitor_SMD:CP_Elec_8x10" H 4138 3600 50  0001 C CNN
-F 3 "~" H 4100 3750 50  0001 C CNN
-F 4 "100uF ±20% 63V 8mm 10mm 902mA @ 100kHz 10000hrs @ 105℃ -55℃~+105℃ SMD,8x10mm Aluminum Electrolytic Capacitors" H 4100 3750 50  0001 C CNN "Notes"
-F 5 "dnf" H 4100 3750 50  0001 C CNN "fit_field"
-F 6 "C487384" H 4100 3750 50  0001 C CNN "DistOrderNr"
-F 7 "LCSC" H 4100 3750 50  0001 C CNN "Distributor"
-F 8 "VKMD1001J101MV" H 4100 3750 50  0001 C CNN "ManPartNr"
-F 9 "Ymin" H 4100 3750 50  0001 C CNN "Manufacturer"
-F 10 "0.0698" H 4100 3750 50  0001 C CNN "PriceEUR"
-F 11 "150" H 4100 3750 50  0001 C CNN "PriceForQty"
-	1    4100 3750
-	1    0    0    -1
-$EndComp
-$Comp
-L Device:CP C?
 U 1 1 60A48C90
 P 7200 3950
 AR Path="/608DBC83/60A48C90" Ref="C?"  Part="1"
-AR Path="/608DBC83/60A447A8/60A48C90" Ref="C21"  Part="1"
-F 0 "C21" H 7318 3996 50  0000 L CNN
+AR Path="/608DBC83/60A447A8/60A48C90" Ref="C32"  Part="1"
+F 0 "C32" H 7318 3996 50  0000 L CNN
 F 1 "100u/25V" H 7318 3905 50  0000 L CNN
-F 2 "TODO" H 7238 3800 50  0001 C CNN
+F 2 "Capacitor_SMD:CP_Elec_6.3x5.9" H 7238 3800 50  0001 C CNN
 F 3 "~" H 7200 3950 50  0001 C CNN
-F 4 "C454667" H 7200 3950 50  0001 C CNN "DistOrderNr"
+F 4 "C320569" H 7200 3950 50  0001 C CNN "DistOrderNr"
 F 5 "LCSC" H 7200 3950 50  0001 C CNN "Distributor"
-F 6 "EEHZA1E101XV" H 7200 3950 50  0001 C CNN "ManPartNr"
-F 7 "Panasonic" H 7200 3950 50  0001 C CNN "Manufacturer"
-F 8 "100uF ±20% 25V 7.7mm 8mm 2A @ 100kHz 30mΩ @ 100kHz 10000hrs @ 105℃ -55℃~+105℃ SMD,7.7x8mm Solid Polymer Electrolytic Capacitor" H 7200 3950 50  0001 C CNN "Notes"
-F 9 "0.4258" H 7200 3950 50  0001 C CNN "PriceEUR"
-F 10 "100" H 7200 3950 50  0001 C CNN "PriceForQty"
+F 6 "SVZ1EM101E06E00RAXXX" H 7200 3950 50  0001 C CNN "ManPartNr"
+F 7 "AISHI" H 7200 3950 50  0001 C CNN "Manufacturer"
+F 8 "100uF ±20% 25V 6.3mm 6mm 2000hrs @ 105℃ -55℃~+105℃ SMD,6.3x6mm Solid Polymer Electrolytic Capacitor" H 7200 3950 50  0001 C CNN "Notes"
+F 9 "0.1485" H 7200 3950 50  0001 C CNN "PriceEUR"
+F 10 "30" H 7200 3950 50  0001 C CNN "PriceForQty"
 	1    7200 3950
 	1    0    0    -1
@@
 P 3700 3750
 AR Path="/608DBC83/60A48C96" Ref="C?"  Part="1"
-AR Path="/608DBC83/60A447A8/60A48C96" Ref="C18"  Part="1"
-F 0 "C18" H 3815 3796 50  0000 L CNN
+AR Path="/608DBC83/60A447A8/60A48C96" Ref="C29"  Part="1"
+F 0 "C29" H 3815 3796 50  0000 L CNN
 F 1 "100n/100V" H 3815 3705 50  0000 L CNN
 F 2 "Capacitor_SMD:C_1206_3216Metric" H 3738 3600 50  0001 C CNN
@@
 $EndComp
 Wire Wire Line
-	4850 3200 4100 3200
-Wire Wire Line
 	3700 3600 3700 3200
 Connection ~ 3700 3200
-Wire Wire Line
-	4100 3600 4100 3200
-Connection ~ 4100 3200
-Wire Wire Line
-	4100 3200 3700 3200
 Wire Wire Line
 	4100 4350 4100 3900
@@
 P 8050 3200
 AR Path="/608DBC83/60A48CE8" Ref="#FLG?"  Part="1"
-AR Path="/608DBC83/60A447A8/60A48CE8" Ref="#FLG02"  Part="1"
-F 0 "#FLG02" H 8050 3275 50  0001 C CNN
+AR Path="/608DBC83/60A447A8/60A48CE8" Ref="#FLG04"  Part="1"
+F 0 "#FLG04" H 8050 3275 50  0001 C CNN
 F 1 "PWR_FLAG" H 8050 3373 50  0000 C CNN
 F 2 "" H 8050 3200 50  0001 C CNN
@@
 P 4700 4000
 AR Path="/608DBC83/60A48CF0" Ref="R?"  Part="1"
-AR Path="/608DBC83/60A447A8/60A48CF0" Ref="R36"  Part="1"
-F 0 "R36" H 4770 4046 50  0000 L CNN
+AR Path="/608DBC83/60A447A8/60A48CF0" Ref="R48"  Part="1"
+F 0 "R48" H 4770 4046 50  0000 L CNN
 F 1 "100R" H 4770 3955 50  0000 L CNN
 F 2 "Resistor_SMD:R_1206_3216Metric" V 4630 4000 50  0001 C CNN
 F 3 "~" H 4700 4000 50  0001 C CNN
-F 4 "0.01" H 4700 4000 50  0001 C CNN "PriceEUR"
+F 4 "0.0037" H 4700 4000 50  0001 C CNN "PriceEUR"
+F 5 "C113307" H 4700 4000 50  0001 C CNN "DistOrderNr"
+F 6 "LCSC" H 4700 4000 50  0001 C CNN "Distributor"
+F 7 "RC1206JR-07100RL" H 4700 4000 50  0001 C CNN "ManPartNr"
+F 8 "YAGEO" H 4700 4000 50  0001 C CNN "Manufacturer"
+F 9 "100Ω ±5% 0.25W ±100ppm/℃ 1206 Chip Resistor" H 4700 4000 50  0001 C CNN "Notes"
+F 10 "500" H 4700 4000 50  0001 C CNN "PriceForQty"
 	1    4700 4000
 	1    0    0    -1
@@
 P 8050 3550
 AR Path="/608DBC83/60A48CF8" Ref="R?"  Part="1"
-AR Path="/608DBC83/60A447A8/60A48CF8" Ref="R39"  Part="1"
-F 0 "R39" H 8120 3596 50  0000 L CNN
+AR Path="/608DBC83/60A447A8/60A48CF8" Ref="R51"  Part="1"
+F 0 "R51" H 8120 3596 50  0000 L CNN
 F 1 "3k3" H 8120 3505 50  0000 L CNN
 F 2 "Resistor_SMD:R_1206_3216Metric" V 7980 3550 50  0001 C CNN
 F 3 "~" H 8050 3550 50  0001 C CNN
 F 4 "0.01" H 8050 3550 50  0001 C CNN "PriceEUR"
+F 5 "C229599" H 8050 3550 50  0001 C CNN "DistOrderNr"
+F 6 "LCSC" H 8050 3550 50  0001 C CNN "Distributor"
 	1    8050 3550
 	1    0    0    -1
@@
 P 8050 4050
 AR Path="/608DBC83/60A48D02" Ref="D?"  Part="1"
-AR Path="/608DBC83/60A447A8/60A48D02" Ref="D9"  Part="1"
-F 0 "D9" V 8089 3932 50  0000 R CNN
+AR Path="/608DBC83/60A447A8/60A48D02" Ref="D13"  Part="1"
+F 0 "D13" V 8089 3932 50  0000 R CNN
 F 1 "grün" V 7998 3932 50  0000 R CNN
 F 2 "LED_SMD:LED_1206_3216Metric" H 8050 4050 50  0001 C CNN
@@
 	8050 3900 8050 3700
 $Comp
-L power:GNDPWR #PWR035
+L power:GNDPWR #PWR057
 U 1 1 60A58AB9
 P 3400 4350
-F 0 "#PWR035" H 3400 4150 50  0001 C CNN
+F 0 "#PWR057" H 3400 4150 50  0001 C CNN
 F 1 "GNDPWR" H 3404 4196 50  0000 C CNN
 F 2 "" H 3400 4300 50  0001 C CNN
@@
 	8050 4350 8350 4350
 $Comp
-L power:GNDPWR #PWR036
+L power:GNDPWR #PWR058
 U 1 1 60A5A11F
 P 8350 4350
-F 0 "#PWR036" H 8350 4150 50  0001 C CNN
+F 0 "#PWR058" H 8350 4150 50  0001 C CNN
 F 1 "GNDPWR" H 8354 4196 50  0000 C CNN
 F 2 "" H 8350 4300 50  0001 C CNN
@@
 Text HLabel 8350 3200 2    50   Output ~ 0
 5V
+Wire Wire Line
+	4100 3200 3700 3200
+Wire Wire Line
+	4850 3200 4100 3200
+Connection ~ 4100 3200
+Wire Wire Line
+	4100 3600 4100 3200
+$Comp
+L Device:CP C?
+U 1 1 60B4B9FB
+P 4100 3750
+AR Path="/608DBC83/60B4B9FB" Ref="C?"  Part="1"
+AR Path="/608DBC83/60A447A8/60B4B9FB" Ref="C30"  Part="1"
+F 0 "C30" H 4218 3796 50  0000 L CNN
+F 1 "100u/25V" H 4218 3705 50  0000 L CNN
+F 2 "Capacitor_SMD:CP_Elec_6.3x5.9" H 4138 3600 50  0001 C CNN
+F 3 "~" H 4100 3750 50  0001 C CNN
+F 4 "C320569" H 4100 3750 50  0001 C CNN "DistOrderNr"
+F 5 "LCSC" H 4100 3750 50  0001 C CNN "Distributor"
+F 6 "SVZ1EM101E06E00RAXXX" H 4100 3750 50  0001 C CNN "ManPartNr"
+F 7 "AISHI" H 4100 3750 50  0001 C CNN "Manufacturer"
+F 8 "100uF ±20% 25V 6.3mm 6mm 2000hrs @ 105℃ -55℃~+105℃ SMD,6.3x6mm Solid Polymer Electrolytic Capacitor" H 4100 3750 50  0001 C CNN "Notes"
+F 9 "0.1485" H 4100 3750 50  0001 C CNN "PriceEUR"
+F 10 "30" H 4100 3750 50  0001 C CNN "PriceForQty"
+	1    4100 3750
+	1    0    0    -1
+$EndComp
 $EndSCHEMATC

Commit message: kleinere Updates im Schaltplan
Parts:
- C30, C32: symbol Device:CP -> jbc-miniregler-rescue:CP-Device
Changed lines of the file:
@@
 	4700 3600 4700 3850
 $Comp
-L Device:CP C?
+L jbc-miniregler-rescue:CP-Device C?
 U 1 1 60A48C90
 P 7200 3950
@@
 	4100 3600 4100 3200
 $Comp
-L Device:CP C?
+L jbc-miniregler-rescue:CP-Device C?
 U 1 1 60B4B9FB
 P 4100 3750

Commit message: wip
Connections:
- net labels added: fb, sw, ~en
- wire segments 50 -> 51
Changed lines of the file:
@@
 	3700 4350 3700 3900
 Wire Wire Line
-	5100 4000 5100 4100
-Wire Wire Line
-	5100 4100 5200 4100
-Wire Wire Line
-	5400 4100 5400 4000
-Wire Wire Line
-	5300 4000 5300 4100
-Connection ~ 5300 4100
-Wire Wire Line
-	5300 4100 5400 4100
-Wire Wire Line
-	5200 4000 5200 4100
-Connection ~ 5200 4100
-Wire Wire Line
-	5200 4100 5250 4100
+	5050 4000 5050 4100
+Wire Wire Line
+	5050 4100 5150 4100
+Wire Wire Line
+	5350 4100 5350 4000
+Wire Wire Line
+	5250 4000 5250 4100
+Connection ~ 5250 4100
+Wire Wire Line
+	5250 4100 5350 4100
+Wire Wire Line
+	5150 4000 5150 4100
+Connection ~ 5150 4100
 Wire Wire Line
 	5250 4350 5250 4100
-Connection ~ 5250 4100
-Wire Wire Line
-	5250 4100 5300 4100
 Wire Wire Line
 	5650 3600 6500 3600
@@
 	4100 4350 4700 4350
 Connection ~ 4700 4350
-Wire Wire Line
-	4700 4350 5250 4350
-Connection ~ 5250 4350
-Wire Wire Line
-	5250 4350 5800 4350
 Connection ~ 5800 4350
 Wire Wire Line
@@
 	1    0    0    -1
 $EndComp
+Text Label 5650 3200 0    50   ~ 0
+sw
+Text Label 4700 3600 0    50   ~ 0
+~en
+Text Label 5900 3600 0    50   ~ 0
+fb
+Connection ~ 5250 4350
+Wire Wire Line
+	5250 4350 5800 4350
+Wire Wire Line
+	5150 4100 5250 4100
+Wire Wire Line
+	4700 4350 5250 4350
+Wire Wire Line
+	5350 4100 5450 4100
+Wire Wire Line
+	5450 4100 5450 4000
+Connection ~ 5350 4100
 $EndSCHEMATC

Commit message: WIP Layout, TODO: DRC
Parts:
- D12: footprint Diode_SMD:D_SMA -> htl_smd:D_SMA_wide
- L2: footprint Inductor_SMD:L_7.3x7.3_H4.5 -> htl_smd:L_7.3x7.3_H4.5_C216198
Connections:
- net GNDPWR: no longer D13.1 (K)
- new net GND: D13.1 (K)
Other:
- moved on the sheet: D13
Changed lines of the file:
@@
 F 0 "L2" H 6150 3415 50  0000 C CNN
 F 1 "47u/1A" H 6150 3324 50  0000 C CNN
-F 2 "Inductor_SMD:L_7.3x7.3_H4.5" H 6150 3200 50  0001 C CNN
+F 2 "htl_smd:L_7.3x7.3_H4.5_C216198" H 6150 3200 50  0001 C CNN
 F 3 "~" H 6150 3200 50  0001 C CNN
 F 4 "LCSC" H 6150 3200 50  0001 C CNN "Distributor"
@@
 F 0 "D12" V 5754 3979 50  0000 L CNN
 F 1 "SS210" V 5845 3979 50  0000 L CNN
-F 2 "Diode_SMD:D_SMA" H 5800 3900 50  0001 C CNN
+F 2 "htl_smd:D_SMA_wide" H 5800 3900 50  0001 C CNN
 F 3 "~" H 5800 3900 50  0001 C CNN
 F 4 "C2683692" H 5800 3900 50  0001 C CNN "DistOrderNr"
@@
 L Device:LED D?
 U 1 1 60A48D02
-P 8050 4050
+P 8050 3900
 AR Path="/608DBC83/60A48D02" Ref="D?"  Part="1"
 AR Path="/608DBC83/60A447A8/60A48D02" Ref="D13"  Part="1"
-F 0 "D13" V 8089 3932 50  0000 R CNN
-F 1 "grün" V 7998 3932 50  0000 R CNN
-F 2 "LED_SMD:LED_1206_3216Metric" H 8050 4050 50  0001 C CNN
-F 3 "~" H 8050 4050 50  0001 C CNN
-F 4 "LCSC" H 8050 4050 50  0001 C CNN "Distributor"
-F 5 "C965825" H 8050 4050 50  0001 C CNN "DistOrderNr"
-F 6 "https://lcsc.com/product-detail/Pre-ordered-Products_XINGLIGHT-XL-3216UGC_C965825.html" H 8050 4050 50  0001 C CNN "Weblink"
-F 7 "0.0067" H 8050 4050 50  0001 C CNN "PriceEUR"
-F 8 "50" H 8050 4050 50  0001 C CNN "PriceForQty"
-	1    8050 4050
+F 0 "D13" V 8089 3782 50  0000 R CNN
+F 1 "grün" V 7998 3782 50  0000 R CNN
+F 2 "LED_SMD:LED_1206_3216Metric" H 8050 3900 50  0001 C CNN
+F 3 "~" H 8050 3900 50  0001 C CNN
+F 4 "LCSC" H 8050 3900 50  0001 C CNN "Distributor"
+F 5 "C965825" H 8050 3900 50  0001 C CNN "DistOrderNr"
+F 6 "https://lcsc.com/product-detail/Pre-ordered-Products_XINGLIGHT-XL-3216UGC_C965825.html" H 8050 3900 50  0001 C CNN "Weblink"
+F 7 "0.0067" H 8050 3900 50  0001 C CNN "PriceEUR"
+F 8 "50" H 8050 3900 50  0001 C CNN "PriceForQty"
+	1    8050 3900
 	0    -1   -1   0
 $EndComp
 Wire Wire Line
-	8050 4350 8050 4200
-Wire Wire Line
-	8050 3900 8050 3700
+	8050 3750 8050 3700
 $Comp
 L power:GNDPWR #PWR057
@@
 	6500 4350 7200 4350
 Connection ~ 7200 4350
-Wire Wire Line
-	7200 4350 8050 4350
-Connection ~ 8050 4350
-Wire Wire Line
-	8050 4350 8350 4350
 $Comp
 L power:GNDPWR #PWR058
@@
 	5450 4100 5450 4000
 Connection ~ 5350 4100
+Wire Wire Line
+	7200 4350 8350 4350
+$Comp
+L power:GND #PWR?
+U 1 1 60BD0F64
+P 8050 4050
+F 0 "#PWR?" H 8050 3800 50  0001 C CNN
+F 1 "GND" H 8055 3877 50  0000 C CNN
+F 2 "" H 8050 4050 50  0001 C CNN
+F 3 "" H 8050 4050 50  0001 C CNN
+	1    8050 4050
+	1    0    0    -1
+$EndComp
 $EndSCHEMATC

Commit message: wip, bugfixes für v21.0.1
Parts:
- R48: DistOrderNr C113307 -> C245445; ManPartNr RC1206JR-07100RL -> CR1206F100RP05Z; Manufacturer YAGEO -> Ever Ohms Tech; Notes 100Ω ±5% 0.25W ±100ppm/℃ 1206 Chip Resistor -> 0.25W ±1% ±100ppm/℃ 100Ω 1206; PriceEUR 0.0037 -> 0.0030
- R49: Notes (none) -> 10kΩ ±5% 0.25W ±100ppm/℃ 3216 Chip Resistor
Changed lines of the file:
@@
 Sheet 8 10
 Title "HTL Lötregler Mini"
-Date "2021-06-01"
-Rev "21.0.0"
+Date "2021-09-22"
+Rev "21.0.1-dev"
 Comp "HTL Steyr"
 Comment1 "Prof. Karl Zeilhofer et al."
@@
 F 5 "C118075" H 6500 3400 50  0001 C CNN "DistOrderNr"
 F 6 "LCSC" H 6500 3400 50  0001 C CNN "Distributor"
+F 7 "10kΩ ±5% 0.25W ±100ppm/℃ 3216 Chip Resistor" H 6500 3400 50  0001 C CNN "Notes"
 	1    6500 3400
 	1    0    0    -1
@@
 F 2 "Resistor_SMD:R_1206_3216Metric" V 4630 4000 50  0001 C CNN
 F 3 "~" H 4700 4000 50  0001 C CNN
-F 4 "0.0037" H 4700 4000 50  0001 C CNN "PriceEUR"
-F 5 "C113307" H 4700 4000 50  0001 C CNN "DistOrderNr"
+F 4 "0.0030" H 4700 4000 50  0001 C CNN "PriceEUR"
+F 5 "C245445" H 4700 4000 50  0001 C CNN "DistOrderNr"
 F 6 "LCSC" H 4700 4000 50  0001 C CNN "Distributor"
-F 7 "RC1206JR-07100RL" H 4700 4000 50  0001 C CNN "ManPartNr"
-F 8 "YAGEO" H 4700 4000 50  0001 C CNN "Manufacturer"
-F 9 "100Ω ±5% 0.25W ±100ppm/℃ 1206 Chip Resistor" H 4700 4000 50  0001 C CNN "Notes"
+F 7 "CR1206F100RP05Z" H 4700 4000 50  0001 C CNN "ManPartNr"
+F 8 "Ever Ohms Tech" H 4700 4000 50  0001 C CNN "Manufacturer"
+F 9 "0.25W ±1% ±100ppm/℃ 100Ω 1206" H 4700 4000 50  0001 C CNN "Notes"
 F 10 "500" H 4700 4000 50  0001 C CNN "PriceForQty"
 	1    4700 4000
