File: kicad/dcdc-5v.sch (KiCad schematic (older format))
At the start: 12 parts, among them U9 XL7005A

Commit message: BOM aktualisiert, Zenerdiode: Pinout IPC-konform gestaltet, ...
siehe https://gitlab.com/kicad/libraries/kicad-symbols/-/issues/3157
Parts:
- C29: Index (none) -> 2
- C30, C32: Index (none) -> 34
- C31: Index (none) -> 31
- D12: Index (none) -> 49
- D13: Index (none) -> 47
- L2: Index (none) -> 24
- R48: Index (none) -> 28
- R49: Index (none) -> 15
- R50, R51: Index (none) -> 26
- U9: Index (none) -> 9
Changed lines of the file:
@@
 F 10 "80V 400mA SOP-8_EP_150mil DC-DC Converters" H 5250 3300 50  0001 C CNN "Notes"
 F 11 "https://lcsc.com/product-detail/DC-DC-Converters_XLSEMI-XL7005A_C50848.html" H 5250 3300 50  0001 C CNN "Weblink"
+F 12 "9" H 5250 3300 50  0001 C CNN "Index"
 	1    5250 3300
 	1    0    0    -1
@@
 F 10 "Sunltech Tech" H 6150 3200 50  0001 C CNN "Manufacturer"
 F 11 "47uH ±20% 1A 266mΩ SMD,7.3x7.3x4.5mm" H 6150 3200 50  0001 C CNN "Notes"
+F 12 "24" H 6150 3200 50  0001 C CNN "Index"
 	1    6150 3200
 	1    0    0    -1
@@
 F 10 "200" H 5800 3900 50  0001 C CNN "PriceForQty"
 F 11 "https://lcsc.com/product-detail/Schottky-Barrier-Diodes-SBD_ZHIDE-SS210A-W_C2683692.html" H 5800 3900 50  0001 C CNN "Weblink"
+F 12 "49" H 5800 3900 50  0001 C CNN "Index"
 	1    5800 3900
 	0    1    1    0
@@
 F 6 "LCSC" H 6500 3400 50  0001 C CNN "Distributor"
 F 7 "10kΩ ±5% 0.25W ±100ppm/℃ 3216 Chip Resistor" H 6500 3400 50  0001 C CNN "Notes"
+F 8 "15" H 6500 3400 50  0001 C CNN "Index"
 	1    6500 3400
 	1    0    0    -1
@@
 F 5 "C229599" H 6500 4000 50  0001 C CNN "DistOrderNr"
 F 6 "LCSC" H 6500 4000 50  0001 C CNN "Distributor"
+F 7 "26" H 6500 4000 50  0001 C CNN "Index"
 	1    6500 4000
 	1    0    0    -1
@@
 F 8 "0.0144" H 6850 3400 50  0001 C CNN "PriceEUR"
 F 9 "50" H 6850 3400 50  0001 C CNN "PriceForQty"
+F 10 "31" H 6850 3400 50  0001 C CNN "Index"
 	1    6850 3400
 	1    0    0    -1
@@
 F 9 "0.1485" H 7200 3950 50  0001 C CNN "PriceEUR"
 F 10 "30" H 7200 3950 50  0001 C CNN "PriceForQty"
+F 11 "34" H 7200 3950 50  0001 C CNN "Index"
 	1    7200 3950
 	1    0    0    -1
@@
 F 9 "0.014" H 3700 3750 50  0001 C CNN "PriceEUR"
 F 10 "200" H 3700 3750 50  0001 C CNN "PriceForQty"
+F 11 "2" H 3700 3750 50  0001 C CNN "Index"
 	1    3700 3750
 	-1   0    0    -1
@@
 F 9 "0.25W ±1% ±100ppm/℃ 100Ω 1206" H 4700 4000 50  0001 C CNN "Notes"
 F 10 "500" H 4700 4000 50  0001 C CNN "PriceForQty"
+F 11 "28" H 4700 4000 50  0001 C CNN "Index"
 	1    4700 4000
 	1    0    0    -1
@@
 F 5 "C229599" H 8050 3550 50  0001 C CNN "DistOrderNr"
 F 6 "LCSC" H 8050 3550 50  0001 C CNN "Distributor"
+F 7 "26" H 8050 3550 50  0001 C CNN "Index"
 	1    8050 3550
 	1    0    0    -1
@@
 F 7 "0.0067" H 8050 3900 50  0001 C CNN "PriceEUR"
 F 8 "50" H 8050 3900 50  0001 C CNN "PriceForQty"
+F 9 "47" H 8050 3900 50  0001 C CNN "Index"
 	1    8050 3900
 	0    -1   -1   0
@@
 F 9 "0.1485" H 4100 3750 50  0001 C CNN "PriceEUR"
 F 10 "30" H 4100 3750 50  0001 C CNN "PriceForQty"
+F 11 "34" H 4100 3750 50  0001 C CNN "Index"
 	1    4100 3750
 	1    0    0    -1
