File: kicad/amplifier.sch (KiCad schematic (older format))
At the start: 21 parts, among them U6 GS8332-SR

Commit message: wip, bugfixes für v21.0.1
Parts:
- R21: Notes (none) -> 10kΩ ±5% 0.25W ±100ppm/℃ 3216 Chip Resistor
- R23, R25, R59, R60, R61, R62: DistOrderNr C113307 -> C245445; ManPartNr RC1206JR-07100RL -> CR1206F100RP05Z; Manufacturer YAGEO -> Ever Ohms Tech; Notes 100Ω ±5% 0.25W ±100ppm/℃ 1206 Chip Resistor -> 0.25W ±1% ±100ppm/℃ 100Ω 1206; PriceEUR 0.0037 -> 0.0030
Changed lines of the file:
@@
 Sheet 4 10
 Title "HTL Lötregler Mini"
-Date "2021-06-01"
-Rev "21.0.0"
+Date "2021-09-22"
+Rev "21.0.1-dev"
 Comp "HTL Steyr"
 Comment1 "Prof. Karl Zeilhofer et al."
@@
 F 2 "Resistor_SMD:R_1206_3216Metric" V 7130 3500 50  0001 C CNN
 F 3 "~" H 7200 3500 50  0001 C CNN
-F 4 "0.0037" H 7200 3500 50  0001 C CNN "PriceEUR"
-F 5 "C113307" H 7200 3500 50  0001 C CNN "DistOrderNr"
+F 4 "0.0030" H 7200 3500 50  0001 C CNN "PriceEUR"
+F 5 "C245445" H 7200 3500 50  0001 C CNN "DistOrderNr"
 F 6 "LCSC" H 7200 3500 50  0001 C CNN "Distributor"
-F 7 "RC1206JR-07100RL" H 7200 3500 50  0001 C CNN "ManPartNr"
-F 8 "YAGEO" H 7200 3500 50  0001 C CNN "Manufacturer"
-F 9 "100Ω ±5% 0.25W ±100ppm/℃ 1206 Chip Resistor" H 7200 3500 50  0001 C CNN "Notes"
+F 7 "CR1206F100RP05Z" H 7200 3500 50  0001 C CNN "ManPartNr"
+F 8 "Ever Ohms Tech" H 7200 3500 50  0001 C CNN "Manufacturer"
+F 9 "0.25W ±1% ±100ppm/℃ 100Ω 1206" H 7200 3500 50  0001 C CNN "Notes"
 F 10 "500" H 7200 3500 50  0001 C CNN "PriceForQty"
 	1    7200 3500
@@
 F 5 "C118075" H 3150 2400 50  0001 C CNN "DistOrderNr"
 F 6 "LCSC" H 3150 2400 50  0001 C CNN "Distributor"
+F 7 "10kΩ ±5% 0.25W ±100ppm/℃ 3216 Chip Resistor" H 3150 2400 50  0001 C CNN "Notes"
 	1    3150 2400
 	0    1    1    0
@@
 F 2 "Resistor_SMD:R_1206_3216Metric" V 7080 6050 50  0001 C CNN
 F 3 "~" H 7150 6050 50  0001 C CNN
-F 4 "0.0037" H 7150 6050 50  0001 C CNN "PriceEUR"
-F 5 "C113307" H 7150 6050 50  0001 C CNN "DistOrderNr"
+F 4 "0.0030" H 7150 6050 50  0001 C CNN "PriceEUR"
+F 5 "C245445" H 7150 6050 50  0001 C CNN "DistOrderNr"
 F 6 "LCSC" H 7150 6050 50  0001 C CNN "Distributor"
-F 7 "RC1206JR-07100RL" H 7150 6050 50  0001 C CNN "ManPartNr"
-F 8 "YAGEO" H 7150 6050 50  0001 C CNN "Manufacturer"
-F 9 "100Ω ±5% 0.25W ±100ppm/℃ 1206 Chip Resistor" H 7150 6050 50  0001 C CNN "Notes"
+F 7 "CR1206F100RP05Z" H 7150 6050 50  0001 C CNN "ManPartNr"
+F 8 "Ever Ohms Tech" H 7150 6050 50  0001 C CNN "Manufacturer"
+F 9 "0.25W ±1% ±100ppm/℃ 100Ω 1206" H 7150 6050 50  0001 C CNN "Notes"
 F 10 "500" H 7150 6050 50  0001 C CNN "PriceForQty"
 	1    7150 6050
@@
 F 2 "Resistor_SMD:R_1206_3216Metric" V 4730 2400 50  0001 C CNN
 F 3 "~" H 4800 2400 50  0001 C CNN
-F 4 "0.0037" H 4800 2400 50  0001 C CNN "PriceEUR"
-F 5 "C113307" H 4800 2400 50  0001 C CNN "DistOrderNr"
+F 4 "0.0030" H 4800 2400 50  0001 C CNN "PriceEUR"
+F 5 "C245445" H 4800 2400 50  0001 C CNN "DistOrderNr"
 F 6 "LCSC" H 4800 2400 50  0001 C CNN "Distributor"
-F 7 "RC1206JR-07100RL" H 4800 2400 50  0001 C CNN "ManPartNr"
-F 8 "YAGEO" H 4800 2400 50  0001 C CNN "Manufacturer"
-F 9 "100Ω ±5% 0.25W ±100ppm/℃ 1206 Chip Resistor" H 4800 2400 50  0001 C CNN "Notes"
+F 7 "CR1206F100RP05Z" H 4800 2400 50  0001 C CNN "ManPartNr"
+F 8 "Ever Ohms Tech" H 4800 2400 50  0001 C CNN "Manufacturer"
+F 9 "0.25W ±1% ±100ppm/℃ 100Ω 1206" H 4800 2400 50  0001 C CNN "Notes"
 F 10 "500" H 4800 2400 50  0001 C CNN "PriceForQty"
 	1    4800 2400
@@
 F 2 "Resistor_SMD:R_1206_3216Metric" V 4730 5250 50  0001 C CNN
 F 3 "~" H 4800 5250 50  0001 C CNN
-F 4 "0.0037" H 4800 5250 50  0001 C CNN "PriceEUR"
-F 5 "C113307" H 4800 5250 50  0001 C CNN "DistOrderNr"
+F 4 "0.0030" H 4800 5250 50  0001 C CNN "PriceEUR"
+F 5 "C245445" H 4800 5250 50  0001 C CNN "DistOrderNr"
 F 6 "LCSC" H 4800 5250 50  0001 C CNN "Distributor"
-F 7 "RC1206JR-07100RL" H 4800 5250 50  0001 C CNN "ManPartNr"
-F 8 "YAGEO" H 4800 5250 50  0001 C CNN "Manufacturer"
-F 9 "100Ω ±5% 0.25W ±100ppm/℃ 1206 Chip Resistor" H 4800 5250 50  0001 C CNN "Notes"
+F 7 "CR1206F100RP05Z" H 4800 5250 50  0001 C CNN "ManPartNr"
+F 8 "Ever Ohms Tech" H 4800 5250 50  0001 C CNN "Manufacturer"
+F 9 "0.25W ±1% ±100ppm/℃ 100Ω 1206" H 4800 5250 50  0001 C CNN "Notes"
 F 10 "500" H 4800 5250 50  0001 C CNN "PriceForQty"
 	1    4800 5250
@@
 F 2 "Resistor_SMD:R_1206_3216Metric" V 7780 2700 50  0001 C CNN
 F 3 "~" H 7850 2700 50  0001 C CNN
-F 4 "0.0037" H 7850 2700 50  0001 C CNN "PriceEUR"
-F 5 "C113307" H 7850 2700 50  0001 C CNN "DistOrderNr"
+F 4 "0.0030" H 7850 2700 50  0001 C CNN "PriceEUR"
+F 5 "C245445" H 7850 2700 50  0001 C CNN "DistOrderNr"
 F 6 "LCSC" H 7850 2700 50  0001 C CNN "Distributor"
-F 7 "RC1206JR-07100RL" H 7850 2700 50  0001 C CNN "ManPartNr"
-F 8 "YAGEO" H 7850 2700 50  0001 C CNN "Manufacturer"
-F 9 "100Ω ±5% 0.25W ±100ppm/℃ 1206 Chip Resistor" H 7850 2700 50  0001 C CNN "Notes"
+F 7 "CR1206F100RP05Z" H 7850 2700 50  0001 C CNN "ManPartNr"
+F 8 "Ever Ohms Tech" H 7850 2700 50  0001 C CNN "Manufacturer"
+F 9 "0.25W ±1% ±100ppm/℃ 100Ω 1206" H 7850 2700 50  0001 C CNN "Notes"
 F 10 "500" H 7850 2700 50  0001 C CNN "PriceForQty"
 	1    7850 2700
@@
 F 2 "Resistor_SMD:R_1206_3216Metric" V 7780 5350 50  0001 C CNN
 F 3 "~" H 7850 5350 50  0001 C CNN
-F 4 "0.0037" H 7850 5350 50  0001 C CNN "PriceEUR"
-F 5 "C113307" H 7850 5350 50  0001 C CNN "DistOrderNr"
+F 4 "0.0030" H 7850 5350 50  0001 C CNN "PriceEUR"
+F 5 "C245445" H 7850 5350 50  0001 C CNN "DistOrderNr"
 F 6 "LCSC" H 7850 5350 50  0001 C CNN "Distributor"
-F 7 "RC1206JR-07100RL" H 7850 5350 50  0001 C CNN "ManPartNr"
-F 8 "YAGEO" H 7850 5350 50  0001 C CNN "Manufacturer"
-F 9 "100Ω ±5% 0.25W ±100ppm/℃ 1206 Chip Resistor" H 7850 5350 50  0001 C CNN "Notes"
+F 7 "CR1206F100RP05Z" H 7850 5350 50  0001 C CNN "ManPartNr"
+F 8 "Ever Ohms Tech" H 7850 5350 50  0001 C CNN "Manufacturer"
+F 9 "0.25W ±1% ±100ppm/℃ 100Ω 1206" H 7850 5350 50  0001 C CNN "Notes"
 F 10 "500" H 7850 5350 50  0001 C CNN "PriceForQty"
 	1    7850 5350

Commit message: BOM aktualisiert, Zenerdiode: Pinout IPC-konform gestaltet, ...
siehe https://gitlab.com/kicad/libraries/kicad-symbols/-/issues/3157
Parts:
- C17, C19: Index (none) -> 40
- C18, C40, C41: Index (none) -> 44
- D5, D6: Index (none) -> 22
- JP8, JP9: DistOrderNr (none) -> NAP4; Distributor (none) -> NAP; Index (none) -> 54
- R19: Index (none) -> 29
- R20: Index (none) -> 12
- R21: Index (none) -> 15
- R22, R24: DistOrderNr (none) -> R3216-22k; Distributor LCSC -> AufLager; Index (none) -> 57
- R23, R25, R59, R60, R61, R62: Index (none) -> 28
- U6: Index (none) -> 19
Changed lines of the file:
@@
 F 10 "500" H 6700 2100 50  0001 C CNN "PriceForQty"
 F 11 "" H 6700 2100 50  0001 C CNN "Weblink"
+F 12 "40" H 6700 2100 50  0001 C CNN "Index"
+F 13 "" H 6700 2100 50  0001 C CNN "NotesAlt"
 	1    6700 2100
 	0    1    1    0
@@
 F 10 "500" H 3550 2700 50  0001 C CNN "PriceForQty"
 F 11 "https://lcsc.com/product-detail/Switching-Diode_BAV99-chip0-23_C181111.html" H 3550 2700 50  0001 C CNN "Weblink"
+F 12 "22" H 3550 2700 50  0001 C CNN "Index"
 	2    3550 2700
 	0    -1   -1   0
@@
 F 10 "500" H 3750 2700 50  0001 C CNN "PriceForQty"
 F 11 "https://lcsc.com/product-detail/Switching-Diode_BAV99-chip0-23_C181111.html" H 3750 2700 50  0001 C CNN "Weblink"
+F 12 "22" H 3750 2700 50  0001 C CNN "Index"
 	1    3750 2700
 	0    1    1    0
@@
 F 3 "~" H 7200 3050 50  0001 C CNN
 F 4 "0.01" H 7200 3050 50  0001 C CNN "PriceEUR"
-F 5 "LCSC" H 7200 3050 50  0001 C CNN "Distributor"
+F 5 "AufLager" H 7200 3050 50  0001 C CNN "Distributor"
+F 6 "R3216-22k" H 7200 3050 50  0001 C CNN "DistOrderNr"
+F 7 "57" H 7200 3050 50  0001 C CNN "Index"
 	1    7200 3050
 	1    0    0    -1
@@
 F 9 "0.25W ±1% ±100ppm/℃ 100Ω 1206" H 7200 3500 50  0001 C CNN "Notes"
 F 10 "500" H 7200 3500 50  0001 C CNN "PriceForQty"
+F 11 "28" H 7200 3500 50  0001 C CNN "Index"
 	1    7200 3500
 	1    0    0    -1
@@
 F 6 "LCSC" H 3150 2400 50  0001 C CNN "Distributor"
 F 7 "10kΩ ±5% 0.25W ±100ppm/℃ 3216 Chip Resistor" H 3150 2400 50  0001 C CNN "Notes"
+F 8 "15" H 3150 2400 50  0001 C CNN "Index"
 	1    3150 2400
 	0    1    1    0
@@
 F 9 "0.0106" H 4250 2700 50  0001 C CNN "PriceEUR"
 F 10 "500" H 4250 2700 50  0001 C CNN "PriceForQty"
+F 11 "44" H 4250 2700 50  0001 C CNN "Index"
 	1    4250 2700
 	1    0    0    -1
@@
 F 3 "~" H 7150 5600 50  0001 C CNN
 F 4 "0.01" H 7150 5600 50  0001 C CNN "PriceEUR"
-F 5 "LCSC" H 7150 5600 50  0001 C CNN "Distributor"
+F 5 "AufLager" H 7150 5600 50  0001 C CNN "Distributor"
+F 6 "R3216-22k" H 7150 5600 50  0001 C CNN "DistOrderNr"
+F 7 "57" H 7150 5600 50  0001 C CNN "Index"
 	1    7150 5600
 	1    0    0    -1
@@
 F 9 "0.25W ±1% ±100ppm/℃ 100Ω 1206" H 7150 6050 50  0001 C CNN "Notes"
 F 10 "500" H 7150 6050 50  0001 C CNN "PriceForQty"
+F 11 "28" H 7150 6050 50  0001 C CNN "Index"
 	1    7150 6050
 	1    0    0    -1
@@
 F 10 "100" H 6500 5350 50  0001 C CNN "PriceForQty"
 F 11 "https://lcsc.com/product-detail/Precision-OpAmps_Gainsil-GS8332-SR_C157713.html" H 6500 5350 50  0001 C CNN "Weblink"
+F 12 "19" H 6500 5350 50  0001 C CNN "Index"
 	2    6500 5350
 	1    0    0    -1
@@
 F 10 "100" H 6550 2700 50  0001 C CNN "PriceForQty"
 F 11 "https://lcsc.com/product-detail/Precision-OpAmps_Gainsil-GS8332-SR_C157713.html" H 6550 2700 50  0001 C CNN "Weblink"
+F 12 "19" H 6550 2700 50  0001 C CNN "Index"
 	1    6550 2700
 	1    0    0    -1
@@
 F 10 "100" H 6550 2700 50  0001 C CNN "PriceForQty"
 F 11 "https://lcsc.com/product-detail/Precision-OpAmps_Gainsil-GS8332-SR_C157713.html" H 6550 2700 50  0001 C CNN "Weblink"
+F 12 "19" H 6550 2700 50  0001 C CNN "Index"
 	3    6550 2700
 	1    0    0    -1
@@
 F 5 "C269765" H 2150 2000 50  0001 C CNN "DistOrderNr"
 F 6 "LCSC" H 2150 2000 50  0001 C CNN "Distributor"
+F 7 "29" H 2150 2000 50  0001 C CNN "Index"
 	1    2150 2000
 	1    0    0    -1
@@
 F 2 "Jumper:SolderJumper-3_P2.0mm_Open_TrianglePad1.0x1.5mm_NumberLabels" H 5850 2600 50  0001 C CNN
 F 3 "~" H 5850 2600 50  0001 C CNN
+F 4 "NAP4" H 5850 2600 50  0001 C CNN "DistOrderNr"
+F 5 "NAP" H 5850 2600 50  0001 C CNN "Distributor"
+F 6 "54" H 5850 2600 50  0001 C CNN "Index"
 	1    5850 2600
 	0    -1   1    0
@@
 F 2 "Jumper:SolderJumper-3_P2.0mm_Open_TrianglePad1.0x1.5mm_NumberLabels" H 7200 3900 50  0001 C CNN
 F 3 "~" H 7200 3900 50  0001 C CNN
+F 4 "NAP4" H 7200 3900 50  0001 C CNN "DistOrderNr"
+F 5 "NAP" H 7200 3900 50  0001 C CNN "Distributor"
+F 6 "54" H 7200 3900 50  0001 C CNN "Index"
 	1    7200 3900
 	-1   0    0    1
@@
 F 9 "0.25W ±1% ±100ppm/℃ 100Ω 1206" H 4800 2400 50  0001 C CNN "Notes"
 F 10 "500" H 4800 2400 50  0001 C CNN "PriceForQty"
+F 11 "28" H 4800 2400 50  0001 C CNN "Index"
 	1    4800 2400
 	0    -1   -1   0
@@
 F 10 "500" H 4100 5550 50  0001 C CNN "PriceForQty"
 F 11 "" H 4100 5550 50  0001 C CNN "Weblink"
+F 12 "40" H 4100 5550 50  0001 C CNN "Index"
+F 13 "" H 4100 5550 50  0001 C CNN "NotesAlt"
 	1    4100 5550
 	-1   0    0    1
@@
 F 9 "1kΩ ±5% 0.25W ±100ppm/℃ 1206 Chip Resistor" H 2800 5250 50  0001 C CNN "Notes"
 F 10 "50" H 2800 5250 50  0001 C CNN "PriceForQty"
+F 11 "12" H 2800 5250 50  0001 C CNN "Index"
 	1    2800 5250
 	0    -1   -1   0
@@
 F 10 "500" H 3450 5500 50  0001 C CNN "PriceForQty"
 F 11 "https://lcsc.com/product-detail/Switching-Diode_BAV99-chip0-23_C181111.html" H 3450 5500 50  0001 C CNN "Weblink"
+F 12 "22" H 3450 5500 50  0001 C CNN "Index"
 	1    3450 5500
 	0    1    1    0
@@
 F 10 "500" H 3250 5500 50  0001 C CNN "PriceForQty"
 F 11 "https://lcsc.com/product-detail/Switching-Diode_BAV99-chip0-23_C181111.html" H 3250 5500 50  0001 C CNN "Weblink"
+F 12 "22" H 3250 5500 50  0001 C CNN "Index"
 	2    3250 5500
 	0    -1   -1   0
@@
 F 9 "0.25W ±1% ±100ppm/℃ 100Ω 1206" H 4800 5250 50  0001 C CNN "Notes"
 F 10 "500" H 4800 5250 50  0001 C CNN "PriceForQty"
+F 11 "28" H 4800 5250 50  0001 C CNN "Index"
 	1    4800 5250
 	0    -1   -1   0
@@
 F 9 "0.25W ±1% ±100ppm/℃ 100Ω 1206" H 7850 2700 50  0001 C CNN "Notes"
 F 10 "500" H 7850 2700 50  0001 C CNN "PriceForQty"
+F 11 "28" H 7850 2700 50  0001 C CNN "Index"
 	1    7850 2700
 	0    -1   -1   0
@@
 F 9 "0.0106" H 8150 3000 50  0001 C CNN "PriceEUR"
 F 10 "500" H 8150 3000 50  0001 C CNN "PriceForQty"
+F 11 "44" H 8150 3000 50  0001 C CNN "Index"
 	1    8150 3000
 	1    0    0    -1
@@
 F 9 "0.25W ±1% ±100ppm/℃ 100Ω 1206" H 7850 5350 50  0001 C CNN "Notes"
 F 10 "500" H 7850 5350 50  0001 C CNN "PriceForQty"
+F 11 "28" H 7850 5350 50  0001 C CNN "Index"
 	1    7850 5350
 	0    -1   -1   0
@@
 F 9 "0.0106" H 8150 5650 50  0001 C CNN "PriceEUR"
 F 10 "500" H 8150 5650 50  0001 C CNN "PriceForQty"
+F 11 "44" H 8150 5650 50  0001 C CNN "Index"
 	1    8150 5650
 	1    0    0    -1
