File: kicad/batteries.sch (KiCad schematic (older format))
At the start: 11 parts, among them J10 Makita Minus, J11 Bosch Minus, J12 ActivEnergy B2-, J13 ActivEnergy B1-, J6 ActivEnergy B2+, J7 ActivEnergy B1+, J8 Makita Plus, J9 Bosch Plus

Commit message: um Option RS485 erweitert
Other:
- note added: "B2+ und B2- sind die Standardanschlüsse für ein 20V-Pack"
Changed lines of the file:
@@
 Text Notes 4600 1350 0    50   ~ 0
 TODO: Footprint überprüfen\nTODO: Geometrien der Akkus
+Text Notes 7150 1800 0    50   ~ 0
+B2+ und B2- sind die Standardanschlüsse für ein 20V-Pack
 $EndSCHEMATC

Commit message: Layout
Parts:
- removed J11: Bosch Minus, htl_connectors:Faston_Tab_6.3mm_vertical, symbol Connector_Generic:Conn_01x01
- removed J9: Bosch Plus, htl_connectors:Faston_Tab_6.3mm_vertical, symbol Connector_Generic:Conn_01x01
- added J1: Makita Plus, htl_connectors:Faston_Tab_6.3mm_vertical, symbol Connector_Generic:Conn_01x01
- added J2: Makita Minus, htl_connectors:Faston_Tab_6.3mm_vertical, symbol Connector_Generic:Conn_01x01
Connections:
- net Minus: now also J2.1 (Pin_1)
- net Plus: now also J1.1 (Pin_1)
Changed lines of the file:
@@
 $EndComp
 Connection ~ 5200 3700
-Wire Wire Line
-	5200 3700 5200 3900
-$Comp
-L Connector_Generic:Conn_01x01 J?
-U 1 1 60BECE6F
-P 5000 3900
-AR Path="/60BECE6F" Ref="J?"  Part="1"
-AR Path="/60BEB366/60BECE6F" Ref="J9"  Part="1"
-F 0 "J9" H 5080 3850 50  0000 L CNN
-F 1 "Bosch Plus" H 5080 3941 50  0000 L CNN
-F 2 "htl_connectors:Faston_Tab_6.3mm_vertical" H 5000 3900 50  0001 C CNN
-F 3 "~" H 5000 3900 50  0001 C CNN
-F 4 "VT FS-P 6,35" H 5000 3900 50  0001 C CNN "DistOrderNr"
-F 5 "Reichelt" H 5000 3900 50  0001 C CNN "Distributor"
-F 6 "03866.A68" H 5000 3900 50  0001 C CNN "ManPartNr"
-F 7 "Vogt" H 5000 3900 50  0001 C CNN "Manufacturer"
-F 8 "Faston Flachstecker vertikal 6.3mm für Leiterplattenmontage" H 5000 3900 50  0001 C CNN "Notes"
-F 9 "0.042" H 5000 3900 50  0001 C CNN "PriceEUR"
-F 10 "1" H 5000 3900 50  0001 C CNN "PriceForQty"
-	1    5000 3900
-	-1   0    0    1
-$EndComp
-Connection ~ 5200 3900
-Wire Wire Line
-	5200 3900 5200 4350
 $Comp
 L Connector_Generic:Conn_01x01 J?
@@
 Connection ~ 5200 2500
 Wire Wire Line
-	5200 2500 5200 3700
+	5200 2500 5200 3500
 Text HLabel 6050 4350 2    50   Output ~ 0
 Plus
@@
 $EndComp
 Connection ~ 5350 3700
-Wire Wire Line
-	5350 3700 5350 3900
-$Comp
-L Connector_Generic:Conn_01x01 J?
-U 1 1 60BFE07F
-P 5550 3900
-AR Path="/60BFE07F" Ref="J?"  Part="1"
-AR Path="/60BEB366/60BFE07F" Ref="J11"  Part="1"
-F 0 "J11" H 5630 3942 50  0000 L CNN
-F 1 "Bosch Minus" H 5630 3851 50  0000 L CNN
-F 2 "htl_connectors:Faston_Tab_6.3mm_vertical" H 5550 3900 50  0001 C CNN
-F 3 "~" H 5550 3900 50  0001 C CNN
-F 4 "VT FS-P 6,35" H 5550 3900 50  0001 C CNN "DistOrderNr"
-F 5 "Reichelt" H 5550 3900 50  0001 C CNN "Distributor"
-F 6 "03866.A68" H 5550 3900 50  0001 C CNN "ManPartNr"
-F 7 "Vogt" H 5550 3900 50  0001 C CNN "Manufacturer"
-F 8 "Faston Flachstecker vertikal 6.3mm für Leiterplattenmontage" H 5550 3900 50  0001 C CNN "Notes"
-F 9 "0.042" H 5550 3900 50  0001 C CNN "PriceEUR"
-F 10 "1" H 5550 3900 50  0001 C CNN "PriceForQty"
-	1    5550 3900
-	1    0    0    -1
-$EndComp
-Connection ~ 5350 3900
-Wire Wire Line
-	5350 3900 5350 4550
 $Comp
 L Jumper:SolderJumper_2_Open JP1
@@
 	4300 1750 5200 1750
 Wire Wire Line
-	5350 2500 5350 3700
+	5350 2500 5350 3500
 Wire Wire Line
 	6050 2500 5350 2500
@@
 Text Notes 7150 1800 0    50   ~ 0
 B2+ und B2- sind die Standardanschlüsse für ein 20V-Pack
+$Comp
+L Connector_Generic:Conn_01x01 J?
+U 1 1 60A928EC
+P 5000 3500
+AR Path="/60A928EC" Ref="J?"  Part="1"
+AR Path="/60BEB366/60A928EC" Ref="J1"  Part="1"
+F 0 "J1" H 5080 3450 50  0000 L CNN
+F 1 "Makita Plus" H 5080 3541 50  0000 L CNN
+F 2 "htl_connectors:Faston_Tab_6.3mm_vertical" H 5000 3500 50  0001 C CNN
+F 3 "~" H 5000 3500 50  0001 C CNN
+F 4 "VT FS-P 6,35" H 5000 3500 50  0001 C CNN "DistOrderNr"
+F 5 "Reichelt" H 5000 3500 50  0001 C CNN "Distributor"
+F 6 "03866.A68" H 5000 3500 50  0001 C CNN "ManPartNr"
+F 7 "Vogt" H 5000 3500 50  0001 C CNN "Manufacturer"
+F 8 "Faston Flachstecker vertikal 6.3mm für Leiterplattenmontage" H 5000 3500 50  0001 C CNN "Notes"
+F 9 "0.042" H 5000 3500 50  0001 C CNN "PriceEUR"
+F 10 "1" H 5000 3500 50  0001 C CNN "PriceForQty"
+	1    5000 3500
+	-1   0    0    1
+$EndComp
+Connection ~ 5200 3500
+Wire Wire Line
+	5200 3500 5200 3700
+$Comp
+L Connector_Generic:Conn_01x01 J?
+U 1 1 60A92BD7
+P 5550 3500
+AR Path="/60A92BD7" Ref="J?"  Part="1"
+AR Path="/60BEB366/60A92BD7" Ref="J2"  Part="1"
+F 0 "J2" H 5630 3542 50  0000 L CNN
+F 1 "Makita Minus" H 5630 3451 50  0000 L CNN
+F 2 "htl_connectors:Faston_Tab_6.3mm_vertical" H 5550 3500 50  0001 C CNN
+F 3 "~" H 5550 3500 50  0001 C CNN
+F 4 "VT FS-P 6,35" H 5550 3500 50  0001 C CNN "DistOrderNr"
+F 5 "Reichelt" H 5550 3500 50  0001 C CNN "Distributor"
+F 6 "03866.A68" H 5550 3500 50  0001 C CNN "ManPartNr"
+F 7 "Vogt" H 5550 3500 50  0001 C CNN "Manufacturer"
+F 8 "Faston Flachstecker vertikal 6.3mm für Leiterplattenmontage" H 5550 3500 50  0001 C CNN "Notes"
+F 9 "0.042" H 5550 3500 50  0001 C CNN "PriceEUR"
+F 10 "1" H 5550 3500 50  0001 C CNN "PriceForQty"
+	1    5550 3500
+	1    0    0    -1
+$EndComp
+Connection ~ 5350 3500
+Wire Wire Line
+	5350 3500 5350 3700
+Wire Wire Line
+	5200 3700 5200 4350
+Wire Wire Line
+	5350 3700 5350 4550
 $EndSCHEMATC

Commit message: WIP Layout, TODO: DRC
Parts:
- JP1, JP2, JP3: footprint Jumper:SolderJumper-2_P1.3mm_Open_RoundedPad1.0x1.5mm -> htl_smd:SolderJumper-2_2.2x8mm_Open
Changed lines of the file:
@@
 F 0 "JP1" H 4700 2705 50  0000 C CNN
 F 1 "20V" H 4700 2614 50  0000 C CNN
-F 2 "Jumper:SolderJumper-2_P1.3mm_Open_RoundedPad1.0x1.5mm" H 4700 2500 50  0001 C CNN
+F 2 "htl_smd:SolderJumper-2_2.2x8mm_Open" H 4700 2500 50  0001 C CNN
 F 3 "~" H 4700 2500 50  0001 C CNN
 F 4 "NAP3" H 4700 2500 50  0001 C CNN "DistOrderNr"
@@
 F 0 "JP3" H 5800 1955 50  0000 C CNN
 F 1 "20V" H 5800 1864 50  0000 C CNN
-F 2 "Jumper:SolderJumper-2_P1.3mm_Open_RoundedPad1.0x1.5mm" H 5800 1750 50  0001 C CNN
+F 2 "htl_smd:SolderJumper-2_2.2x8mm_Open" H 5800 1750 50  0001 C CNN
 F 3 "~" H 5800 1750 50  0001 C CNN
 F 4 "NAP3" H 5800 1750 50  0001 C CNN "DistOrderNr"
@@
 F 0 "JP2" H 5600 2355 50  0000 C CNN
 F 1 "40V" H 5600 2264 50  0000 C CNN
-F 2 "Jumper:SolderJumper-2_P1.3mm_Open_RoundedPad1.0x1.5mm" H 5600 2150 50  0001 C CNN
+F 2 "htl_smd:SolderJumper-2_2.2x8mm_Open" H 5600 2150 50  0001 C CNN
 F 3 "~" H 5600 2150 50  0001 C CNN
 F 4 "NAP3" H 5600 2150 50  0001 C CNN "DistOrderNr"

Commit message: BOM aktualisiert, Zenerdiode: Pinout IPC-konform gestaltet, ...
siehe https://gitlab.com/kicad/libraries/kicad-symbols/-/issues/3157
Parts:
- J1, J10, J12, J13, J2, J6, J7, J8: Index (none) -> 59
- JP1, JP2, JP3: Index (none) -> 53
Changed lines of the file:
@@
 F 9 "0.042" H 4100 1750 50  0001 C CNN "PriceEUR"
 F 10 "1" H 4100 1750 50  0001 C CNN "PriceForQty"
+F 11 "59" H 4100 1750 50  0001 C CNN "Index"
 	1    4100 1750
 	-1   0    0    1
@@
 F 9 "0.042" H 6250 2500 50  0001 C CNN "PriceEUR"
 F 10 "1" H 6250 2500 50  0001 C CNN "PriceForQty"
+F 11 "59" H 6250 2500 50  0001 C CNN "Index"
 	1    6250 2500
 	1    0    0    -1
@@
 F 9 "0.042" H 5000 3700 50  0001 C CNN "PriceEUR"
 F 10 "1" H 5000 3700 50  0001 C CNN "PriceForQty"
+F 11 "59" H 5000 3700 50  0001 C CNN "Index"
 	1    5000 3700
 	-1   0    0    1
@@
 F 9 "0.042" H 4100 2500 50  0001 C CNN "PriceEUR"
 F 10 "1" H 4100 2500 50  0001 C CNN "PriceForQty"
+F 11 "59" H 4100 2500 50  0001 C CNN "Index"
 	1    4100 2500
 	-1   0    0    1
@@
 F 9 "0.042" H 5550 3700 50  0001 C CNN "PriceEUR"
 F 10 "1" H 5550 3700 50  0001 C CNN "PriceForQty"
+F 11 "59" H 5550 3700 50  0001 C CNN "Index"
 	1    5550 3700
 	1    0    0    -1
@@
 F 5 "NAP" H 4700 2500 50  0001 C CNN "Distributor"
 F 6 "0.00" H 4700 2500 50  0001 C CNN "PriceEUR"
+F 7 "53" H 4700 2500 50  0001 C CNN "Index"
 	1    4700 2500
 	1    0    0    -1
@@
 F 9 "0.042" H 6250 1750 50  0001 C CNN "PriceEUR"
 F 10 "1" H 6250 1750 50  0001 C CNN "PriceForQty"
+F 11 "59" H 6250 1750 50  0001 C CNN "Index"
 	1    6250 1750
 	1    0    0    -1
@@
 F 5 "NAP" H 5800 1750 50  0001 C CNN "Distributor"
 F 6 "0.00" H 5800 1750 50  0001 C CNN "PriceEUR"
+F 7 "53" H 5800 1750 50  0001 C CNN "Index"
 	1    5800 1750
 	1    0    0    -1
@@
 F 5 "NAP" H 5600 2150 50  0001 C CNN "Distributor"
 F 6 "0.00" H 5600 2150 50  0001 C CNN "PriceEUR"
+F 7 "53" H 5600 2150 50  0001 C CNN "Index"
 	1    5600 2150
 	1    0    0    -1
@@
 F 9 "0.042" H 5000 3500 50  0001 C CNN "PriceEUR"
 F 10 "1" H 5000 3500 50  0001 C CNN "PriceForQty"
+F 11 "59" H 5000 3500 50  0001 C CNN "Index"
 	1    5000 3500
 	-1   0    0    1
@@
 F 9 "0.042" H 5550 3500 50  0001 C CNN "PriceEUR"
 F 10 "1" H 5550 3500 50  0001 C CNN "PriceForQty"
+F 11 "59" H 5550 3500 50  0001 C CNN "Index"
 	1    5550 3500
 	1    0    0    -1
