File: kicad/controller.sch (KiCad schematic (older format))
At the start: 12 parts, among them U12 TL431, U2 74LVC1G125, U3 NST175

Commit message: Workaround zu Isssue#7, USB Bootproblem
Parts:
- added R66: 3k3, Resistor_SMD:R_1206_3216Metric, symbol Device:R
Connections:
- net Arduino Nano/D10: now also R66.2
- net VUSB: now also R66.1
- no-connect marks 4 -> 3
Changed lines of the file:
@@
 	5450 2900 5350 2900
 Wire Wire Line
-	2000 2400 5450 2400
+	2000 2400 4300 2400
 Text HLabel 1600 4550 0    50   Input ~ 0
 Lötkolbenständer
@@
 Text Notes 3650 5200 0    50   ~ 0
 Kondensator \nwichtig für ESD-Schutz
-Wire Wire Line
-	4500 4050 4600 4050
-NoConn ~ 4500 4050
 Text HLabel 3350 3950 0    50   Output ~ 0
 ComDriverEnable
@@
 	1    0    0    -1
 $EndComp
+Wire Wire Line
+	4300 4050 4300 2850
+Wire Wire Line
+	4300 4050 4600 4050
+Connection ~ 4300 2400
+Wire Wire Line
+	4300 2400 5450 2400
+$Comp
+L Device:R R66
+U 1 1 61598C99
+P 4300 2700
+F 0 "R66" H 4230 2746 50  0000 R CNN
+F 1 "3k3" H 4230 2655 50  0000 R CNN
+F 2 "Resistor_SMD:R_1206_3216Metric" V 4230 2700 50  0001 C CNN
+F 3 "~" H 4300 2700 50  0001 C CNN
+F 4 "0.01" H 4300 2700 50  0001 C CNN "PriceEUR"
+F 5 "C229599" H 4300 2700 50  0001 C CNN "DistOrderNr"
+F 6 "LCSC" H 4300 2700 50  0001 C CNN "Distributor"
+	1    4300 2700
+	1    0    0    -1
+$EndComp
+Wire Wire Line
+	4300 2550 4300 2400
 $EndSCHEMATC

Commit message: BOM aktualisiert, Zenerdiode: Pinout IPC-konform gestaltet, ...
siehe https://gitlab.com/kicad/libraries/kicad-symbols/-/issues/3157
Parts:
- C5, C6: Index (none) -> 40
- D2: Index (none) -> 22
- R6, R7: Index (none) -> 15
- R63, R64: Index (none) -> 12
- R66, R8, R9: Index (none) -> 26
- U12: Index (none) -> 21
- U2: Index (none) -> 5
- U3: Index (none) -> 48; NotesAlt (none) -> NST175-H, MSOP-8, 0.65mm Raster, wird aber nicht verbaut, w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
Changed lines of the file:
@@
 F 5 "C229599" H 7000 3800 50  0001 C CNN "DistOrderNr"
 F 6 "LCSC" H 7000 3800 50  0001 C CNN "Distributor"
+F 7 "26" H 7000 3800 50  0001 C CNN "Index"
 	1    7000 3800
 	1    0    0    -1
@@
 F 5 "C229599" H 7300 3800 50  0001 C CNN "DistOrderNr"
 F 6 "LCSC" H 7300 3800 50  0001 C CNN "Distributor"
+F 7 "26" H 7300 3800 50  0001 C CNN "Index"
 	1    7300 3800
 	1    0    0    -1
@@
 F 8 "10" H 9450 4150 50  0001 C CNN "PriceForQty"
 F 9 "https://lcsc.com/product-detail/Temperature-Sensors_NOVOSENSE-NST175-QSPR_C967852.html" H 9450 4150 50  0001 C CNN "Weblink"
+F 10 "48" H 9450 4150 50  0001 C CNN "Index"
+F 11 "NST175-H, MSOP-8, 0.65mm Raster, wird aber nicht verbaut, weil teuer und nicht nötig" H 9450 4150 50  0001 C CNN "NotesAlt"
 	1    9450 4150
 	1    0    0    -1
@@
 F 10 "500" H 10300 4100 50  0001 C CNN "PriceForQty"
 F 11 "" H 10300 4100 50  0001 C CNN "Weblink"
+F 12 "40" H 10300 4100 50  0001 C CNN "Index"
+F 13 "" H 10300 4100 50  0001 C CNN "NotesAlt"
 	1    10300 4100
 	1    0    0    -1
@@
 F 6 "100" H 2000 2750 50  0001 C CNN "PriceForQty"
 F 7 "LCSC" H 2000 2750 50  0001 C CNN "Distributor"
+F 8 "5" H 2000 2750 50  0001 C CNN "Index"
 	1    2000 2750
 	1    0    0    -1
@@
 F 6 "LCSC" H 1900 4550 50  0001 C CNN "Distributor"
 F 7 "10kΩ ±5% 0.25W ±100ppm/℃ 3216 Chip Resistor" H 1900 4550 50  0001 C CNN "Notes"
+F 8 "15" H 1900 4550 50  0001 C CNN "Index"
 	1    1900 4550
 	0    -1   -1   0
@@
 F 6 "LCSC" H 2350 4300 50  0001 C CNN "Distributor"
 F 7 "10kΩ ±5% 0.25W ±100ppm/℃ 3216 Chip Resistor" H 2350 4300 50  0001 C CNN "Notes"
+F 8 "15" H 2350 4300 50  0001 C CNN "Index"
 	1    2350 4300
 	1    0    0    -1
@@
 F 10 "500" H 2350 5100 50  0001 C CNN "PriceForQty"
 F 11 "https://lcsc.com/product-detail/Switching-Diode_BAV99-chip0-23_C181111.html" H 2350 5100 50  0001 C CNN "Weblink"
+F 12 "22" H 2350 5100 50  0001 C CNN "Index"
 	1    2350 5100
 	0    1    1    0
@@
 F 10 "500" H 2800 5100 50  0001 C CNN "PriceForQty"
 F 11 "https://lcsc.com/product-detail/Switching-Diode_BAV99-chip0-23_C181111.html" H 2800 5100 50  0001 C CNN "Weblink"
+F 12 "22" H 2800 5100 50  0001 C CNN "Index"
 	2    2800 5100
 	0    -1   -1   0
@@
 F 10 "500" H 3300 5100 50  0001 C CNN "PriceForQty"
 F 11 "" H 3300 5100 50  0001 C CNN "Weblink"
+F 12 "40" H 3300 5100 50  0001 C CNN "Index"
+F 13 "" H 3300 5100 50  0001 C CNN "NotesAlt"
 	1    3300 5100
 	1    0    0    -1
@@
 F 9 "1kΩ ±5% 0.25W ±100ppm/℃ 1206 Chip Resistor" H 6350 2650 50  0001 C CNN "Notes"
 F 10 "50" H 6350 2650 50  0001 C CNN "PriceForQty"
+F 11 "12" H 6350 2650 50  0001 C CNN "Index"
 	1    6350 2650
 	1    0    0    -1
@@
 F 9 "1kΩ ±5% 0.25W ±100ppm/℃ 1206 Chip Resistor" H 6600 2650 50  0001 C CNN "Notes"
 F 10 "50" H 6600 2650 50  0001 C CNN "PriceForQty"
+F 11 "12" H 6600 2650 50  0001 C CNN "Index"
 	1    6600 2650
 	1    0    0    -1
@@
 F 8 "https://lcsc.com/product-detail/Voltage-References_Guangdong-Hottech-TL431_C181103.html" H 6350 3250 50  0001 C CNN "Weblink"
 F 9 "2.5V, +/-0.5%, +/-50ppm/K, SOT-23, Ref-Kath-Ano" H 6350 3250 50  0001 C CNN "Notes"
+F 10 "21" H 6350 3250 50  0001 C CNN "Index"
 	1    6350 3250
 	1    0    0    -1
@@
 F 5 "C229599" H 4300 2700 50  0001 C CNN "DistOrderNr"
 F 6 "LCSC" H 4300 2700 50  0001 C CNN "Distributor"
+F 7 "26" H 4300 2700 50  0001 C CNN "Index"
 	1    4300 2700
 	1    0    0    -1
