File: kicad/jbc-miniregler.sch (KiCad schematic (older format))
At the start: 26 parts, among them J1 Power IN, J2 COM, J3 Lötkolben, SW1 UP, SW2 DOWN, SW3 ENTER, SW4 BACK, U1 OLED-128x32-Module

Commit message: BOM ist nun fast fertig
Parts:
- FID1, FID2, H1, H2, H3, H4: PriceEUR (none) -> 0.00
- Item1: renamed from Item2; PriceEUR (none) -> 0.1656; PriceForQty (none) -> 100
- Item2: renamed from Item3; value PCB, 2 Layer, 35um Cu, 1.6mm, TODO size -> PCB, 1 Layer, 35um Cu, 1.6mm, ca. 100x110; PriceEUR (none) -> 3.71; PriceForQty (none) -> 100
- J1: footprint TODO -> Connector_Phoenix_MSTB:PhoenixContact_MSTBA_2,5_2-G-5,08_1x02_P5.08mm_Horizontal; Notes (none) -> 2 poles, 5.08mm, 15A 250V AWG14~22 1.5mm² P=5.08mm Spring C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; PriceEUR (none) -> 0.1172; PriceForQty (none) -> 100
- J2, J3: footprint TODO -> Connector_Phoenix_MSTB:PhoenixContact_MSTBA_2,5_3-G-5,08_1x03_P5.08mm_Horizontal; Notes (none) -> 3 poles, 5.08mm, 15A 250V AWG14~22 1.5mm² P=5.08mm Spring C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; PriceEUR (none) -> 0.1347; PriceForQty (none) -> 100
- R1, R2, R3, R4: value 4k7 -> 10k; PriceEUR (none) -> 0.01
- R5: PriceEUR (none) -> 0.01
- SW1, SW2, SW3, SW4: ManPartNr (none) -> TS-1187A-B-A-B; Manufacturer (none) -> XKB Connectivity; Notes (none) -> SPST 50mA @ 12VDC Vertical Round Button 160gf SMD Tactile S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; PriceEUR (none) -> 0.01; PriceForQty (none) -> 500; Weblink (none) -> https://lcsc.com/product-detail/Tactile-Switches_XKB-Connec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
- U1: footprint TODO -> htl_modules:OLED-128x32
Other:
- note added: "TODOs:\n* ERC\n* Footprint Federklemmen\n* Footprint Panasonic ELKOs\n* ATmega328 statt Arduino\n"
Changed lines of the file:
@@
 F 0 "J1" H 1018 2417 50  0000 C CNN
 F 1 "Power IN" H 1018 2326 50  0000 C CNN
-F 2 "TODO" H 1100 2100 50  0001 C CNN
+F 2 "Connector_Phoenix_MSTB:PhoenixContact_MSTBA_2,5_2-G-5,08_1x02_P5.08mm_Horizontal" H 1100 2100 50  0001 C CNN
 F 3 "~" H 1100 2100 50  0001 C CNN
 F 4 "C475144" H 1100 2100 50  0001 C CNN "DistOrderNr"
 F 5 "LCSC" H 1100 2100 50  0001 C CNN "Distributor"
+F 6 "0.1172" H 1100 2100 50  0001 C CNN "PriceEUR"
+F 7 "100" H 1100 2100 50  0001 C CNN "PriceForQty"
+F 8 "2 poles, 5.08mm, 15A 250V AWG14~22 1.5mm² P=5.08mm Spring Clamp System Terminal Block" H 1100 2100 50  0001 C CNN "Notes"
 	1    1100 2100
 	-1   0    0    -1
@@
 F 0 "J3" H 8468 1525 50  0000 C CNN
 F 1 "Lötkolben" H 8468 1616 50  0000 C CNN
-F 2 "TODO" H 8550 1850 50  0001 C CNN
+F 2 "Connector_Phoenix_MSTB:PhoenixContact_MSTBA_2,5_3-G-5,08_1x03_P5.08mm_Horizontal" H 8550 1850 50  0001 C CNN
 F 3 "~" H 8550 1850 50  0001 C CNN
 F 4 "C475145" H 8550 1850 50  0001 C CNN "DistOrderNr"
 F 5 "LCSC" H 8550 1850 50  0001 C CNN "Distributor"
+F 6 "0.1347" H 8550 1850 50  0001 C CNN "PriceEUR"
+F 7 "100" H 8550 1850 50  0001 C CNN "PriceForQty"
+F 8 "3 poles, 5.08mm, 15A 250V AWG14~22 1.5mm² P=5.08mm Spring Clamp System Terminal Block" H 8550 1850 50  0001 C CNN "Notes"
 	1    8550 1850
 	1    0    0    1
@@
 F 0 "J2" H 1018 3967 50  0000 C CNN
 F 1 "COM" H 1018 3876 50  0000 C CNN
-F 2 "TODO" H 1100 3650 50  0001 C CNN
+F 2 "Connector_Phoenix_MSTB:PhoenixContact_MSTBA_2,5_3-G-5,08_1x03_P5.08mm_Horizontal" H 1100 3650 50  0001 C CNN
 F 3 "~" H 1100 3650 50  0001 C CNN
 F 4 "C475145" H 1100 3650 50  0001 C CNN "DistOrderNr"
 F 5 "LCSC" H 1100 3650 50  0001 C CNN "Distributor"
+F 6 "0.1347" H 1100 3650 50  0001 C CNN "PriceEUR"
+F 7 "100" H 1100 3650 50  0001 C CNN "PriceForQty"
+F 8 "3 poles, 5.08mm, 15A 250V AWG14~22 1.5mm² P=5.08mm Spring Clamp System Terminal Block" H 1100 3650 50  0001 C CNN "Notes"
 	1    1100 3650
 	-1   0    0    -1
@@
 F 4 "C318884" H 3250 5900 50  0001 C CNN "DistOrderNr"
 F 5 "LCSC" H 3250 5900 50  0001 C CNN "Distributor"
+F 6 "TS-1187A-B-A-B" H 3250 5900 50  0001 C CNN "ManPartNr"
+F 7 "XKB Connectivity" H 3250 5900 50  0001 C CNN "Manufacturer"
+F 8 " 	SPST 50mA @ 12VDC Vertical Round Button 160gf SMD Tactile Switches " H 3250 5900 50  0001 C CNN "Notes"
+F 9 "0.01" H 3250 5900 50  0001 C CNN "PriceEUR"
+F 10 "500" H 3250 5900 50  0001 C CNN "PriceForQty"
+F 11 "https://lcsc.com/product-detail/Tactile-Switches_XKB-Connectivity-TS-1187A-B-A-B_C318884.html" H 3250 5900 50  0001 C CNN "Weblink"
 	1    3250 5900
 	0    -1   -1   0
@@
 F 4 "C318884" H 4050 5900 50  0001 C CNN "DistOrderNr"
 F 5 "LCSC" H 4050 5900 50  0001 C CNN "Distributor"
+F 6 "TS-1187A-B-A-B" H 4050 5900 50  0001 C CNN "ManPartNr"
+F 7 "XKB Connectivity" H 4050 5900 50  0001 C CNN "Manufacturer"
+F 8 " 	SPST 50mA @ 12VDC Vertical Round Button 160gf SMD Tactile Switches " H 4050 5900 50  0001 C CNN "Notes"
+F 9 "0.01" H 4050 5900 50  0001 C CNN "PriceEUR"
+F 10 "500" H 4050 5900 50  0001 C CNN "PriceForQty"
+F 11 "https://lcsc.com/product-detail/Tactile-Switches_XKB-Connectivity-TS-1187A-B-A-B_C318884.html" H 4050 5900 50  0001 C CNN "Weblink"
 	1    4050 5900
 	0    -1   -1   0
@@
 AR Path="/60AB2E71" Ref="R3"  Part="1"
 F 0 "R3" H 3320 4846 50  0000 L CNN
-F 1 "4k7" H 3320 4755 50  0000 L CNN
+F 1 "10k" H 3320 4755 50  0000 L CNN
 F 2 "Resistor_SMD:R_1206_3216Metric" V 3180 4800 50  0001 C CNN
 F 3 "~" H 3250 4800 50  0001 C CNN
+F 4 "0.01" H 3250 4800 50  0001 C CNN "PriceEUR"
 	1    3250 4800
 	1    0    0    -1
@@
 AR Path="/60AB2E77" Ref="R4"  Part="1"
 F 0 "R4" H 4120 4846 50  0000 L CNN
-F 1 "4k7" H 4120 4755 50  0000 L CNN
+F 1 "10k" H 4120 4755 50  0000 L CNN
 F 2 "Resistor_SMD:R_1206_3216Metric" V 3980 4800 50  0001 C CNN
 F 3 "~" H 4050 4800 50  0001 C CNN
+F 4 "0.01" H 4050 4800 50  0001 C CNN "PriceEUR"
 	1    4050 4800
 	1    0    0    -1
@@
 F 4 "C318884" H 1650 5900 50  0001 C CNN "DistOrderNr"
 F 5 "LCSC" H 1650 5900 50  0001 C CNN "Distributor"
+F 6 "TS-1187A-B-A-B" H 1650 5900 50  0001 C CNN "ManPartNr"
+F 7 "XKB Connectivity" H 1650 5900 50  0001 C CNN "Manufacturer"
+F 8 " 	SPST 50mA @ 12VDC Vertical Round Button 160gf SMD Tactile Switches " H 1650 5900 50  0001 C CNN "Notes"
+F 9 "0.01" H 1650 5900 50  0001 C CNN "PriceEUR"
+F 10 "500" H 1650 5900 50  0001 C CNN "PriceForQty"
+F 11 "https://lcsc.com/product-detail/Tactile-Switches_XKB-Connectivity-TS-1187A-B-A-B_C318884.html" H 1650 5900 50  0001 C CNN "Weblink"
 	1    1650 5900
 	0    -1   -1   0
@@
 F 4 "C318884" H 2500 5900 50  0001 C CNN "DistOrderNr"
 F 5 "LCSC" H 2500 5900 50  0001 C CNN "Distributor"
+F 6 "TS-1187A-B-A-B" H 2500 5900 50  0001 C CNN "ManPartNr"
+F 7 "XKB Connectivity" H 2500 5900 50  0001 C CNN "Manufacturer"
+F 8 " 	SPST 50mA @ 12VDC Vertical Round Button 160gf SMD Tactile Switches " H 2500 5900 50  0001 C CNN "Notes"
+F 9 "0.01" H 2500 5900 50  0001 C CNN "PriceEUR"
+F 10 "500" H 2500 5900 50  0001 C CNN "PriceForQty"
+F 11 "https://lcsc.com/product-detail/Tactile-Switches_XKB-Connectivity-TS-1187A-B-A-B_C318884.html" H 2500 5900 50  0001 C CNN "Weblink"
 	1    2500 5900
 	0    -1   -1   0
@@
 AR Path="/60AC53EC" Ref="R1"  Part="1"
 F 0 "R1" H 1720 4846 50  0000 L CNN
-F 1 "4k7" H 1720 4755 50  0000 L CNN
+F 1 "10k" H 1720 4755 50  0000 L CNN
 F 2 "Resistor_SMD:R_1206_3216Metric" V 1580 4800 50  0001 C CNN
 F 3 "~" H 1650 4800 50  0001 C CNN
+F 4 "0.01" H 1650 4800 50  0001 C CNN "PriceEUR"
 	1    1650 4800
 	1    0    0    -1
@@
 AR Path="/60AC53F2" Ref="R2"  Part="1"
 F 0 "R2" H 2570 4846 50  0000 L CNN
-F 1 "4k7" H 2570 4755 50  0000 L CNN
+F 1 "10k" H 2570 4755 50  0000 L CNN
 F 2 "Resistor_SMD:R_1206_3216Metric" V 2430 4800 50  0001 C CNN
 F 3 "~" H 2500 4800 50  0001 C CNN
+F 4 "0.01" H 2500 4800 50  0001 C CNN "PriceEUR"
 	1    2500 4800
 	1    0    0    -1
@@
 F 2 "Resistor_SMD:R_1206_3216Metric" V 6130 2150 50  0001 C CNN
 F 3 "~" H 6200 2150 50  0001 C CNN
+F 4 "0.01" H 6200 2150 50  0001 C CNN "PriceEUR"
 	1    6200 2150
 	1    0    0    -1
@@
 F 0 "U1" H 7450 4887 60  0000 C CNN
 F 1 "OLED-128x32-Module" H 7450 4781 60  0000 C CNN
-F 2 "TODO" H 6650 4050 60  0001 C CNN
+F 2 "htl_modules:OLED-128x32" H 6650 4050 60  0001 C CNN
 F 3 "" H 6650 4050 60  0001 C CNN
 F 4 "AliExpress, SAMIORE Store" H 7450 4500 50  0001 C CNN "Distributor"
@@
 Standardwerte:\nKondensatoren: 10%, X7R, C3216, 50V\nWiderstände: 1%, 250mW, R3216
 $Comp
-L htl_virtual:Item Item3
+L htl_virtual:Item Item2
 U 1 1 60B4CFB2
 P 9200 6400
-F 0 "Item3" H 9330 6446 50  0000 L CNN
-F 1 "PCB, 2 Layer, 35um Cu, 1.6mm, TODO size" H 9330 6355 50  0000 L CNN
+F 0 "Item2" H 9330 6446 50  0000 L CNN
+F 1 "PCB, 1 Layer, 35um Cu, 1.6mm, ca. 100x110" H 9330 6355 50  0000 L CNN
 F 2 "htl_virtual:Virtual-Item" H 9200 6330 50  0001 C CNN
 F 3 "~" V 9200 6400 50  0001 C CNN
@@
 F 5 "Multi-CB" H 9200 6400 50  0001 C CNN "Distributor"
 F 6 "Multi-CB" H 9200 6400 50  0001 C CNN "Manufacturer"
+F 7 "3.71" H 9200 6400 50  0001 C CNN "PriceEUR"
+F 8 "100" H 9200 6400 50  0001 C CNN "PriceForQty"
 	1    9200 6400
 	1    0    0    -1
 $EndComp
 $Comp
-L htl_virtual:Item Item2
+L htl_virtual:Item Item1
 U 1 1 60B4D7DC
 P 9200 6200
-F 0 "Item2" H 9330 6246 50  0000 L CNN
+F 0 "Item1" H 9330 6246 50  0000 L CNN
 F 1 "Stencil, 120um, 25mm Rand, Edelstahl" H 9330 6155 50  0000 L CNN
 F 2 "htl_virtual:Virtual-Item" H 9200 6130 50  0001 C CNN
@@
 F 5 "Multi-CB" H 9200 6200 50  0001 C CNN "Distributor"
 F 6 "Multi-CB" H 9200 6200 50  0001 C CNN "Manufacturer"
+F 7 "0.1656" H 9200 6200 50  0001 C CNN "PriceEUR"
+F 8 "100" H 9200 6200 50  0001 C CNN "PriceForQty"
 	1    9200 6200
 	1    0    0    -1
@@
 F 7 "NAP" H 9950 5050 50  0001 C CNN "Manufacturer"
 F 8 "Not a Part" H 9950 5050 50  0001 C CNN "Notes"
+F 9 "0.00" H 9950 5050 50  0001 C CNN "PriceEUR"
 	1    9950 5050
 	1    0    0    -1
@@
 F 7 "NAP" H 9950 5250 50  0001 C CNN "Manufacturer"
 F 8 "Not a Part" H 9950 5250 50  0001 C CNN "Notes"
+F 9 "0.00" H 9950 5250 50  0001 C CNN "PriceEUR"
 	1    9950 5250
 	1    0    0    -1
@@
 F 7 "NAP" H 9950 5450 50  0001 C CNN "Manufacturer"
 F 8 "Not a Part" H 9950 5450 50  0001 C CNN "Notes"
+F 9 "0.00" H 9950 5450 50  0001 C CNN "PriceEUR"
 	1    9950 5450
 	1    0    0    -1
@@
 F 7 "NAP" H 9950 5650 50  0001 C CNN "Manufacturer"
 F 8 "Not a Part" H 9950 5650 50  0001 C CNN "Notes"
+F 9 "0.00" H 9950 5650 50  0001 C CNN "PriceEUR"
 	1    9950 5650
 	1    0    0    -1
@@
 F 4 "NAP" H 9950 4650 50  0001 C CNN "DistOrderNr"
 F 5 "Not a Part" H 9950 4650 50  0001 C CNN "Manufacturer"
+F 6 "0.00" H 9950 4650 50  0001 C CNN "PriceEUR"
 	1    9950 4650
 	1    0    0    -1
@@
 F 4 "NAP" H 9950 4450 50  0001 C CNN "DistOrderNr"
 F 5 "Not a Part" H 9950 4450 50  0001 C CNN "Manufacturer"
+F 6 "0.00" H 9950 4450 50  0001 C CNN "PriceEUR"
 	1    9950 4450
 	1    0    0    -1
 $EndComp
+Text Notes 8200 3750 0    150  ~ 0
+TODOs:\n* ERC\n* Footprint Federklemmen\n* Footprint Panasonic ELKOs\n* ATmega328 statt Arduino\n
 $EndSCHEMATC

Commit message: BOM Fertig, 3D auch fast fertig. Ein paar Footrpints fehlen noch.
Parts:
- removed J1: Power IN, Connector_Phoenix_MSTB:PhoenixContact_MSTBA_2,5_2-G-5,08_1x02_P5.08mm_Horizontal, symbol Connector:Screw_Terminal_01x02
- added J1: COM, Connector_Phoenix_MSTB:PhoenixContact_MSTBA_2,5_3-G-5,08_1x03_P5.08mm_Horizontal, symbol Connector:Screw_Terminal_01x03
- FID1, FID2: DistOrderNr NAP -> NAP1; Distributor (none) -> NAP
- H1, H2, H3, H4: DistOrderNr NAP -> NAP2
- Item1: DistOrderNr Custom -> Custom1
- Item2: DistOrderNr Custom -> Custom2
- R1, R2, R3, R4: DistOrderNr (none) -> C118075; Distributor (none) -> LCSC
- R5: DistOrderNr (none) -> C104601; Distributor (none) -> LCSC; ManPartNr (none) -> RTT03101JTP; Manufacturer (none) -> RALEC; Notes (none) -> 1kΩ ±5% 0.25W ±100ppm/℃ 1206 Chip Resistor; PriceEUR 0.01 -> 0.0042; PriceForQty (none) -> 50
- SW1, SW2, SW3, SW4: Notes SPST 50mA @ 12VDC Vertical Round Button 160gf SMD Tactile Switches -> SPST 50mA @ 12VDC Vertical Round Button 160gf SMD Tactile Switches
Connections:
- wire segments 87 -> 94
Other:
- note added: "TODO: Footprint Federklemmen\n"
- note removed: "TODOs:\n* ERC\n* Footprint Federklemmen\n* Footprint Panasonic ELKOs\n* ATmega328 statt Arduino\n"
Changed lines of the file:
@@
 $Descr A4 11693 8268
 encoding utf-8
-Sheet 1 8
+Sheet 1 10
 Title "JBC-Miniregler"
 Date "2021-05-02"
@@
 F15 "SCL" B R 5950 4500 50
 F16 "SDA" B R 5950 4400 50
+F17 "Lötkolbenständer" I L 4550 2800 50
 $EndSheet
 $Sheet
@@
 $EndSheet
 $Comp
-L Connector:Screw_Terminal_01x02 J1
-U 1 1 609B47F3
-P 1100 2100
-F 0 "J1" H 1018 2417 50  0000 C CNN
-F 1 "Power IN" H 1018 2326 50  0000 C CNN
-F 2 "Connector_Phoenix_MSTB:PhoenixContact_MSTBA_2,5_2-G-5,08_1x02_P5.08mm_Horizontal" H 1100 2100 50  0001 C CNN
-F 3 "~" H 1100 2100 50  0001 C CNN
-F 4 "C475144" H 1100 2100 50  0001 C CNN "DistOrderNr"
-F 5 "LCSC" H 1100 2100 50  0001 C CNN "Distributor"
-F 6 "0.1172" H 1100 2100 50  0001 C CNN "PriceEUR"
-F 7 "100" H 1100 2100 50  0001 C CNN "PriceForQty"
-F 8 "2 poles, 5.08mm, 15A 250V AWG14~22 1.5mm² P=5.08mm Spring Clamp System Terminal Block" H 1100 2100 50  0001 C CNN "Notes"
-	1    1100 2100
-	-1   0    0    -1
-$EndComp
-$Comp
 L Connector:Screw_Terminal_01x03 J3
 U 1 1 609B52E2
@@
 $EndComp
 Wire Wire Line
-	1800 2050 1300 2050
-Wire Wire Line
-	1300 2250 1400 2250
-Wire Wire Line
 	7650 1750 8350 1750
 Wire Wire Line
@@
 	1800 3650 1300 3650
 Wire Wire Line
-	1300 3750 1400 3750
-Wire Wire Line
-	1300 2100 1300 2050
-Wire Wire Line
-	1300 2200 1300 2250
+	1300 3750 1500 3750
 $Sheet
 S 1800 3150 1400 700
@@
 F 6 "TS-1187A-B-A-B" H 3250 5900 50  0001 C CNN "ManPartNr"
 F 7 "XKB Connectivity" H 3250 5900 50  0001 C CNN "Manufacturer"
-F 8 " 	SPST 50mA @ 12VDC Vertical Round Button 160gf SMD Tactile Switches " H 3250 5900 50  0001 C CNN "Notes"
+F 8 "SPST 50mA @ 12VDC Vertical Round Button 160gf SMD Tactile Switches" H 3250 5900 50  0001 C CNN "Notes"
 F 9 "0.01" H 3250 5900 50  0001 C CNN "PriceEUR"
 F 10 "500" H 3250 5900 50  0001 C CNN "PriceForQty"
@@
 F 6 "TS-1187A-B-A-B" H 4050 5900 50  0001 C CNN "ManPartNr"
 F 7 "XKB Connectivity" H 4050 5900 50  0001 C CNN "Manufacturer"
-F 8 " 	SPST 50mA @ 12VDC Vertical Round Button 160gf SMD Tactile Switches " H 4050 5900 50  0001 C CNN "Notes"
+F 8 "SPST 50mA @ 12VDC Vertical Round Button 160gf SMD Tactile Switches" H 4050 5900 50  0001 C CNN "Notes"
 F 9 "0.01" H 4050 5900 50  0001 C CNN "PriceEUR"
 F 10 "500" H 4050 5900 50  0001 C CNN "PriceForQty"
@@
 F 3 "~" H 3250 4800 50  0001 C CNN
 F 4 "0.01" H 3250 4800 50  0001 C CNN "PriceEUR"
+F 5 "C118075" H 3250 4800 50  0001 C CNN "DistOrderNr"
+F 6 "LCSC" H 3250 4800 50  0001 C CNN "Distributor"
 	1    3250 4800
 	1    0    0    -1
@@
 F 3 "~" H 4050 4800 50  0001 C CNN
 F 4 "0.01" H 4050 4800 50  0001 C CNN "PriceEUR"
+F 5 "C118075" H 4050 4800 50  0001 C CNN "DistOrderNr"
+F 6 "LCSC" H 4050 4800 50  0001 C CNN "Distributor"
 	1    4050 4800
 	1    0    0    -1
@@
 F 6 "TS-1187A-B-A-B" H 1650 5900 50  0001 C CNN "ManPartNr"
 F 7 "XKB Connectivity" H 1650 5900 50  0001 C CNN "Manufacturer"
-F 8 " 	SPST 50mA @ 12VDC Vertical Round Button 160gf SMD Tactile Switches " H 1650 5900 50  0001 C CNN "Notes"
+F 8 "SPST 50mA @ 12VDC Vertical Round Button 160gf SMD Tactile Switches" H 1650 5900 50  0001 C CNN "Notes"
 F 9 "0.01" H 1650 5900 50  0001 C CNN "PriceEUR"
 F 10 "500" H 1650 5900 50  0001 C CNN "PriceForQty"
@@
 F 6 "TS-1187A-B-A-B" H 2500 5900 50  0001 C CNN "ManPartNr"
 F 7 "XKB Connectivity" H 2500 5900 50  0001 C CNN "Manufacturer"
-F 8 " 	SPST 50mA @ 12VDC Vertical Round Button 160gf SMD Tactile Switches " H 2500 5900 50  0001 C CNN "Notes"
+F 8 "SPST 50mA @ 12VDC Vertical Round Button 160gf SMD Tactile Switches" H 2500 5900 50  0001 C CNN "Notes"
 F 9 "0.01" H 2500 5900 50  0001 C CNN "PriceEUR"
 F 10 "500" H 2500 5900 50  0001 C CNN "PriceForQty"
@@
 F 3 "~" H 1650 4800 50  0001 C CNN
 F 4 "0.01" H 1650 4800 50  0001 C CNN "PriceEUR"
+F 5 "C118075" H 1650 4800 50  0001 C CNN "DistOrderNr"
+F 6 "LCSC" H 1650 4800 50  0001 C CNN "Distributor"
 	1    1650 4800
 	1    0    0    -1
@@
 F 3 "~" H 2500 4800 50  0001 C CNN
 F 4 "0.01" H 2500 4800 50  0001 C CNN "PriceEUR"
+F 5 "C118075" H 2500 4800 50  0001 C CNN "DistOrderNr"
+F 6 "LCSC" H 2500 4800 50  0001 C CNN "Distributor"
 	1    2500 4800
 	1    0    0    -1
@@
 F 2 "Resistor_SMD:R_1206_3216Metric" V 6130 2150 50  0001 C CNN
 F 3 "~" H 6200 2150 50  0001 C CNN
-F 4 "0.01" H 6200 2150 50  0001 C CNN "PriceEUR"
+F 4 "0.0042" H 6200 2150 50  0001 C CNN "PriceEUR"
+F 5 "C104601" H 6200 2150 50  0001 C CNN "DistOrderNr"
+F 6 "LCSC" H 6200 2150 50  0001 C CNN "Distributor"
+F 7 "RTT03101JTP" H 6200 2150 50  0001 C CNN "ManPartNr"
+F 8 "RALEC" H 6200 2150 50  0001 C CNN "Manufacturer"
+F 9 "1kΩ ±5% 0.25W ±100ppm/℃ 1206 Chip Resistor" H 6200 2150 50  0001 C CNN "Notes"
+F 10 "50" H 6200 2150 50  0001 C CNN "PriceForQty"
 	1    6200 2150
 	1    0    0    -1
@@
 	6200 1950 5950 1950
 Wire Wire Line
-	1400 3750 1400 2250
-Connection ~ 1400 2250
-Wire Wire Line
-	1400 2250 1800 2250
+	1500 3750 1500 2250
+Connection ~ 1500 2250
 Wire Wire Line
 	3550 3300 3550 4450
@@
 F 2 "htl_virtual:Virtual-Item" H 9200 6330 50  0001 C CNN
 F 3 "~" V 9200 6400 50  0001 C CNN
-F 4 "Custom" H 9200 6400 50  0001 C CNN "DistOrderNr"
+F 4 "Custom2" H 9200 6400 50  0001 C CNN "DistOrderNr"
 F 5 "Multi-CB" H 9200 6400 50  0001 C CNN "Distributor"
 F 6 "Multi-CB" H 9200 6400 50  0001 C CNN "Manufacturer"
@@
 F 2 "htl_virtual:Virtual-Item" H 9200 6130 50  0001 C CNN
 F 3 "~" V 9200 6200 50  0001 C CNN
-F 4 "Custom" H 9200 6200 50  0001 C CNN "DistOrderNr"
+F 4 "Custom1" H 9200 6200 50  0001 C CNN "DistOrderNr"
 F 5 "Multi-CB" H 9200 6200 50  0001 C CNN "Distributor"
 F 6 "Multi-CB" H 9200 6200 50  0001 C CNN "Manufacturer"
@@
 F 2 "htl_mechanical:mountinghole_d4mm_R5mm" H 9950 5050 50  0001 C CNN
 F 3 "~" H 9950 5050 50  0001 C CNN
-F 4 "NAP" H 9950 5050 50  0001 C CNN "DistOrderNr"
+F 4 "NAP2" H 9950 5050 50  0001 C CNN "DistOrderNr"
 F 5 "NAP" H 9950 5050 50  0001 C CNN "Distributor"
 F 6 "NAP" H 9950 5050 50  0001 C CNN "ManPartNr"
@@
 F 2 "htl_mechanical:mountinghole_d4mm_R5mm" H 9950 5250 50  0001 C CNN
 F 3 "~" H 9950 5250 50  0001 C CNN
-F 4 "NAP" H 9950 5250 50  0001 C CNN "DistOrderNr"
+F 4 "NAP2" H 9950 5250 50  0001 C CNN "DistOrderNr"
 F 5 "NAP" H 9950 5250 50  0001 C CNN "Distributor"
 F 6 "NAP" H 9950 5250 50  0001 C CNN "ManPartNr"
@@
 F 2 "htl_mechanical:mountinghole_d4mm_R5mm" H 9950 5450 50  0001 C CNN
 F 3 "~" H 9950 5450 50  0001 C CNN
-F 4 "NAP" H 9950 5450 50  0001 C CNN "DistOrderNr"
+F 4 "NAP2" H 9950 5450 50  0001 C CNN "DistOrderNr"
 F 5 "NAP" H 9950 5450 50  0001 C CNN "Distributor"
 F 6 "NAP" H 9950 5450 50  0001 C CNN "ManPartNr"
@@
 F 2 "htl_mechanical:mountinghole_d4mm_R5mm" H 9950 5650 50  0001 C CNN
 F 3 "~" H 9950 5650 50  0001 C CNN
-F 4 "NAP" H 9950 5650 50  0001 C CNN "DistOrderNr"
+F 4 "NAP2" H 9950 5650 50  0001 C CNN "DistOrderNr"
 F 5 "NAP" H 9950 5650 50  0001 C CNN "Distributor"
 F 6 "NAP" H 9950 5650 50  0001 C CNN "ManPartNr"
@@
 F 2 "htl_mechanical:paste-fiducial" H 9950 4650 50  0001 C CNN
 F 3 "~" H 9950 4650 50  0001 C CNN
-F 4 "NAP" H 9950 4650 50  0001 C CNN "DistOrderNr"
+F 4 "NAP1" H 9950 4650 50  0001 C CNN "DistOrderNr"
 F 5 "Not a Part" H 9950 4650 50  0001 C CNN "Manufacturer"
 F 6 "0.00" H 9950 4650 50  0001 C CNN "PriceEUR"
+F 7 "NAP" H 9950 4650 50  0001 C CNN "Distributor"
 	1    9950 4650
 	1    0    0    -1
@@
 F 2 "htl_mechanical:paste-fiducial" H 9950 4450 50  0001 C CNN
 F 3 "~" H 9950 4450 50  0001 C CNN
-F 4 "NAP" H 9950 4450 50  0001 C CNN "DistOrderNr"
+F 4 "NAP1" H 9950 4450 50  0001 C CNN "DistOrderNr"
 F 5 "Not a Part" H 9950 4450 50  0001 C CNN "Manufacturer"
 F 6 "0.00" H 9950 4450 50  0001 C CNN "PriceEUR"
+F 7 "NAP" H 9950 4450 50  0001 C CNN "Distributor"
 	1    9950 4450
 	1    0    0    -1
 $EndComp
-Text Notes 8200 3750 0    150  ~ 0
-TODOs:\n* ERC\n* Footprint Federklemmen\n* Footprint Panasonic ELKOs\n* ATmega328 statt Arduino\n
+Text Notes 8200 2100 0    50   ~ 0
+TODO: Footprint Federklemmen\n
+Text Label 3350 2300 0    50   ~ 0
+5V
+$Comp
+L Connector:Screw_Terminal_01x03 J1
+U 1 1 60B4DA3D
+P 1050 2250
+F 0 "J1" H 968 2567 50  0000 C CNN
+F 1 "COM" H 968 2476 50  0000 C CNN
+F 2 "Connector_Phoenix_MSTB:PhoenixContact_MSTBA_2,5_3-G-5,08_1x03_P5.08mm_Horizontal" H 1050 2250 50  0001 C CNN
+F 3 "~" H 1050 2250 50  0001 C CNN
+F 4 "C475145" H 1050 2250 50  0001 C CNN "DistOrderNr"
+F 5 "LCSC" H 1050 2250 50  0001 C CNN "Distributor"
+F 6 "0.1347" H 1050 2250 50  0001 C CNN "PriceEUR"
+F 7 "100" H 1050 2250 50  0001 C CNN "PriceForQty"
+F 8 "3 poles, 5.08mm, 15A 250V AWG14~22 1.5mm² P=5.08mm Spring Clamp System Terminal Block" H 1050 2250 50  0001 C CNN "Notes"
+	1    1050 2250
+	-1   0    0    -1
+$EndComp
+Wire Wire Line
+	1250 2250 1500 2250
+Wire Wire Line
+	1300 2150 1250 2150
+Wire Wire Line
+	1300 2050 1300 2150
+Wire Wire Line
+	1250 2350 1250 2800
+Wire Wire Line
+	1250 2800 4550 2800
+Wire Wire Line
+	1300 2050 1400 2050
+$Sheet
+S 1800 800  1400 700
+U 60BEB366
+F0 "Batterie Varianten" 50
+F1 "batteries.sch" 50
+F2 "Plus" O L 1800 950 50
+F3 "Minus" O L 1800 1350 50
+$EndSheet
+Wire Wire Line
+	1800 950  1400 950
+Wire Wire Line
+	1400 950  1400 2050
+Connection ~ 1400 2050
+Wire Wire Line
+	1400 2050 1800 2050
+Wire Wire Line
+	1800 1350 1500 1350
+Wire Wire Line
+	1500 1350 1500 2250
+Wire Wire Line
+	1500 2250 1800 2250
 $EndSCHEMATC

Commit message: Reviews und ein paar Verbesserungen
Parts:
- D1: Notes LED, green, SMD3216 -> LED, red, SMD3216
- R1: Notes (none) -> 10kΩ ±5% 0.25W ±100ppm/℃ 3216 Chip Resistor
- X1: renamed from J1; value COM -> POWER; footprint Connector_Phoenix_MSTB:PhoenixContact_MSTBA_2,5_3-G-5,08_1x03_P5.08mm_Horizontal -> htl_connectors:Federklemme_KF142_3P_P5.08mm_C475145
- X2: renamed from J2; footprint Connector_Phoenix_MSTB:PhoenixContact_MSTBA_2,5_3-G-5,08_1x03_P5.08mm_Horizontal -> htl_connectors:Federklemme_KF142_3P_P5.08mm_C475145
- X3: renamed from J3; footprint Connector_Phoenix_MSTB:PhoenixContact_MSTBA_2,5_3-G-5,08_1x03_P5.08mm_Horizontal -> htl_connectors:Federklemme_KF142_3P_P5.08mm_C475145
Other:
- note added: "TODO: Footprint\nHier gibts noch ein problem mit der x-Ausrichtung\nDas 3D-Modell passt offenbar nicht zu 2D-Skizze\nPins sollten zum Drahtloch leicht versetzt sein."
- note added: "TODO: umstellen auf RS485\nfür die Bus-Fähigkeit\nLCSC C269866"
- note removed: "TODO: Footprint Federklemmen\n"
- moved on the sheet: C1, C2, C3, C4, SW1, SW2, SW3, SW4
