File: kicad/power-stage.sch (KiCad schematic (older format))
At the start: 13 parts, among them Q1 KND3508A, U7 PN7006A

Commit message: wip, bugfixes für v21.0.1
Parts:
- C21: value 1u -> 1u/100V; DistOrderNr C1848 -> C70463; ManPartNr CL31B105KBHNNNE -> CC1206KKX7R0BB105; Manufacturer Samsung -> YAGEO; Notes 1uF ±10% 50V X7R Multilayer Ceramic Capacitors MLCC -> X7R ±10% 100V 1uF 1206 Multilayer Ceramic Capacitors MLCC; PriceEUR 0.0225 -> 0.0535; PriceForQty 100 -> 50; Weblink (none) -> https://www.lcsc.com/product-detail/Multilayer-Ceramic-Capa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
- R29: DistOrderNr C113307 -> C245445; ManPartNr RC1206JR-07100RL -> CR1206F100RP05Z; Manufacturer YAGEO -> Ever Ohms Tech; Notes 100Ω ±5% 0.25W ±100ppm/℃ 1206 Chip Resistor -> 0.25W ±1% ±100ppm/℃ 100Ω 1206; PriceEUR 0.0037 -> 0.0030
- R30: Notes (none) -> 10kΩ ±5% 0.25W ±100ppm/℃ 3216 Chip Resistor
Connections:
- net GND: no longer D16.2 (A)
- net HTC-: now also D16.2 (A)
Other:
- moved on the sheet: D16
Changed lines of the file:
@@
 Sheet 5 10
 Title "HTL Lötregler Mini"
-Date "2021-06-01"
-Rev "21.0.0"
+Date "2021-09-22"
+Rev "21.0.1-dev"
 Comp "HTL Steyr"
 Comment1 "Prof. Karl Zeilhofer et al."
@@
 F 5 "C118075" H 5600 3900 50  0001 C CNN "DistOrderNr"
 F 6 "LCSC" H 5600 3900 50  0001 C CNN "Distributor"
+F 7 "10kΩ ±5% 0.25W ±100ppm/℃ 3216 Chip Resistor" H 5600 3900 50  0001 C CNN "Notes"
 	1    5600 3900
 	1    0    0    -1
@@
 P 4500 2900
 F 0 "C21" H 4615 2946 50  0000 L CNN
-F 1 "1u" H 4615 2855 50  0000 L CNN
+F 1 "1u/100V" H 4615 2855 50  0000 L CNN
 F 2 "Capacitor_SMD:C_1206_3216Metric" H 4538 2750 50  0001 C CNN
 F 3 "~" H 4500 2900 50  0001 C CNN
-F 4 "C1848" H 4500 2900 50  0001 C CNN "DistOrderNr"
+F 4 "C70463" H 4500 2900 50  0001 C CNN "DistOrderNr"
 F 5 "LCSC" H 4500 2900 50  0001 C CNN "Distributor"
-F 6 "CL31B105KBHNNNE" H 4500 2900 50  0001 C CNN "ManPartNr"
-F 7 "Samsung" H 4500 2900 50  0001 C CNN "Manufacturer"
-F 8 "1uF ±10% 50V X7R Multilayer Ceramic Capacitors MLCC" H 4500 2900 50  0001 C CNN "Notes"
-F 9 "0.0225" H 4500 2900 50  0001 C CNN "PriceEUR"
-F 10 "100" H 4500 2900 50  0001 C CNN "PriceForQty"
+F 6 "CC1206KKX7R0BB105" H 4500 2900 50  0001 C CNN "ManPartNr"
+F 7 "YAGEO" H 4500 2900 50  0001 C CNN "Manufacturer"
+F 8 "X7R ±10% 100V 1uF 1206 Multilayer Ceramic Capacitors MLCC" H 4500 2900 50  0001 C CNN "Notes"
+F 9 "0.0535 " H 4500 2900 50  0001 C CNN "PriceEUR"
+F 10 "50" H 4500 2900 50  0001 C CNN "PriceForQty"
+F 11 "https://www.lcsc.com/product-detail/Multilayer-Ceramic-Capacitors-MLCC-SMD-SMT_HUI-JU-NC1206B105K101CEPN_C710469.html" H 4500 2900 50  0001 C CNN "Weblink"
 	1    4500 2900
 	1    0    0    -1
@@
 	6650 4300 7550 4300
 Wire Wire Line
-	5600 3650 7550 3650
+	5600 3650 6650 3650
 $Comp
 L power:GNDPWR #PWR044
@@
 F 2 "Resistor_SMD:R_1206_3216Metric" V 4680 3200 50  0001 C CNN
 F 3 "~" H 4750 3200 50  0001 C CNN
-F 4 "0.0037" H 4750 3200 50  0001 C CNN "PriceEUR"
-F 5 "C113307" H 4750 3200 50  0001 C CNN "DistOrderNr"
+F 4 "0.0030" H 4750 3200 50  0001 C CNN "PriceEUR"
+F 5 "C245445" H 4750 3200 50  0001 C CNN "DistOrderNr"
 F 6 "LCSC" H 4750 3200 50  0001 C CNN "Distributor"
-F 7 "RC1206JR-07100RL" H 4750 3200 50  0001 C CNN "ManPartNr"
-F 8 "YAGEO" H 4750 3200 50  0001 C CNN "Manufacturer"
-F 9 "100Ω ±5% 0.25W ±100ppm/℃ 1206 Chip Resistor" H 4750 3200 50  0001 C CNN "Notes"
+F 7 "CR1206F100RP05Z" H 4750 3200 50  0001 C CNN "ManPartNr"
+F 8 "Ever Ohms Tech" H 4750 3200 50  0001 C CNN "Manufacturer"
+F 9 "0.25W ±1% ±100ppm/℃ 100Ω 1206" H 4750 3200 50  0001 C CNN "Notes"
 F 10 "500" H 4750 3200 50  0001 C CNN "PriceForQty"
 	1    4750 3200
@@
 L htl_semiconductors:D_Schottky D16
 U 1 1 60D9E4E3
-P 5100 3900
-F 0 "D16" H 5100 3675 50  0000 C CNN
-F 1 "SS210" H 5100 3766 50  0000 C CNN
-F 2 "htl_smd:D_SMA_wide" H 5100 3900 50  0001 C CNN
-F 3 "~" H 5100 3900 50  0001 C CNN
-F 4 "C2683692" H 5100 3900 50  0001 C CNN "DistOrderNr"
-F 5 "LCSC" H 5100 3900 50  0001 C CNN "Distributor"
-F 6 "SS210A-W" H 5100 3900 50  0001 C CNN "ManPartNr"
-F 7 "ZHIDE" H 5100 3900 50  0001 C CNN "Manufacturer"
-F 8 "100V 2A 850mV @ 2A SMA(DO-214AC) Schottky Barrier Diodes" H 5100 3900 50  0001 C CNN "Notes"
-F 9 "0.0155" H 5100 3900 50  0001 C CNN "PriceEUR"
-F 10 "200" H 5100 3900 50  0001 C CNN "PriceForQty"
-F 11 "https://lcsc.com/product-detail/Schottky-Barrier-Diodes-SBD_ZHIDE-SS210A-W_C2683692.html" H 5100 3900 50  0001 C CNN "Weblink"
-	1    5100 3900
+P 6650 3950
+F 0 "D16" H 6650 3725 50  0000 C CNN
+F 1 "SS210" H 6650 3816 50  0000 C CNN
+F 2 "htl_smd:D_SMA_wide" H 6650 3950 50  0001 C CNN
+F 3 "~" H 6650 3950 50  0001 C CNN
+F 4 "C2683692" H 6650 3950 50  0001 C CNN "DistOrderNr"
+F 5 "LCSC" H 6650 3950 50  0001 C CNN "Distributor"
+F 6 "SS210A-W" H 6650 3950 50  0001 C CNN "ManPartNr"
+F 7 "ZHIDE" H 6650 3950 50  0001 C CNN "Manufacturer"
+F 8 "100V 2A 850mV @ 2A SMA(DO-214AC) Schottky Barrier Diodes" H 6650 3950 50  0001 C CNN "Notes"
+F 9 "0.0155" H 6650 3950 50  0001 C CNN "PriceEUR"
+F 10 "200" H 6650 3950 50  0001 C CNN "PriceForQty"
+F 11 "https://lcsc.com/product-detail/Schottky-Barrier-Diodes-SBD_ZHIDE-SS210A-W_C2683692.html" H 6650 3950 50  0001 C CNN "Weblink"
+	1    6650 3950
 	0    1    1    0
 $EndComp
-$Comp
-L power:GND #PWR064
-U 1 1 60D9F0D3
-P 5100 4150
-F 0 "#PWR064" H 5100 3900 50  0001 C CNN
-F 1 "GND" H 5105 3977 50  0000 C CNN
-F 2 "" H 5100 4150 50  0001 C CNN
-F 3 "" H 5100 4150 50  0001 C CNN
-	1    5100 4150
-	1    0    0    -1
-$EndComp
-Wire Wire Line
-	5100 4150 5100 4050
-Wire Wire Line
-	5100 3750 5100 3650
+Wire Wire Line
+	6650 3650 6650 3800
+Wire Wire Line
+	6650 4100 6650 4300
+Connection ~ 6650 3650
+Wire Wire Line
+	6650 3650 7550 3650
+Connection ~ 6650 4300
 $EndSCHEMATC

Commit message: Workaround zu Isssue#7, USB Bootproblem
Other:
- note added: "Pulldown\nfür Reset-Zustand"
Changed lines of the file:
@@
 	6650 3650 7550 3650
 Connection ~ 6650 4300
+Text Notes 1700 4550 0    50   ~ 0
+Pulldown\nfür Reset-Zustand
 $EndSCHEMATC

Commit message: BOM aktualisiert, Zenerdiode: Pinout IPC-konform gestaltet, ...
siehe https://gitlab.com/kicad/libraries/kicad-symbols/-/issues/3157
Parts:
- C20: Index (none) -> 7
- C21: Index (none) -> 10
- D16, D7: Index (none) -> 49
- Q1: Index (none) -> 14
- R26, R27, R28: Index (none) -> 12
- R29: Index (none) -> 28
- R30: Index (none) -> 15
- R31: Index (none) -> 42
- R65: DistOrderNr (none) -> R3216-56k; Distributor LCSC -> AufLager; Index (none) -> 58
- U7: Index (none) -> 38; NotesAlt (none) -> https://www.lcsc.com/product-detail/Gate-Drive-ICs_EG-Micro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
Changed lines of the file:
@@
 F 9 "100" H 5500 3200 50  0001 C CNN "PriceForQty"
 F 10 "https://lcsc.com/product-detail/MOSFET_KIA-Semicon-Tech-KND3508A_C116513.html" H 5500 3200 50  0001 C CNN "Weblink"
+F 11 "14" H 5500 3200 50  0001 C CNN "Index"
 	1    5500 3200
 	1    0    0    -1
@@
 F 6 "LCSC" H 5600 3900 50  0001 C CNN "Distributor"
 F 7 "10kΩ ±5% 0.25W ±100ppm/℃ 3216 Chip Resistor" H 5600 3900 50  0001 C CNN "Notes"
+F 8 "15" H 5600 3900 50  0001 C CNN "Index"
 	1    5600 3900
 	1    0    0    -1
@@
 F 10 "50" H 4500 2900 50  0001 C CNN "PriceForQty"
 F 11 "https://www.lcsc.com/product-detail/Multilayer-Ceramic-Capacitors-MLCC-SMD-SMT_HUI-JU-NC1206B105K101CEPN_C710469.html" H 4500 2900 50  0001 C CNN "Weblink"
+F 12 "10" H 4500 2900 50  0001 C CNN "Index"
 	1    4500 2900
 	1    0    0    -1
@@
 F 10 "200" H 4000 2500 50  0001 C CNN "PriceForQty"
 F 11 "https://lcsc.com/product-detail/Schottky-Barrier-Diodes-SBD_ZHIDE-SS210A-W_C2683692.html" H 4000 2500 50  0001 C CNN "Weblink"
+F 12 "49" H 4000 2500 50  0001 C CNN "Index"
 	1    4000 2500
 	-1   0    0    1
@@
 F 9 "0.0233" H 2650 2900 50  0001 C CNN "PriceEUR"
 F 10 "100" H 2650 2900 50  0001 C CNN "PriceForQty"
+F 11 "7" H 2650 2900 50  0001 C CNN "Index"
 	1    2650 2900
 	1    0    0    -1
@@
 F 9 "1kΩ ±5% 0.25W ±100ppm/℃ 1206 Chip Resistor" H 2000 3750 50  0001 C CNN "Notes"
 F 10 "50" H 2000 3750 50  0001 C CNN "PriceForQty"
+F 11 "12" H 2000 3750 50  0001 C CNN "Index"
 	1    2000 3750
 	1    0    0    -1
@@
 F 8 "100" H 3750 3300 50  0001 C CNN "PriceForQty"
 F 9 "https://lcsc.com/product-detail/Full-bridge-half-bridge-Driver_Wuxi-Chipown-Micro-electronics-PN7006ASEC-R1_C414194.html" H 3750 3300 50  0001 C CNN "Weblink"
+F 10 "38" H 3750 3300 50  0001 C CNN "Index"
+F 11 "https://www.lcsc.com/product-detail/Gate-Drive-ICs_EG-Micro-EG3112_C111908.html" H 3750 3300 50  0001 C CNN "NotesAlt"
 	1    3750 3300
 	1    0    0    -1
@@
 F 9 "1kΩ ±5% 0.25W ±100ppm/℃ 1206 Chip Resistor" H 4250 3800 50  0001 C CNN "Notes"
 F 10 "50" H 4250 3800 50  0001 C CNN "PriceForQty"
+F 11 "12" H 4250 3800 50  0001 C CNN "Index"
 	1    4250 3800
 	1    0    0    -1
@@
 F 9 "1kΩ ±5% 0.25W ±100ppm/℃ 1206 Chip Resistor" H 3250 3800 50  0001 C CNN "Notes"
 F 10 "50" H 3250 3800 50  0001 C CNN "PriceForQty"
+F 11 "12" H 3250 3800 50  0001 C CNN "Index"
 	1    3250 3800
 	1    0    0    -1
@@
 F 6 "0.2596" H 6650 4600 50  0001 C CNN "PriceEUR"
 F 7 "100" H 6650 4600 50  0001 C CNN "PriceForQty"
+F 8 "42" H 6650 4600 50  0001 C CNN "Index"
 	1    6650 4600
 	1    0    0    -1
@@
 F 9 "0.25W ±1% ±100ppm/℃ 100Ω 1206" H 4750 3200 50  0001 C CNN "Notes"
 F 10 "500" H 4750 3200 50  0001 C CNN "PriceForQty"
+F 11 "28" H 4750 3200 50  0001 C CNN "Index"
 	1    4750 3200
 	0    1    1    0
@@
 F 3 "~" H 5100 3400 50  0001 C CNN
 F 4 "0.01" H 5100 3400 50  0001 C CNN "PriceEUR"
-F 5 "LCSC" H 5100 3400 50  0001 C CNN "Distributor"
+F 5 "AufLager" H 5100 3400 50  0001 C CNN "Distributor"
+F 6 "R3216-56k" H 5100 3400 50  0001 C CNN "DistOrderNr"
+F 7 "58" H 5100 3400 50  0001 C CNN "Index"
 	1    5100 3400
 	1    0    0    -1
@@
 F 10 "200" H 6650 3950 50  0001 C CNN "PriceForQty"
 F 11 "https://lcsc.com/product-detail/Schottky-Barrier-Diodes-SBD_ZHIDE-SS210A-W_C2683692.html" H 6650 3950 50  0001 C CNN "Weblink"
+F 12 "49" H 6650 3950 50  0001 C CNN "Index"
 	1    6650 3950
 	0    1    1    0
