File: kicad/uart-rs232-rs485.sch (KiCad schematic (older format))
At the start: 17 parts, among them U10 MAX3232

Commit message: um Option RS485 erweitert
Parts:
- added R? (x2): 10R, Resistor_SMD:R_1206_3216Metric, symbol Device:R
- added R? (x2): 1k, Resistor_SMD:R_1206_3216Metric, symbol Device:R
Connections:
- net 5V: now also R?.1
- net GNDPWR: now also R?.2
- net RxD_B: now also R?.1; no longer D15.1 (A), JP?.2 (C)
- net at JP?.1 (A), U?.6 (A): now also R?.2
- net at JP?.1 (A), U?.7 (B): now also R?.1
- net TXD_A: no longer names the net of D14.1 (A), JP?.2 (C)
- net TXD_A: now also R?.2
- net UART_Rx1 renamed UART_RxD
- net UART_Tx1 renamed UART_TxD
- new net: D15.1 (A), JP?.2 (C), R?.2
- new net TxD_A: R?.1
Changed lines of the file:
@@
 	4950 1250 4800 1250
 Text HLabel 1650 3950 0    50   Input ~ 0
-UART_Tx1
+UART_TxD
 Wire Wire Line
 	2250 2750 3400 2750
@@
 Wire Wire Line
 	3250 3350 3400 3350
-Text HLabel 9950 4150 2    50   Input ~ 0
+Text HLabel 10450 4150 2    50   Input ~ 0
 RxD_B
-Text HLabel 9950 3800 2    50   Output ~ 0
-TXD_A
+Text HLabel 10450 3800 2    50   Output ~ 0
+TxD_A
 Wire Wire Line
 	5150 3350 5000 3350
@@
 $EndComp
 Text HLabel 1650 4350 0    50   Output ~ 0
-UART_Rx1
+UART_RxD
 NoConn ~ 3250 2950
 NoConn ~ 3250 3350
@@
 	8500 4150 9700 4150
 Wire Wire Line
-	9950 3800 9050 3800
+	10450 3800 10300 3800
 Wire Wire Line
 	9050 4300 9050 3800
@@
 Connection ~ 9700 4150
 Wire Wire Line
-	9700 4150 9950 4150
+	9700 4150 10000 4150
 $Comp
 L Jumper:SolderJumper_3_Open JP?
@@
 	8100 4000 8100 5700
 Wire Wire Line
-	8100 5700 5450 5700
-Wire Wire Line
-	5450 5400 8350 5400
+	8100 5700 6350 5700
+Wire Wire Line
+	5450 5400 6550 5400
 Wire Wire Line
 	8350 5400 8350 4350
@@
 Wire Wire Line
 	5050 6250 5050 6100
+$Comp
+L Device:R R?
+U 1 1 609BC636
+P 10150 3800
+F 0 "R?" V 9943 3800 50  0000 C CNN
+F 1 "10R" V 10034 3800 50  0000 C CNN
+F 2 "Resistor_SMD:R_1206_3216Metric" V 10080 3800 50  0001 C CNN
+F 3 "~" H 10150 3800 50  0001 C CNN
+	1    10150 3800
+	0    1    1    0
+$EndComp
+Wire Wire Line
+	10000 3800 9050 3800
+$Comp
+L Device:R R?
+U 1 1 609BC9D3
+P 10150 4150
+F 0 "R?" V 9943 4150 50  0000 C CNN
+F 1 "10R" V 10034 4150 50  0000 C CNN
+F 2 "Resistor_SMD:R_1206_3216Metric" V 10080 4150 50  0001 C CNN
+F 3 "~" H 10150 4150 50  0001 C CNN
+	1    10150 4150
+	0    1    1    0
+$EndComp
+Wire Wire Line
+	10300 4150 10450 4150
+$Comp
+L Device:R R?
+U 1 1 609BF4B9
+P 6350 5100
+AR Path="/608DBC83/609BF4B9" Ref="R?"  Part="1"
+AR Path="/60A756E2/609BF4B9" Ref="R?"  Part="1"
+F 0 "R?" H 6420 5146 50  0000 L CNN
+F 1 "1k" H 6420 5055 50  0000 L CNN
+F 2 "Resistor_SMD:R_1206_3216Metric" V 6280 5100 50  0001 C CNN
+F 3 "~" H 6350 5100 50  0001 C CNN
+F 4 "0.0042" H 6350 5100 50  0001 C CNN "PriceEUR"
+F 5 "C104601" H 6350 5100 50  0001 C CNN "DistOrderNr"
+F 6 "LCSC" H 6350 5100 50  0001 C CNN "Distributor"
+F 7 "RTT03101JTP" H 6350 5100 50  0001 C CNN "ManPartNr"
+F 8 "RALEC" H 6350 5100 50  0001 C CNN "Manufacturer"
+F 9 "1kΩ ±5% 0.25W ±100ppm/℃ 1206 Chip Resistor" H 6350 5100 50  0001 C CNN "Notes"
+F 10 "50" H 6350 5100 50  0001 C CNN "PriceForQty"
+	1    6350 5100
+	1    0    0    -1
+$EndComp
+Text Label 6200 4650 0    50   ~ 0
+5V_COM
+Wire Wire Line
+	6200 4650 6350 4650
+Wire Wire Line
+	6350 4650 6350 4950
+Wire Wire Line
+	6350 5250 6350 5700
+Connection ~ 6350 5700
+Wire Wire Line
+	6350 5700 5450 5700
+$Comp
+L Device:R R?
+U 1 1 609C36A8
+P 6550 6000
+AR Path="/608DBC83/609C36A8" Ref="R?"  Part="1"
+AR Path="/60A756E2/609C36A8" Ref="R?"  Part="1"
+F 0 "R?" H 6620 6046 50  0000 L CNN
+F 1 "1k" H 6620 5955 50  0000 L CNN
+F 2 "Resistor_SMD:R_1206_3216Metric" V 6480 6000 50  0001 C CNN
+F 3 "~" H 6550 6000 50  0001 C CNN
+F 4 "0.0042" H 6550 6000 50  0001 C CNN "PriceEUR"
+F 5 "C104601" H 6550 6000 50  0001 C CNN "DistOrderNr"
+F 6 "LCSC" H 6550 6000 50  0001 C CNN "Distributor"
+F 7 "RTT03101JTP" H 6550 6000 50  0001 C CNN "ManPartNr"
+F 8 "RALEC" H 6550 6000 50  0001 C CNN "Manufacturer"
+F 9 "1kΩ ±5% 0.25W ±100ppm/℃ 1206 Chip Resistor" H 6550 6000 50  0001 C CNN "Notes"
+F 10 "50" H 6550 6000 50  0001 C CNN "PriceForQty"
+	1    6550 6000
+	1    0    0    -1
+$EndComp
+$Comp
+L power:GNDPWR #PWR?
+U 1 1 609C3BAE
+P 6550 6250
+F 0 "#PWR?" H 6550 6050 50  0001 C CNN
+F 1 "GNDPWR" H 6554 6096 50  0000 C CNN
+F 2 "" H 6550 6200 50  0001 C CNN
+F 3 "" H 6550 6200 50  0001 C CNN
+	1    6550 6250
+	1    0    0    -1
+$EndComp
+Wire Wire Line
+	6550 6250 6550 6150
+Wire Wire Line
+	6550 5850 6550 5400
+Connection ~ 6550 5400
+Wire Wire Line
+	6550 5400 8350 5400
 $EndSCHEMATC

Commit message: Layout
Parts:
- gave numbers to parts that had none: 11
Connections:
- net 5V: now also C39.2
- net at JP6.2 (C), R57.2: no longer D14.1 (A)
- net at JP6.3 (B), R52.1: now also D14.1 (A)
- net at JP7.2 (C), R58.2: no longer D15.1 (A)
- net at JP7.3 (B), R53.1: now also D15.1 (A)
Other:
- moved on the sheet: D14, D15
Changed lines of the file:
@@
 L htl_semiconductors:DiodeTVS_Bidirek D14
 U 1 1 60A953FA
-P 9050 4450
-F 0 "D14" V 9012 4529 50  0000 L CNN
-F 1 "SMAJ8.0CA" V 9096 4529 40  0000 L CNN
-F 2 "Diode_SMD:D_SMA" V 9134 4529 60  0001 L CNN
-F 3 "" H 9000 4450 60  0000 C CNN
-F 4 "C908814" H 9050 4450 50  0001 C CNN "DistOrderNr"
-F 5 "LCSC" H 9050 4450 50  0001 C CNN "Distributor"
-F 6 "SMAJ8.0CA" H 9050 4450 50  0001 C CNN "ManPartNr"
-F 7 "GOODWORK" H 9050 4450 50  0001 C CNN "Manufacturer"
-F 8 "Bidirectional 8V 8.89V 13.6V 29.4A SMA(DO-214AC) TVS" H 9050 4450 50  0001 C CNN "Notes"
-F 9 "0.0243" H 9050 4450 50  0001 C CNN "PriceEUR"
-F 10 "100" H 9050 4450 50  0001 C CNN "PriceForQty"
-F 11 "https://lcsc.com/product-detail/Pre-ordered-transistors_GOODWORK-SMAJ8-0CA_C908814.html" H 9050 4450 50  0001 C CNN "Weblink"
-	1    9050 4450
+P 7150 3450
+F 0 "D14" V 7112 3529 50  0000 L CNN
+F 1 "SMAJ8.0CA" V 7196 3529 40  0000 L CNN
+F 2 "Diode_SMD:D_SMA" V 7234 3529 60  0001 L CNN
+F 3 "" H 7100 3450 60  0000 C CNN
+F 4 "C908814" H 7150 3450 50  0001 C CNN "DistOrderNr"
+F 5 "LCSC" H 7150 3450 50  0001 C CNN "Distributor"
+F 6 "SMAJ8.0CA" H 7150 3450 50  0001 C CNN "ManPartNr"
+F 7 "GOODWORK" H 7150 3450 50  0001 C CNN "Manufacturer"
+F 8 "Bidirectional 8V 8.89V 13.6V 29.4A SMA(DO-214AC) TVS" H 7150 3450 50  0001 C CNN "Notes"
+F 9 "0.0243" H 7150 3450 50  0001 C CNN "PriceEUR"
+F 10 "100" H 7150 3450 50  0001 C CNN "PriceForQty"
+F 11 "https://lcsc.com/product-detail/Pre-ordered-transistors_GOODWORK-SMAJ8-0CA_C908814.html" H 7150 3450 50  0001 C CNN "Weblink"
+	1    7150 3450
 	0    1    1    0
 $EndComp
@@
 L htl_semiconductors:DiodeTVS_Bidirek D15
 U 1 1 60A993E0
-P 9700 4450
-F 0 "D15" V 9662 4529 50  0000 L CNN
-F 1 "SMAJ8.0CA" V 9746 4529 40  0000 L CNN
-F 2 "Diode_SMD:D_SMA" V 9784 4529 60  0001 L CNN
-F 3 "" H 9650 4450 60  0000 C CNN
-F 4 "C908814" H 9700 4450 50  0001 C CNN "DistOrderNr"
-F 5 "LCSC" H 9700 4450 50  0001 C CNN "Distributor"
-F 6 "SMAJ8.0CA" H 9700 4450 50  0001 C CNN "ManPartNr"
-F 7 "GOODWORK" H 9700 4450 50  0001 C CNN "Manufacturer"
-F 8 "Bidirectional 8V 8.89V 13.6V 29.4A SMA(DO-214AC) TVS" H 9700 4450 50  0001 C CNN "Notes"
-F 9 "0.0243" H 9700 4450 50  0001 C CNN "PriceEUR"
-F 10 "100" H 9700 4450 50  0001 C CNN "PriceForQty"
-F 11 "https://lcsc.com/product-detail/Pre-ordered-transistors_GOODWORK-SMAJ8-0CA_C908814.html" H 9700 4450 50  0001 C CNN "Weblink"
-	1    9700 4450
+P 7800 3450
+F 0 "D15" V 7762 3529 50  0000 L CNN
+F 1 "SMAJ8.0CA" V 7846 3529 40  0000 L CNN
+F 2 "Diode_SMD:D_SMA" V 7884 3529 60  0001 L CNN
+F 3 "" H 7750 3450 60  0000 C CNN
+F 4 "C908814" H 7800 3450 50  0001 C CNN "DistOrderNr"
+F 5 "LCSC" H 7800 3450 50  0001 C CNN "Distributor"
+F 6 "SMAJ8.0CA" H 7800 3450 50  0001 C CNN "ManPartNr"
+F 7 "GOODWORK" H 7800 3450 50  0001 C CNN "Manufacturer"
+F 8 "Bidirectional 8V 8.89V 13.6V 29.4A SMA(DO-214AC) TVS" H 7800 3450 50  0001 C CNN "Notes"
+F 9 "0.0243" H 7800 3450 50  0001 C CNN "PriceEUR"
+F 10 "100" H 7800 3450 50  0001 C CNN "PriceForQty"
+F 11 "https://lcsc.com/product-detail/Pre-ordered-transistors_GOODWORK-SMAJ8-0CA_C908814.html" H 7800 3450 50  0001 C CNN "Weblink"
+	1    7800 3450
 	0    1    1    0
 $EndComp
@@
 	4200 3850 4200 4000
 $Comp
-L Interface_UART:MAX3486 U?
+L Interface_UART:MAX3486 U11
 U 1 1 60976A63
 P 5050 5500
-F 0 "U?" H 4500 6100 50  0000 C CNN
+F 0 "U11" H 4500 6100 50  0000 C CNN
 F 1 "YD3082EESA" H 4700 6000 50  0000 C CNN
 F 2 "Package_SO:SO-8_3.9x4.9mm_P1.27mm" H 5050 4800 50  0001 C CNN
@@
 RS485-Treiber
 $Comp
-L power:GNDPWR #PWR?
+L power:GNDPWR #PWR0101
 U 1 1 60981A41
-P 9400 4850
-F 0 "#PWR?" H 9400 4650 50  0001 C CNN
-F 1 "GNDPWR" H 9404 4696 50  0000 C CNN
-F 2 "" H 9400 4800 50  0001 C CNN
-F 3 "" H 9400 4800 50  0001 C CNN
-	1    9400 4850
-	1    0    0    -1
-$EndComp
-Wire Wire Line
-	9050 4600 9050 4750
-Wire Wire Line
-	9050 4750 9400 4750
-Wire Wire Line
-	9700 4750 9700 4600
-Wire Wire Line
-	9400 4850 9400 4750
-Connection ~ 9400 4750
-Wire Wire Line
-	9400 4750 9700 4750
-Wire Wire Line
-	8500 4150 9700 4150
+P 7500 3850
+F 0 "#PWR0101" H 7500 3650 50  0001 C CNN
+F 1 "GNDPWR" H 7504 3696 50  0000 C CNN
+F 2 "" H 7500 3800 50  0001 C CNN
+F 3 "" H 7500 3800 50  0001 C CNN
+	1    7500 3850
+	1    0    0    -1
+$EndComp
+Wire Wire Line
+	7150 3600 7150 3750
+Wire Wire Line
+	7150 3750 7500 3750
+Wire Wire Line
+	7800 3750 7800 3600
+Wire Wire Line
+	7500 3850 7500 3750
+Connection ~ 7500 3750
+Wire Wire Line
+	7500 3750 7800 3750
 Wire Wire Line
 	10450 3800 10300 3800
 Wire Wire Line
-	9050 4300 9050 3800
-Connection ~ 9050 3800
-Wire Wire Line
-	9050 3800 8250 3800
-Wire Wire Line
-	9700 4300 9700 4150
-Connection ~ 9700 4150
-Wire Wire Line
-	9700 4150 10000 4150
-$Comp
-L Jumper:SolderJumper_3_Open JP?
+	7150 3300 7150 2750
+Wire Wire Line
+	7800 3300 7800 3150
+$Comp
+L Jumper:SolderJumper_3_Open JP6
 U 1 1 6098A36F
 P 8100 3800
-F 0 "JP?" V 8146 3868 50  0000 L CNN
+F 0 "JP6" V 8146 3868 50  0000 L CNN
 F 1 "COM" V 8055 3868 50  0000 L CNN
 F 2 "Jumper:SolderJumper-3_P2.0mm_Open_TrianglePad1.0x1.5mm_NumberLabels" H 8100 3800 50  0001 C CNN
@@
 $EndComp
 $Comp
-L Jumper:SolderJumper_3_Open JP?
+L Jumper:SolderJumper_3_Open JP7
 U 1 1 6098BF4F
 P 8350 4150
-F 0 "JP?" V 8396 4218 50  0000 L CNN
+F 0 "JP7" V 8396 4218 50  0000 L CNN
 F 1 "COM" V 8305 4218 50  0000 L CNN
 F 2 "Jumper:SolderJumper-3_P2.0mm_Open_TrianglePad1.0x1.5mm_NumberLabels" H 8350 4150 50  0001 C CNN
@@
 	8100 3600 8100 2750
 Wire Wire Line
-	6850 2750 8100 2750
+	6850 2750 7150 2750
 Wire Wire Line
 	8350 3150 8350 3950
 Wire Wire Line
-	6850 3150 8350 3150
+	6850 3150 7800 3150
 Wire Wire Line
 	8100 4000 8100 5700
@@
 	4900 4800 5050 4800
 Wire Wire Line
-	5050 4800 5050 5000
+	5050 4800 5050 4900
 $Comp
 L Device:C C?
@@
 AR Path="/5FA85ABF/5F7FE44C/60992A97" Ref="C?"  Part="1"
 AR Path="/608DBC83/60A7272B/60992A97" Ref="C?"  Part="1"
-AR Path="/60A756E2/60992A97" Ref="C?"  Part="1"
-F 0 "C?" V 5248 4900 50  0000 C CNN
+AR Path="/60A756E2/60992A97" Ref="C39"  Part="1"
+F 0 "C39" V 5248 4900 50  0000 C CNN
 F 1 "100n" V 5339 4900 50  0000 C CNN
 F 2 "Capacitor_SMD:C_1206_3216Metric" H 5538 4750 50  0001 C CNN
@@
 AR Path="/5FA85ABF/5F7FE44C/60992A9E" Ref="#PWR?"  Part="1"
 AR Path="/608DBC83/60A7272B/60992A9E" Ref="#PWR?"  Part="1"
-AR Path="/60A756E2/60992A9E" Ref="#PWR?"  Part="1"
-F 0 "#PWR?" H 5800 4650 50  0001 C CNN
+AR Path="/60A756E2/60992A9E" Ref="#PWR0102"  Part="1"
+F 0 "#PWR0102" H 5800 4650 50  0001 C CNN
 F 1 "GND" V 5805 4772 50  0000 R CNN
 F 2 "" H 5800 4900 50  0001 C CNN
@@
 	5800 4900 5650 4900
 $Comp
-L Jumper:SolderJumper_3_Open JP?
+L Jumper:SolderJumper_3_Open JP4
 U 1 1 60993DCC
 P 2250 3950
-F 0 "JP?" V 2296 4018 50  0000 L CNN
+F 0 "JP4" V 2296 4018 50  0000 L CNN
 F 1 "UART" V 2205 4018 50  0000 L CNN
 F 2 "Jumper:SolderJumper-3_P2.0mm_Open_TrianglePad1.0x1.5mm_NumberLabels" H 2250 3950 50  0001 C CNN
@@
 $EndComp
 $Comp
-L Jumper:SolderJumper_3_Open JP?
+L Jumper:SolderJumper_3_Open JP5
 U 1 1 60994A79
 P 2550 4350
-F 0 "JP?" V 2596 4418 50  0000 L CNN
+F 0 "JP5" V 2596 4418 50  0000 L CNN
 F 1 "UART" V 2505 4418 50  0000 L CNN
 F 2 "Jumper:SolderJumper-3_P2.0mm_Open_TrianglePad1.0x1.5mm_NumberLabels" H 2550 4350 50  0001 C CNN
@@
 P 3900 5950
 AR Path="/608DBC3C/609A0BB7" Ref="R?"  Part="1"
-AR Path="/60A756E2/609A0BB7" Ref="R?"  Part="1"
-F 0 "R?" H 3970 5996 50  0000 L CNN
+AR Path="/60A756E2/609A0BB7" Ref="R54"  Part="1"
+F 0 "R54" H 3970 5996 50  0000 L CNN
 F 1 "3k3" H 3970 5905 50  0000 L CNN
 F 2 "Resistor_SMD:R_1206_3216Metric" V 3830 5950 50  0001 C CNN
@@
 	3900 5550 4650 5550
 $Comp
-L power:GNDPWR #PWR?
+L power:GNDPWR #PWR0103
 U 1 1 609A54EB
 P 3900 6250
-F 0 "#PWR?" H 3900 6050 50  0001 C CNN
+F 0 "#PWR0103" H 3900 6050 50  0001 C CNN
 F 1 "GNDPWR" H 3904 6096 50  0000 C CNN
 F 2 "" H 3900 6200 50  0001 C CNN
@@
 	3900 6250 3900 6100
 $Comp
-L power:GNDPWR #PWR?
+L power:GNDPWR #PWR0104
 U 1 1 609A70BD
 P 5050 6250
-F 0 "#PWR?" H 5050 6050 50  0001 C CNN
+F 0 "#PWR0104" H 5050 6050 50  0001 C CNN
 F 1 "GNDPWR" H 5054 6096 50  0000 C CNN
 F 2 "" H 5050 6200 50  0001 C CNN
@@
 	5050 6250 5050 6100
 $Comp
-L Device:R R?
+L Device:R R57
 U 1 1 609BC636
 P 10150 3800
-F 0 "R?" V 9943 3800 50  0000 C CNN
+F 0 "R57" V 9943 3800 50  0000 C CNN
 F 1 "10R" V 10034 3800 50  0000 C CNN
 F 2 "Resistor_SMD:R_1206_3216Metric" V 10080 3800 50  0001 C CNN
@@
 	0    1    1    0
 $EndComp
-Wire Wire Line
-	10000 3800 9050 3800
-$Comp
-L Device:R R?
+$Comp
+L Device:R R58
 U 1 1 609BC9D3
 P 10150 4150
-F 0 "R?" V 9943 4150 50  0000 C CNN
+F 0 "R58" V 9943 4150 50  0000 C CNN
 F 1 "10R" V 10034 4150 50  0000 C CNN
 F 2 "Resistor_SMD:R_1206_3216Metric" V 10080 4150 50  0001 C CNN
@@
 P 6350 5100
 AR Path="/608DBC83/609BF4B9" Ref="R?"  Part="1"
-AR Path="/60A756E2/609BF4B9" Ref="R?"  Part="1"
-F 0 "R?" H 6420 5146 50  0000 L CNN
+AR Path="/60A756E2/609BF4B9" Ref="R55"  Part="1"
+F 0 "R55" H 6420 5146 50  0000 L CNN
 F 1 "1k" H 6420 5055 50  0000 L CNN
 F 2 "Resistor_SMD:R_1206_3216Metric" V 6280 5100 50  0001 C CNN
@@
 P 6550 6000
 AR Path="/608DBC83/609C36A8" Ref="R?"  Part="1"
-AR Path="/60A756E2/609C36A8" Ref="R?"  Part="1"
-F 0 "R?" H 6620 6046 50  0000 L CNN
+AR Path="/60A756E2/609C36A8" Ref="R56"  Part="1"
+F 0 "R56" H 6620 6046 50  0000 L CNN
 F 1 "1k" H 6620 5955 50  0000 L CNN
 F 2 "Resistor_SMD:R_1206_3216Metric" V 6480 6000 50  0001 C CNN
@@
 $EndComp
 $Comp
-L power:GNDPWR #PWR?
+L power:GNDPWR #PWR0105
 U 1 1 609C3BAE
 P 6550 6250
-F 0 "#PWR?" H 6550 6050 50  0001 C CNN
+F 0 "#PWR0105" H 6550 6050 50  0001 C CNN
 F 1 "GNDPWR" H 6554 6096 50  0000 C CNN
 F 2 "" H 6550 6200 50  0001 C CNN
@@
 Wire Wire Line
 	6550 5400 8350 5400
+Connection ~ 7800 3150
+Wire Wire Line
+	7800 3150 8350 3150
+Wire Wire Line
+	8500 4150 10000 4150
+Wire Wire Line
+	8250 3800 10000 3800
+Connection ~ 7150 2750
+Wire Wire Line
+	7150 2750 8100 2750
+Connection ~ 5050 4900
+Wire Wire Line
+	5050 4900 5050 5000
 $EndSCHEMATC

Commit message: WIP Layout, TODO: DRC
Connections:
- net GND is gone; now on net GNDPWR: C34.1, C36.1, C37.1, C39.1
Changed lines of the file:
@@
 Wire Wire Line
 	5550 2550 6050 2550
-$Comp
-L power:GND #PWR?
-U 1 1 5F65EFB3
-P 6050 2550
-AR Path="/5F64F622/5F65CD72/5F65EFB3" Ref="#PWR?"  Part="1"
-AR Path="/5F64F622/5F70BF21/5F65EFB3" Ref="#PWR?"  Part="1"
-AR Path="/5F70C6BF/5F65EFB3" Ref="#PWR?"  Part="1"
-AR Path="/5F76DFEB/5F65EFB3" Ref="#PWR?"  Part="1"
-AR Path="/5F772CBD/5F65EFB3" Ref="#PWR?"  Part="1"
-AR Path="/5F777959/5F65EFB3" Ref="#PWR?"  Part="1"
-AR Path="/5F7F8851/5F7FE442/5F65EFB3" Ref="#PWR?"  Part="1"
-AR Path="/5F7F8851/5F7FE44C/5F65EFB3" Ref="#PWR?"  Part="1"
-AR Path="/5F8070C3/5F7FE442/5F65EFB3" Ref="#PWR?"  Part="1"
-AR Path="/5F8070C3/5F7FE44C/5F65EFB3" Ref="#PWR?"  Part="1"
-AR Path="/5F8AD0E2/5F7FE442/5F65EFB3" Ref="#PWR?"  Part="1"
-AR Path="/5F8AD0E2/5F7FE44C/5F65EFB3" Ref="#PWR?"  Part="1"
-AR Path="/5FA85ABF/5F7FE442/5F65EFB3" Ref="#PWR?"  Part="1"
-AR Path="/5FA85ABF/5F7FE44C/5F65EFB3" Ref="#PWR?"  Part="1"
-AR Path="/608DBC83/60A7272B/5F65EFB3" Ref="#PWR?"  Part="1"
-AR Path="/60A756E2/5F65EFB3" Ref="#PWR062"  Part="1"
-F 0 "#PWR062" H 6050 2300 50  0001 C CNN
-F 1 "GND" V 6055 2422 50  0000 R CNN
-F 2 "" H 6050 2550 50  0001 C CNN
-F 3 "" H 6050 2550 50  0001 C CNN
-	1    6050 2550
-	0    -1   -1   0
-$EndComp
-$Comp
-L power:GND #PWR?
-U 1 1 5F65EFB9
-P 6050 2250
-AR Path="/5F64F622/5F65CD72/5F65EFB9" Ref="#PWR?"  Part="1"
-AR Path="/5F64F622/5F70BF21/5F65EFB9" Ref="#PWR?"  Part="1"
-AR Path="/5F70C6BF/5F65EFB9" Ref="#PWR?"  Part="1"
-AR Path="/5F76DFEB/5F65EFB9" Ref="#PWR?"  Part="1"
-AR Path="/5F772CBD/5F65EFB9" Ref="#PWR?"  Part="1"
-AR Path="/5F777959/5F65EFB9" Ref="#PWR?"  Part="1"
-AR Path="/5F7F8851/5F7FE442/5F65EFB9" Ref="#PWR?"  Part="1"
-AR Path="/5F7F8851/5F7FE44C/5F65EFB9" Ref="#PWR?"  Part="1"
-AR Path="/5F8070C3/5F7FE442/5F65EFB9" Ref="#PWR?"  Part="1"
-AR Path="/5F8070C3/5F7FE44C/5F65EFB9" Ref="#PWR?"  Part="1"
-AR Path="/5F8AD0E2/5F7FE442/5F65EFB9" Ref="#PWR?"  Part="1"
-AR Path="/5F8AD0E2/5F7FE44C/5F65EFB9" Ref="#PWR?"  Part="1"
-AR Path="/5FA85ABF/5F7FE442/5F65EFB9" Ref="#PWR?"  Part="1"
-AR Path="/5FA85ABF/5F7FE44C/5F65EFB9" Ref="#PWR?"  Part="1"
-AR Path="/608DBC83/60A7272B/5F65EFB9" Ref="#PWR?"  Part="1"
-AR Path="/60A756E2/5F65EFB9" Ref="#PWR061"  Part="1"
-F 0 "#PWR061" H 6050 2000 50  0001 C CNN
-F 1 "GND" V 6055 2122 50  0000 R CNN
-F 2 "" H 6050 2250 50  0001 C CNN
-F 3 "" H 6050 2250 50  0001 C CNN
-	1    6050 2250
-	0    -1   -1   0
-$EndComp
 Wire Wire Line
 	5950 2250 6050 2250
@@
 Wire Wire Line
 	4200 1250 4500 1250
-$Comp
-L power:GND #PWR?
-U 1 1 5F65EFCC
-P 4950 1250
-AR Path="/5F64F622/5F65CD72/5F65EFCC" Ref="#PWR?"  Part="1"
-AR Path="/5F64F622/5F70BF21/5F65EFCC" Ref="#PWR?"  Part="1"
-AR Path="/5F70C6BF/5F65EFCC" Ref="#PWR?"  Part="1"
-AR Path="/5F76DFEB/5F65EFCC" Ref="#PWR?"  Part="1"
-AR Path="/5F772CBD/5F65EFCC" Ref="#PWR?"  Part="1"
-AR Path="/5F777959/5F65EFCC" Ref="#PWR?"  Part="1"
-AR Path="/5F7F8851/5F7FE442/5F65EFCC" Ref="#PWR?"  Part="1"
-AR Path="/5F7F8851/5F7FE44C/5F65EFCC" Ref="#PWR?"  Part="1"
-AR Path="/5F8070C3/5F7FE442/5F65EFCC" Ref="#PWR?"  Part="1"
-AR Path="/5F8070C3/5F7FE44C/5F65EFCC" Ref="#PWR?"  Part="1"
-AR Path="/5F8AD0E2/5F7FE442/5F65EFCC" Ref="#PWR?"  Part="1"
-AR Path="/5F8AD0E2/5F7FE44C/5F65EFCC" Ref="#PWR?"  Part="1"
-AR Path="/5FA85ABF/5F7FE442/5F65EFCC" Ref="#PWR?"  Part="1"
-AR Path="/5FA85ABF/5F7FE44C/5F65EFCC" Ref="#PWR?"  Part="1"
-AR Path="/608DBC83/60A7272B/5F65EFCC" Ref="#PWR?"  Part="1"
-AR Path="/60A756E2/5F65EFCC" Ref="#PWR060"  Part="1"
-F 0 "#PWR060" H 4950 1000 50  0001 C CNN
-F 1 "GND" V 4955 1122 50  0000 R CNN
-F 2 "" H 4950 1250 50  0001 C CNN
-F 3 "" H 4950 1250 50  0001 C CNN
-	1    4950 1250
-	0    -1   -1   0
-$EndComp
 Wire Wire Line
 	4950 1250 4800 1250
@@
 Wire Wire Line
 	5050 4900 5350 4900
-$Comp
-L power:GND #PWR?
-U 1 1 60992A9E
-P 5800 4900
-AR Path="/5F64F622/5F65CD72/60992A9E" Ref="#PWR?"  Part="1"
-AR Path="/5F64F622/5F70BF21/60992A9E" Ref="#PWR?"  Part="1"
-AR Path="/5F70C6BF/60992A9E" Ref="#PWR?"  Part="1"
-AR Path="/5F76DFEB/60992A9E" Ref="#PWR?"  Part="1"
-AR Path="/5F772CBD/60992A9E" Ref="#PWR?"  Part="1"
-AR Path="/5F777959/60992A9E" Ref="#PWR?"  Part="1"
-AR Path="/5F7F8851/5F7FE442/60992A9E" Ref="#PWR?"  Part="1"
-AR Path="/5F7F8851/5F7FE44C/60992A9E" Ref="#PWR?"  Part="1"
-AR Path="/5F8070C3/5F7FE442/60992A9E" Ref="#PWR?"  Part="1"
-AR Path="/5F8070C3/5F7FE44C/60992A9E" Ref="#PWR?"  Part="1"
-AR Path="/5F8AD0E2/5F7FE442/60992A9E" Ref="#PWR?"  Part="1"
-AR Path="/5F8AD0E2/5F7FE44C/60992A9E" Ref="#PWR?"  Part="1"
-AR Path="/5FA85ABF/5F7FE442/60992A9E" Ref="#PWR?"  Part="1"
-AR Path="/5FA85ABF/5F7FE44C/60992A9E" Ref="#PWR?"  Part="1"
-AR Path="/608DBC83/60A7272B/60992A9E" Ref="#PWR?"  Part="1"
-AR Path="/60A756E2/60992A9E" Ref="#PWR0102"  Part="1"
-F 0 "#PWR0102" H 5800 4650 50  0001 C CNN
-F 1 "GND" V 5805 4772 50  0000 R CNN
-F 2 "" H 5800 4900 50  0001 C CNN
-F 3 "" H 5800 4900 50  0001 C CNN
-	1    5800 4900
-	0    -1   -1   0
-$EndComp
 Wire Wire Line
 	5800 4900 5650 4900
@@
 Wire Wire Line
 	5050 4900 5050 5000
+$Comp
+L power:GNDPWR #PWR0106
+U 1 1 60B7151F
+P 4950 1250
+F 0 "#PWR0106" H 4950 1050 50  0001 C CNN
+F 1 "GNDPWR" H 4954 1096 50  0000 C CNN
+F 2 "" H 4950 1200 50  0001 C CNN
+F 3 "" H 4950 1200 50  0001 C CNN
+	1    4950 1250
+	0    -1   -1   0
+$EndComp
+$Comp
+L power:GNDPWR #PWR0102
+U 1 1 60B7CDD7
+P 5800 4900
+F 0 "#PWR0102" H 5800 4700 50  0001 C CNN
+F 1 "GNDPWR" H 5804 4746 50  0000 C CNN
+F 2 "" H 5800 4850 50  0001 C CNN
+F 3 "" H 5800 4850 50  0001 C CNN
+	1    5800 4900
+	0    -1   -1   0
+$EndComp
+$Comp
+L power:GNDPWR #PWR0107
+U 1 1 60B8E8B5
+P 6050 2250
+F 0 "#PWR0107" H 6050 2050 50  0001 C CNN
+F 1 "GNDPWR" H 6054 2096 50  0000 C CNN
+F 2 "" H 6050 2200 50  0001 C CNN
+F 3 "" H 6050 2200 50  0001 C CNN
+	1    6050 2250
+	0    -1   -1   0
+$EndComp
+$Comp
+L power:GNDPWR #PWR0108
+U 1 1 60B8EEF0
+P 6050 2550
+F 0 "#PWR0108" H 6050 2350 50  0001 C CNN
+F 1 "GNDPWR" H 6054 2396 50  0000 C CNN
+F 2 "" H 6050 2500 50  0001 C CNN
+F 3 "" H 6050 2500 50  0001 C CNN
+	1    6050 2550
+	0    -1   -1   0
+$EndComp
 $EndSCHEMATC
