File: kicad/arduino-nano.sch (KiCad schematic (older format))
At the start: 28 parts, among them J4 USB_B, J5 AVR ISP, SW5 Reset, U4 CH340C, U5 ATmega328P-AU, Y1 16MHz

Commit message: Kleine Anpassungen in KiCad-SCH und Firmware
Parts:
- U4: symbol htl_ics:CH340C -> jbc-miniregler-rescue:CH340C-htl_ics
Changed lines of the file:
@@
 	3750 5500 3750 5800
 $Comp
-L htl_ics:CH340C U?
+L jbc-miniregler-rescue:CH340C-htl_ics U?
 U 1 1 60944AF4
 P 3750 6400
@@
 AR Path="/608DBC3C/60930C19/60930D3D/60944AF4" Ref="U?"  Part="1"
 AR Path="/608DBC3C/60930C19/60944AF4" Ref="U4"  Part="1"
+AR Path="/60944AF4" Ref="U4"  Part="1"
 F 0 "U4" H 3350 7000 50  0000 C CNN
 F 1 "CH340C" H 3950 5850 50  0000 C CNN
