File: kicad/dcdc-12v.kicad_sch (KiCad schematic)
At the start: 12 parts, among them U2 XL7005A

Commit message: BOM auf Lieferbarkeit aktualisiert, TODO: DRC bereinigen
Parts:
- R20, R21: DistOrderNr C229599 -> C137292
Changed lines of the file:
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@@
       (effects (font (size 1.27 1.27)) hide)
     )
-    (property "DistOrderNr" "C229599" (id 5) (at 167.64 107.95 0)
+    (property "DistOrderNr" "C137292" (id 5) (at 167.64 107.95 0)
       (effects (font (size 1.27 1.27)) hide)
     )
@@
       (effects (font (size 1.27 1.27)) hide)
     )
-    (property "DistOrderNr" "C229599" (id 5) (at 207.01 96.52 0)
-      (effects (font (size 1.27 1.27)) hide)
-    )
+    (property "DistOrderNr" "C137292" (id 5) (at 207.01 96.52 0)
+      (effects (font (size 1.27 1.27)) hide)
+    )
