File: kicad/dcdc-3,3v.kicad_sch (KiCad schematic)
At the start: 12 parts, among them U3 XL7005A

Commit message: BOM auf Lieferbarkeit aktualisiert, TODO: DRC bereinigen
Parts:
- R25: DistOrderNr C140005 -> C25392
Changed lines of the file:
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@@
       (effects (font (size 1.27 1.27)) hide)
     )
-    (property "DistOrderNr" "C140005" (id 5) (at 204.47 90.17 0)
+    (property "DistOrderNr" "C25392" (id 5) (at 204.47 90.17 0)
       (effects (font (size 1.27 1.27)) hide)
     )
