File: kicad/power-supply.kicad_sch (KiCad schematic)
At the start: 25 parts, among them Q1 2N7002, Q2 MMBT3904, Q3 MMBT3904, Q4 ZXMP10A13FTA, SW5 Ein/Aus, X4 GND-Öse

Commit message: BOM auf Lieferbarkeit aktualisiert, TODO: DRC bereinigen
Parts:
- F1, Item4: DistOrderNr C182320 -> C3130
- Q1: DistOrderNr C181082 -> C350313
Changed lines of the file:
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@@
       (effects (font (size 1.27 1.27)) hide)
     )
-    (property "DistOrderNr" "C182320" (id 5) (at 43.18 38.1 0)
+    (property "DistOrderNr" "C3130" (id 5) (at 43.18 38.1 0)
       (effects (font (size 1.27 1.27)) hide)
     )
@@
       (effects (font (size 1.27 1.27)) (justify left) hide)
     )
-    (property "DistOrderNr" "C181082" (id 4) (at 45.72 133.35 0)
+    (property "DistOrderNr" "C350313" (id 4) (at 45.72 133.35 0)
       (effects (font (size 1.27 1.27)) hide)
     )
@@
       (effects (font (size 1.27 1.27)) hide)
     )
-    (property "DistOrderNr" "C182320" (id 5) (at 43.18 20.32 0)
-      (effects (font (size 1.27 1.27)) hide)
-    )
+    (property "DistOrderNr" "C3130" (id 5) (at 43.18 20.32 0)
+      (effects (font (size 1.27 1.27)) hide)
+    )
