File: kicad/uart-rs232-rs485.kicad_sch (KiCad schematic)
At the start: 21 parts, among them U4 MAX3232, U5 YD3082EESA

Commit message: BOM auf Lieferbarkeit aktualisiert, TODO: DRC bereinigen
Parts:
- R26: DistOrderNr C229599 -> C137292
Changed lines of the file:
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@@
       (effects (font (size 1.27 1.27)) hide)
     )
-    (property "DistOrderNr" "C229599" (id 5) (at 99.06 151.13 0)
+    (property "DistOrderNr" "C137292" (id 5) (at 99.06 151.13 0)
       (effects (font (size 1.27 1.27)) hide)
     )
